Commit message: Updated to the latest meshes from Mike1.

File: robots/BHD280_URDF.URDF (robot description, URDF)
Before this commit: robot BHD280_URDF, 9 links, 8 joints
Links:
- link finger0_1: mass 31321.121421294 -> 31321.1214212939
- link finger2_1: mass 31321.121421294 -> 31321.1214212939
Joints:
- joint j01: origin xyz=0.0500000000000006 0.000799999999999964 0 rpy=1.5707963267949 0 0 -> xyz=0.0500000000000007 0.000799999999999971 0 rpy=1.5707963267949 0 0
- joint j10: axis -0.00584481507867448 0 -0.999982918922466 -> 0.0058448 0 0.99998; origin xyz=0.025 0 0.0754000000000004 rpy=-9.28709853220239E-30 -0.00584484835748173 -1.5707963267949 -> xyz=0.025 0 0.0754 rpy=-9.2871E-30 -0.0058448 -1.5708
- joint j11: origin xyz=0.0499991459461259 0.000799999999999367 -0.000292240753933651 rpy=1.5707963267949 0 -4.93038065763132E-32 -> xyz=0.0499991459461259 0.000799999999999367 -0.000292240753933679 rpy=1.5707963267949 0 -4.93038065763132E-32
- joint j12: origin xyz=0.0699356847396164 0.00300000000001083 0.000199999999999378 rpy=1.95799899548702E-16 2.29686057908074E-16 0.700079983587682 -> xyz=0.0699356847396015 0.00300000000003377 0.000199999999999378 rpy=1.95799899548702E-16 2.29686057908074E-16 0.700079983587682

File: robots/HERB_BASE_URDF.URDF (robot description, URDF)
Before this commit: robot HERB_BASE_URDF, 5 links, 4 joints
Joints:
- joint head/wam2: axis 0 0 1 -> 0 0 -1; origin xyz=0 0 0 rpy=1.5708 0 4.208E-14 -> xyz=0 0 0 rpy=1.5707963267949 0 4.20797196041016E-14

File: robots/WAM_URDF.URDF (robot description, URDF)
Before this commit: robot WAM_URDF, 8 links, 7 joints
Links:
- link wam1: mass 12.6535414859625 -> 12.6535414859626
Joints:
- joint j3: origin xyz=0 0 0 rpy=1.5707963267949 -3.94430452610506E-31 4.02814495500316E-16 -> xyz=0 0 0 rpy=1.5708 -3.9443E-31 4.0281E-16
- joint j4: origin xyz=0.0450000000000029 0 0.550000000000001 rpy=-1.5707963267949 0 0 -> xyz=0.045 0 0.55 rpy=-1.5708 0 0
- joint j7: origin xyz=0 0 0 rpy=1.5707963267949 0 0 -> xyz=0 0 0 rpy=1.5708 0 0
