Commit message: set wam4 adjacent to wam7 for both arms

File: robots/wam.urdf.xacro (robot description, xacro)
@@ -1,4 +1,179 @@
-<robot xmlns:xacro="http://www.ros.org/wiki/xacro" name="wam">
-    <xacro:include filename="wam.urdf.xacro"/>
-    <xacro:wam prefix=""/>
-</robot>
+<robot xmlns:xacro="http://www.ros.org/wiki/xacro" name="wam"><xacro:macro params="prefix" name="wam"><link name="${prefix}/wam_base">
+    <visual>
+      <origin xyz="0 0 0" rpy="0 0 0"/>
+      <geometry>
+        <mesh filename="package://herb_description/meshes/wam_base.STL"/>
+      </geometry>
+      <material name="">
+        <color rgba="0.792156862745098 0.819607843137255 0.933333333333333 1"/>
+      </material>
+    </visual>
+    <inertial>
+      <origin xyz="-0.02017671 -0.26604706 -0.14071720"/>
+      <mass value="9.97059584"/>
+      <inertia ixx="0.10916849" ixy="0.00640270" ixz="0.02557874" iyy="0.18294303" iyz="0.00161433" izz="0.11760385"/>
+    </inertial>
+  <collision><geometry><mesh filename="package://herb_description/meshes/wam_base_collision.STL"/></geometry></collision></link>
+  <link name="${prefix}/wam1">
+    <visual>
+      <origin xyz="0 0 0" rpy="0 0 0"/>
+      <geometry>
+        <mesh filename="package://herb_description/meshes/wam1.STL"/>
+      </geometry>
+      <material name="">
+        <color rgba="0.792156862745098 0.819607843137255 0.933333333333333 1"/>
+      </material>
+    </visual>
+    <inertial>
+      <origin xyz="-0.00443422 0.12189039 -0.00066489"/>
+      <mass value="10.76768767"/>
+      <inertia ixx="0.13488033" ixy="-0.00213041" ixz="-0.00012485" iyy="0.11328369" iyz="0.00068555" izz="0.09046330"/>
+    </inertial>
+  <collision><geometry><mesh filename="package://herb_description/meshes/wam1_collision.STL"/></geometry></collision></link>
+  <joint name="${prefix}/j1" type="revolute">
+    <origin xyz="0.22 0.14 0.346" rpy="-1.1127E-16 0 0"/>
+    <parent link="${prefix}/wam_base"/>
+    <child link="${prefix}/wam1"/>
+    <axis xyz="0 0 1"/>
+  <!-- HERB's J1 joints are modified to have a +180 degree offset. -->
+    <limit effort="1.8" lower="0.523598775598" upper="5.75958653158" velocity="0.75"/>
+  </joint>
+  <link name="${prefix}/wam2">
+    <visual>
+      <origin xyz="0 0 0" rpy="0 0 0"/>
+      <geometry>
+        <mesh filename="package://herb_description/meshes/wam2.STL"/>
+      </geometry>
+      <material name="">
+        <color rgba="0.792156862745098 0.819607843137255 0.933333333333333 1"/>
+      </material>
+    </visual>
+    <inertial>
+      <origin xyz="-0.00236983 0.03105614 0.01542114"/>
+      <mass value="3.87493756"/>
+      <inertia ixx="0.02140958" ixy="0.00027172" ixz="+0.00002461" iyy="0.01377875" iyz="-0.00181920" izz="0.01558906"/>
+    </inertial>
+  <collision><geometry><mesh filename="package://herb_description/meshes/wam2_collision.STL"/></geometry></collision></link>
+  <joint name="${prefix}/j2" type="revolute">
+    <origin xyz="0 0 0" rpy="-1.5708 -4.0281E-16 -3.9443E-31"/>
+    <parent link="${prefix}/wam1"/>
+    <child link="${prefix}/wam2"/>
+    <axis xyz="0 0 1"/>
+  <limit effort="1.8" lower="-1.97222205475" upper="1.97222205475" velocity="0.75"/>
+  </joint>
+  <link name="${prefix}/wam3">
+    <visual>
+      <origin xyz="0 0 0" rpy="0 0 0"/>
+      <geometry>
+        <mesh filename="package://herb_description/meshes/wam3.STL"/>
+      </geometry>
+      <material name="">
+        <color rgba="0.792156862745098 0.819607843137255 0.933333333333333 1"/>
+      </material>
+    </visual>
+    <inertial>
+      <origin xyz="-0.03825858 0.20750770 0.00003309"/>
+      <mass value="1.80228141"/>
+      <inertia ixx="0.05911077" ixy="-0.00249612" ixz="0.00000738" iyy="0.00324550" iyz="-0.00001767" izz="0.05927043"/>
+    </inertial>
+  <collision><geometry><mesh filename="package://herb_description/meshes/wam3_collision.STL"/></geometry></collision></link>
+  <joint name="${prefix}/j3" type="revolute">
+    <origin xyz="0 0 0" rpy="1.5708 -3.9443E-31 4.0281E-16"/>
+    <parent link="${prefix}/wam2"/>
+    <child link="${prefix}/wam3"/>
+    <axis xyz="0 0 1"/>
+  <limit effort="1.8" lower="-2.74016692563" upper="2.74016692563" velocity="2.0"/>
+  </joint>
+  <link name="${prefix}/wam4">
+    <visual>
+      <origin xyz="0 0 0" rpy="0 0 0"/>
+      <geometry>
+        <mesh filename="package://herb_description/meshes/wam4.STL"/>
+      </geometry>
+      <material name="">
+        <color rgba="0.792156862745098 0.819607843137255 0.933333333333333 1"/>
+      </material>
+    </visual>
+    <inertial>
+      <origin xyz="0.00498512 -0.00022942 0.13271662"/>
+      <mass value="2.40016804"/>
+      <inertia ixx="0.01491672" ixy="0.00001741" ixz="-0.00150604" iyy="0.01482922" iyz="-0.00002109" izz="0.00294463"/>
+    </inertial>
+  <collision><geometry><mesh filename="package://herb_description/meshes/wam4_collision.STL"/></geometry></collision></link>
+  <joint name="${prefix}/j4" type="revolute">
+    <origin xyz="0.045 0 0.55" rpy="-1.5708 0 0"/>
+    <parent link="${prefix}/wam3"/>
+    <child link="${prefix}/wam4"/>
+    <axis xyz="0 0 1"/>
+  <limit effort="1.6" lower="-0.872664625997" upper="3.14159265359" velocity="2.0"/>
+  </joint>
+  <link name="${prefix}/wam5">
+    <visual>
+      <origin xyz="0 0 0" rpy="0 0 0"/>
+      <geometry>
+        <mesh filename="package://herb_description/meshes/wam5.STL"/>
+      </geometry>
+      <material name="">
+        <color rgba="0.792156862745098 0.819607843137255 0.933333333333333 1"/>
+      </material>
+    </visual>
+    <inertial>
+      <origin xyz="0.00008921 0.00511217 0.00435824"/>
+      <mass value="0.12376019"/>
+      <inertia ixx="0.00005029" ixy="0.00000020" ixz="-0.00000005" iyy="0.00007582" iyz="-0.00000359" izz="0.00006270"/>
+    </inertial>
+  <collision><geometry><mesh filename="package://herb_description/meshes/wam5_collision.STL"/></geometry></collision></link>
+  <joint name="${prefix}/j5" type="revolute">
+    <origin xyz="-0.045 0 0" rpy="1.5708 0 0"/>
+    <parent link="${prefix}/wam4"/>
+    <child link="${prefix}/wam5"/>
+    <axis xyz="0 0 1"/>
+  <limit effort="0.6" lower="-4.76474885794" upper="1.23918376892" velocity="2.5"/>
+  </joint>
+  <link name="${prefix}/wam6">
+    <visual>
+      <origin xyz="0 0 0" rpy="0 0 0"/>
+      <geometry>
+        <mesh filename="package://herb_description/meshes/wam6.STL"/>
+      </geometry>
+      <material name="">
+        <color rgba="0.792156862745098 0.819607843137255 0.933333333333333 1"/>
+      </material>
+    </visual>
+    <inertial>
+      <origin xyz="-0.00012262 -0.01703194 0.02468336"/>
+      <mass value="0.41797364"/>
+      <inertia ixx="0.00055516" ixy="0.00000061" ixz="-0.00000074" iyy="0.00024367" iyz="-0.00004590" izz="0.00045358"/>
+    </inertial>
+  <collision><geometry><mesh filename="package://herb_description/meshes/wam6_collision.STL"/></geometry></collision></link>
+  <joint name="${prefix}/j6" type="revolute">
+    <origin xyz="0 0 0.3" rpy="-1.5708 0 0"/>
+    <parent link="${prefix}/wam5"/>
+    <child link="${prefix}/wam6"/>
+    <axis xyz="0 0 1"/>
+  <limit effort="0.6" lower="-1.5707963268" upper="1.5707963268" velocity="2.5"/>
+  </joint>
+  <link name="${prefix}/wam7">
+    <visual>
+      <origin xyz="0 0 0" rpy="0 0 0"/>
+      <geometry>
+        <mesh filename="package://herb_description/meshes/wam7.STL"/>
+      </geometry>
+      <material name="">
+        <color rgba="0.792156862745098 0.819607843137255 0.933333333333333 1"/>
+      </material>
+    </visual>
+    <inertial>
+      <origin xyz="-0.00007974 0.00016313 -0.00323552"/>
+      <mass value="0.06864753"/>
+      <inertia ixx="0.00003773" ixy="-0.00000019" ixz="0.00000000" iyy="0.00003806" iyz="0.00000000" izz="0.00007408"/>
+    </inertial>
+  <collision><geometry><mesh filename="package://herb_description/meshes/wam7_collision.STL"/></geometry></collision></link>
+  <joint name="${prefix}/j7" type="revolute">
+    <origin xyz="0 0 0" rpy="1.5708 0 0"/>
+    <parent link="${prefix}/wam6"/>
+    <child link="${prefix}/wam7"/>
+    <axis xyz="0 0 1"/>
+  <limit effort="0.174" lower="-3.00196631343" upper="3.00196631343" velocity="2.5"/>
+  </joint>
+</xacro:macro></robot>
