Commit message: Fixing bug in xacro definition

File: robots/bh280_standalone.srdf.xacro (robot description, xacro)
@@ -1,71 +1,69 @@
 <robot xmlns:xacro="http://www.ros.org/wiki/xacro" name="bh280">
-    <xacro:macro name="bh280_hand">
-        <group name="hand">
-            <link name="/hand_base"/>
-            <link name="/finger0_0"/>
-            <link name="/finger0_1"/>
-            <link name="/finger0_2"/>
-            <link name="/finger1_0"/>
-            <link name="/finger1_1"/>
-            <link name="/finger1_2"/>
-            <link name="/finger2_1"/>
-            <link name="/finger2_2"/>
-        </group>
-        <!-- Disable collisions between the fingers. -->
-        <disable_collisions link1="/finger0_0" link2="/finger1_0"/>
-        <disable_collisions link1="/finger0_0" link2="/finger0_1"/>
-        <disable_collisions link1="/finger0_0" link2="/finger0_2"/>
-        <disable_collisions link1="/finger0_0" link2="/finger1_1"/>
-        <disable_collisions link1="/finger0_0" link2="/finger1_2"/>
-        <disable_collisions link1="/finger0_0" link2="/finger2_1"/>
-        <disable_collisions link1="/finger0_0" link2="/finger2_2"/>
-        <disable_collisions link1="/finger1_0" link2="/finger0_1"/>
-        <disable_collisions link1="/finger1_0" link2="/finger0_2"/>
-        <disable_collisions link1="/finger1_0" link2="/finger1_1"/>
-        <disable_collisions link1="/finger1_0" link2="/finger1_2"/>
-        <disable_collisions link1="/finger1_0" link2="/finger2_1"/>
-        <disable_collisions link1="/finger1_0" link2="/finger2_2"/>
-        <disable_collisions link1="/finger0_1" link2="/finger0_2"/>
-        <disable_collisions link1="/finger0_1" link2="/finger1_1"/>
-        <disable_collisions link1="/finger0_1" link2="/finger1_2"/>
-        <disable_collisions link1="/finger0_1" link2="/finger2_1"/>
-        <disable_collisions link1="/finger0_1" link2="/finger2_2"/>
-        <disable_collisions link1="/finger0_2" link2="/finger1_1"/>
-        <disable_collisions link1="/finger0_2" link2="/finger1_2"/>
-        <disable_collisions link1="/finger0_2" link2="/finger2_1"/>
-        <disable_collisions link1="/finger0_2" link2="/finger2_2"/>
-        <disable_collisions link1="/finger1_1" link2="/finger1_2"/>
-        <disable_collisions link1="/finger1_1" link2="/finger2_1"/>
-        <disable_collisions link1="/finger1_1" link2="/finger2_2"/>
-        <disable_collisions link1="/finger1_2" link2="/finger2_1"/>
-        <disable_collisions link1="/finger1_2" link2="/finger2_2"/>
-        <disable_collisions link1="/finger2_1" link2="/finger2_2"/>
-        <!-- Disable collisions between the fingers and the palm. -->
-        <disable_collisions link1="/hand_base" link2="/finger1_0"/>
-        <disable_collisions link1="/hand_base" link2="/finger0_1"/>
-        <disable_collisions link1="/hand_base" link2="/finger0_2"/>
-        <disable_collisions link1="/hand_base" link2="/finger1_1"/>
-        <disable_collisions link1="/hand_base" link2="/finger1_2"/>
-        <disable_collisions link1="/hand_base" link2="/finger2_1"/>
-        <disable_collisions link1="/hand_base" link2="/finger2_2"/>
-        <!-- Sphere representation for CHOMP -->
-        <link_sphere_approximation link="/finger0_1">
-            <sphere center="0.05 -0.01 0.0" radius="0.04"/>
-        </link_sphere_approximation>
-        <link_sphere_approximation link="/finger1_1">
-            <sphere center="0.05 -0.01 0.0" radius="0.04"/>
-        </link_sphere_approximation>
-        <link_sphere_approximation link="/finger2_1">
-            <sphere center="0.05 -0.01 0.0" radius="0.04"/>
-        </link_sphere_approximation>
-        <link_sphere_approximation link="/finger0_2">
-            <sphere center="0.05 0.0 0.0" radius="0.04"/>
-        </link_sphere_approximation>
-        <link_sphere_approximation link="/finger1_2">
-            <sphere center="0.05 0.0 0.0" radius="0.04"/>
-        </link_sphere_approximation>
-        <link_sphere_approximation link="/finger2_2">
-            <sphere center="0.05 0.0 0.0" radius="0.04"/>
-        </link_sphere_approximation>
-    </xacro:macro>
+   <group name="hand">
+        <link name="/hand_base"/>
+        <link name="/finger0_0"/>
+        <link name="/finger0_1"/>
+        <link name="/finger0_2"/>
+        <link name="/finger1_0"/>
+        <link name="/finger1_1"/>
+        <link name="/finger1_2"/>
+        <link name="/finger2_1"/>
+        <link name="/finger2_2"/>
+    </group>
+    <!-- Disable collisions between the fingers. -->
+    <disable_collisions link1="/finger0_0" link2="/finger1_0"/>
+    <disable_collisions link1="/finger0_0" link2="/finger0_1"/>
+    <disable_collisions link1="/finger0_0" link2="/finger0_2"/>
+    <disable_collisions link1="/finger0_0" link2="/finger1_1"/>
+    <disable_collisions link1="/finger0_0" link2="/finger1_2"/>
+    <disable_collisions link1="/finger0_0" link2="/finger2_1"/>
+    <disable_collisions link1="/finger0_0" link2="/finger2_2"/>
+    <disable_collisions link1="/finger1_0" link2="/finger0_1"/>
+    <disable_collisions link1="/finger1_0" link2="/finger0_2"/>
+    <disable_collisions link1="/finger1_0" link2="/finger1_1"/>
+    <disable_collisions link1="/finger1_0" link2="/finger1_2"/>
+    <disable_collisions link1="/finger1_0" link2="/finger2_1"/>
+    <disable_collisions link1="/finger1_0" link2="/finger2_2"/>
+    <disable_collisions link1="/finger0_1" link2="/finger0_2"/>
+    <disable_collisions link1="/finger0_1" link2="/finger1_1"/>
+    <disable_collisions link1="/finger0_1" link2="/finger1_2"/>
+    <disable_collisions link1="/finger0_1" link2="/finger2_1"/>
+    <disable_collisions link1="/finger0_1" link2="/finger2_2"/>
+    <disable_collisions link1="/finger0_2" link2="/finger1_1"/>
+    <disable_collisions link1="/finger0_2" link2="/finger1_2"/>
+    <disable_collisions link1="/finger0_2" link2="/finger2_1"/>
+    <disable_collisions link1="/finger0_2" link2="/finger2_2"/>
+    <disable_collisions link1="/finger1_1" link2="/finger1_2"/>
+    <disable_collisions link1="/finger1_1" link2="/finger2_1"/>
+    <disable_collisions link1="/finger1_1" link2="/finger2_2"/>
+    <disable_collisions link1="/finger1_2" link2="/finger2_1"/>
+    <disable_collisions link1="/finger1_2" link2="/finger2_2"/>
+    <disable_collisions link1="/finger2_1" link2="/finger2_2"/>
+    <!-- Disable collisions between the fingers and the palm. -->
+    <disable_collisions link1="/hand_base" link2="/finger1_0"/>
+    <disable_collisions link1="/hand_base" link2="/finger0_1"/>
+    <disable_collisions link1="/hand_base" link2="/finger0_2"/>
+    <disable_collisions link1="/hand_base" link2="/finger1_1"/>
+    <disable_collisions link1="/hand_base" link2="/finger1_2"/>
+    <disable_collisions link1="/hand_base" link2="/finger2_1"/>
+    <disable_collisions link1="/hand_base" link2="/finger2_2"/>
+    <!-- Sphere representation for CHOMP -->
+    <link_sphere_approximation link="/finger0_1">
+        <sphere center="0.05 -0.01 0.0" radius="0.04"/>
+    </link_sphere_approximation>
+    <link_sphere_approximation link="/finger1_1">
+        <sphere center="0.05 -0.01 0.0" radius="0.04"/>
+    </link_sphere_approximation>
+    <link_sphere_approximation link="/finger2_1">
+        <sphere center="0.05 -0.01 0.0" radius="0.04"/>
+    </link_sphere_approximation>
+    <link_sphere_approximation link="/finger0_2">
+        <sphere center="0.05 0.0 0.0" radius="0.04"/>
+    </link_sphere_approximation>
+    <link_sphere_approximation link="/finger1_2">
+        <sphere center="0.05 0.0 0.0" radius="0.04"/>
+    </link_sphere_approximation>
+    <link_sphere_approximation link="/finger2_2">
+        <sphere center="0.05 0.0 0.0" radius="0.04"/>
+    </link_sphere_approximation>
 </robot>
