Commit message: Added the HERB model.

File: robots/HERB_BASE_URDF.URDF (robot description, URDF)
Before this commit: robot HERB_BASE_URDF, 5 links, 4 joints
Links:
- removed link head_pan
- removed link head_tilt
- removed link segway_left
- removed link segway_right
- added link head/wam1, mass 0.699914058257394; collision mesh filename=package://HERB_BASE_URDF/meshes/head_wam1.STL; visual mesh filename=package://HERB_BASE_URDF/meshes/head_wam1.STL
- added link head/wam2, mass 1.54049400601598; collision mesh filename=package://HERB_BASE_URDF/meshes/head_wam2.STL; visual mesh filename=package://HERB_BASE_URDF/meshes/head_wam2.STL
- added link segway_wheel_left, mass 6.7355511743555; collision mesh filename=package://HERB_BASE_URDF/meshes/segway_wheel_left.STL; visual mesh filename=package://HERB_BASE_URDF/meshes/segway_wheel_left.STL
- added link segway_wheel_right, mass 6.7355511743555; collision mesh filename=package://HERB_BASE_URDF/meshes/segway_wheel_right.STL; visual mesh filename=package://HERB_BASE_URDF/meshes/segway_wheel_right.STL
Joints:
- removed joint head_pan
- removed joint head_tilt
- removed joint segway_left
- removed joint segway_right
- added joint head/wam1: type continuous, parent herb_base, child head/wam1, origin xyz=-0.219074999999998 3.49999999989525E-05 1.2737592 rpy=0 0 0, axis 0 0 1
- added joint head/wam2: type continuous, parent head/wam1, child head/wam2, origin xyz=0 0 0 rpy=1.5707963267949 0 4.20797196041016E-14, axis 0 0 -1
- added joint segway_wheel_left: type continuous, parent herb_base, child segway_wheel_left, origin xyz=0 0.231771918932663 0.23158735611353 rpy=-1.5707963267949 -0.115508699092541 0, axis 0 0 -1
- added joint segway_wheel_right: type continuous, parent herb_base, child segway_wheel_right, origin xyz=0 -0.231771918932663 0.231587356113537 rpy=-1.5707963267949 0.0751085369855802 3.14159265358979, axis 0 0 1

File: robots/WAM_URDF.URDF (robot description, URDF)
Before this commit: robot WAM_URDF, 8 links, 7 joints
Links:
- removed link wam0
- added link wam_base, mass 2.67334422899553; collision mesh filename=package://WAM_URDF/meshes/wam_base.STL; visual mesh filename=package://WAM_URDF/meshes/wam_base.STL
- link wam3: mass 5.1434E-05 -> 5.1434314783609E-05
- link wam4: mass 1.5356 -> 1.53559449158938
- link wam6: mass 0.18643 -> 0.186433706842734
- link wam7: mass 0.036704 -> 0.110863010879355
Joints:
- joint j1: origin xyz=0.22 0.14 0.346 rpy=-1.1127E-16 0 0 -> xyz=0.22 0.14 0.346 rpy=-1.11266916865798E-16 0 0; parent wam0 -> wam_base
- joint j2: origin xyz=0 0 0 rpy=-1.5708 -4.0281E-16 -3.9443E-31 -> xyz=0 0 0 rpy=-1.5707963267949 -4.02814495500316E-16 -3.94430452610506E-31
- joint j7: origin xyz=0 -0.0539500000000008 0 rpy=1.5707963267949 0 0 -> xyz=0 -0.0600000000000009 0 rpy=1.5707963267949 0 0

File: robots/herb.urdf.xacro (robot description, xacro)
@@ -10,6 +10,6 @@
         <xacro:wam prefix="${prefix}"/>
         <joint name="${prefix}/mount" type="fixed">
-            <!-- The force/torque sensor is 2 cm thick. -->
-            <origin xyz="0 0 0.02" rpy="0 0 ${-pi/2}"/>
+            <!-- The force/torque sensor is 12 mm thick. -->
+            <origin xyz="0 0 0.012" rpy="0 0 ${-pi/2}"/>
             <parent link="${prefix}/wam7"/>
             <child link="${prefix}/base_link"/>
@@ -21,10 +21,10 @@
         <xacro:wam_ft_bh280 prefix="/right"/>
         <joint name="/left/wam_mount" type="fixed">
-            <origin rpy="0 ${-pi/2} ${pi}"/>
+            <origin xyz="-0.2667 0.3307 0.68505" rpy="0 ${-pi/2} ${pi}"/>
             <parent link="/herb_base"/>
             <child link="/left/wam_base"/>
         </joint>
         <joint name="/right/wam_mount" type="fixed">
-            <origin rpy="0 ${-pi/2} ${pi}"/>
+            <origin xyz="-0.2667 -0.05069 0.68505" rpy="0 ${-pi/2} ${pi}"/>
             <parent link="/herb_base"/>
             <child link="/right/wam_base"/>

Commit message: Updated model

File: robots/HERB_BASE_URDF.URDF (robot description, URDF)
Before this commit: robot HERB_BASE_URDF, 5 links, 4 joints
Links:
- link head/wam2: mass 1.54049400601598 -> 1.54049400601599
- link herb_base: mass 118.073177712457 -> 118.064183849969
Joints:
- joint head/wam2: axis 0 0 -1 -> 0 0 1; origin xyz=0 0 0 rpy=1.5707963267949 0 4.20797196041016E-14 -> xyz=0 0 0 rpy=1.5708 0 4.208E-14

File: robots/WAM_URDF.URDF (robot description, URDF)
Before this commit: robot WAM_URDF, 8 links, 7 joints
Links:
- link wam1: mass 12.6535414859626 -> 12.6535414859625
- link wam2: mass 0.437815219798137 -> 0.437815219798136
Joints:
- joint j1: axis 0 0 -1 -> 0 0 1; origin xyz=0.22 0.14 0.346 rpy=-1.11266916865798E-16 0 0 -> xyz=0.22 0.14 0.346 rpy=-1.1127E-16 0 0
- joint j2: axis 0 0 -1 -> 0 0 1; origin xyz=0 0 0 rpy=-1.5707963267949 -4.02814495500316E-16 -3.94430452610506E-31 -> xyz=0 0 0 rpy=-1.5708 -4.0281E-16 -3.9443E-31
- joint j5: axis 0 0 -1 -> 0 0 1; origin xyz=-0.0449999999999992 0 0 rpy=1.5707963267949 0 0 -> xyz=-0.045 0 0 rpy=1.5708 0 0
- joint j6: axis 0 0 -1 -> 0 0 1; origin xyz=0 0 0.3 rpy=-1.5707963267949 0 0 -> xyz=0 0 0.3 rpy=-1.5708 0 0

Commit message: Fixed HERB's tilt axis.

File: robots/HERB_BASE_URDF.URDF (robot description, URDF)
Before this commit: robot HERB_BASE_URDF, 5 links, 4 joints
Joints:
- joint head/wam2: axis 0 0 -1 -> 0 0 1

Commit message: Updated WAM and head transforms for HERB 2.5.
Thanks to Michael Dawson-Haggerty for exporting the new measurements from
SolidWorks and verifying their accuracy on the real hardware.

File: robots/HERB_BASE_URDF.URDF (robot description, URDF)
Before this commit: robot HERB_BASE_URDF, 5 links, 4 joints
Joints:
- joint head/wam1: origin xyz=-0.219074999999998 3.49999999989525E-05 1.2737592 rpy=0 0 0 -> xyz=-0.219043 0 1.282513 rpy=0 0 0

File: robots/herb.urdf.xacro (robot description, xacro)
@@ -21,10 +21,10 @@
         <xacro:herb_base prefix=""/>
         <joint name="/left/wam_mount" type="fixed">
-            <origin xyz="-0.2667 0.3307 0.68505" rpy="0 ${-pi/2} ${pi}"/>
+            <origin xyz="-0.266700 0.332276 0.694588" rpy="0 ${-pi/2} ${pi}"/>
             <parent link="/herb_base"/>
             <child link="/left/wam_base"/>
         </joint>
         <joint name="/right/wam_mount" type="fixed">
-            <origin xyz="-0.2667 -0.05069 0.68505" rpy="0 ${-pi/2} ${pi}"/>
+            <origin xyz="-0.266700 -0.049121 0.694588" rpy="0 ${-pi/2} ${pi}"/>
             <parent link="/herb_base"/>
             <child link="/right/wam_base"/>

Commit message: first attempt fixed head model

File: robots/HERB_BASE_URDF.URDF (robot description, URDF)
Before this commit: robot HERB_BASE_URDF, 5 links, 4 joints
Joints:
- joint head/wam1: axis 0 0 1 -> (none); type continuous -> fixed
- joint head/wam2: axis 0 0 1 -> (none); origin xyz=0 0 0 rpy=1.5707963267949 0 4.20797196041016E-14 -> xyz=0 0 0 rpy=1.5707963267949 0 -2.99999999999958E-01; type continuous -> fixed

Commit message: seemingly correct fixed head tilt transform

File: robots/HERB_BASE_URDF.URDF (robot description, URDF)
Before this commit: robot HERB_BASE_URDF, 5 links, 4 joints
Joints:
- joint head/wam1: axis (none) -> 0 0 1
- joint head/wam2: axis (none) -> 0 0 1; origin xyz=0 0 0 rpy=1.5707963267949 0 -2.99999999999958E-01 -> xyz=0 0 0 rpy=1.5707963267949 0.3 4.20797196041016E-14; type fixed -> continuous
