Commit message: move meshes into subfolders

File: robots/bh280.urdf.xacro (robot description, xacro)
@@ -5,14 +5,14 @@
         <origin xyz="0 0 0" rpy="0 0 0"/>
         <geometry>
-          <mesh filename="package://herb_description/meshes/hand_base.dae"/>
-        </geometry>
-        <material name="">
-          <color rgba="0.752941176470588 0.752941176470588 0.752941176470588 1"/>
-        </material>
-      </visual>
-      <geometry_group name="fine_collision">
-        <origin rpy="0 0 0" xyz="0 0 0"/>
-        <geometry>
-          <mesh filename="package://herb_description/meshes/hand_base.STL"/>
+          <mesh filename="package://herb_description/meshes/bh280/hand_base.dae"/>
+        </geometry>
+        <material name="">
+          <color rgba="0.752941176470588 0.752941176470588 0.752941176470588 1"/>
+        </material>
+      </visual>
+      <geometry_group name="fine_collision">
+        <origin rpy="0 0 0" xyz="0 0 0"/>
+        <geometry>
+          <mesh filename="package://herb_description/meshes/bh280/hand_base.STL"/>
         </geometry>
       </geometry_group>
@@ -27,5 +27,5 @@
       <collision>
         <geometry>
-          <mesh filename="package://herb_description/meshes/hand_base_collision.STL"/>
+          <mesh filename="package://herb_description/meshes/bh280/hand_base_collision.STL"/>
         </geometry>
       </collision>
@@ -35,14 +35,14 @@
         <origin xyz="0 0 0" rpy="0 0 0"/>
         <geometry>
-          <mesh filename="package://herb_description/meshes/finger0_0.dae"/>
-        </geometry>
-        <material name="">
-          <color rgba="0.752941176470588 0.752941176470588 0.752941176470588 1"/>
-        </material>
-      </visual>
-      <geometry_group name="fine_collision">
-        <origin rpy="0 0 0" xyz="0 0 0"/>
-        <geometry>
-          <mesh filename="package://herb_description/meshes/finger0_0.STL"/>
+          <mesh filename="package://herb_description/meshes/bh280/finger0_0.dae"/>
+        </geometry>
+        <material name="">
+          <color rgba="0.752941176470588 0.752941176470588 0.752941176470588 1"/>
+        </material>
+      </visual>
+      <geometry_group name="fine_collision">
+        <origin rpy="0 0 0" xyz="0 0 0"/>
+        <geometry>
+          <mesh filename="package://herb_description/meshes/bh280/finger0_0.STL"/>
         </geometry>
       </geometry_group>
@@ -57,5 +57,5 @@
       <collision>
         <geometry>
-          <mesh filename="package://herb_description/meshes/finger0_0_collision.STL"/>
+          <mesh filename="package://herb_description/meshes/bh280/finger0_0_collision.STL"/>
         </geometry>
       </collision>
@@ -72,14 +72,14 @@
         <origin xyz="0 0 0" rpy="0 0 0"/>
         <geometry>
-          <mesh filename="package://herb_description/meshes/finger0_1.dae"/>
-        </geometry>
-        <material name="">
-          <color rgba="0.752941176470588 0.752941176470588 0.752941176470588 1"/>
-        </material>
-      </visual>
-      <geometry_group name="fine_collision">
-        <origin rpy="0 0 0" xyz="0 0 0"/>
-        <geometry>
-          <mesh filename="package://herb_description/meshes/finger0_1.STL"/>
+          <mesh filename="package://herb_description/meshes/bh280/finger0_1.dae"/>
+        </geometry>
+        <material name="">
+          <color rgba="0.752941176470588 0.752941176470588 0.752941176470588 1"/>
+        </material>
+      </visual>
+      <geometry_group name="fine_collision">
+        <origin rpy="0 0 0" xyz="0 0 0"/>
+        <geometry>
+          <mesh filename="package://herb_description/meshes/bh280/finger0_1.STL"/>
         </geometry>
       </geometry_group>
@@ -94,5 +94,5 @@
       <collision>
         <geometry>
-          <mesh filename="package://herb_description/meshes/finger0_1_collision.STL"/>
+          <mesh filename="package://herb_description/meshes/bh280/finger0_1_collision.STL"/>
         </geometry>
       </collision>
@@ -109,5 +109,5 @@
         <origin xyz="0 0 0" rpy="0 0 0"/>
         <geometry>
-          <mesh filename="package://herb_description/meshes/finger0_2.dae"/>
+          <mesh filename="package://herb_description/meshes/bh280/finger0_2.dae"/>
         </geometry>
         <material name="">
@@ -118,5 +118,5 @@
         <origin rpy="0 0 0" xyz="0 0 0"/>
         <geometry>
-          <mesh filename="package://herb_description/meshes/finger0_2.STL"/>
+          <mesh filename="package://herb_description/meshes/bh280/finger0_2.STL"/>
         </geometry>
       </geometry_group>
@@ -131,5 +131,5 @@
       <collision>
         <geometry>
-          <mesh filename="package://herb_description/meshes/finger0_2_collision.STL"/>
+          <mesh filename="package://herb_description/meshes/bh280/finger0_2_collision.STL"/>
         </geometry>
       </collision>
@@ -147,14 +147,14 @@
         <origin xyz="0 0 0" rpy="0 0 0"/>
         <geometry>
-          <mesh filename="package://herb_description/meshes/finger1_0.dae"/>
-        </geometry>
-        <material name="">
-          <color rgba="0.752941176470588 0.752941176470588 0.752941176470588 1"/>
-        </material>
-      </visual>
-      <geometry_group name="fine_collision">
-        <origin rpy="0 0 0" xyz="0 0 0"/>
-        <geometry>
-          <mesh filename="package://herb_description/meshes/finger1_0.STL"/>
+          <mesh filename="package://herb_description/meshes/bh280/finger1_0.dae"/>
+        </geometry>
+        <material name="">
+          <color rgba="0.752941176470588 0.752941176470588 0.752941176470588 1"/>
+        </material>
+      </visual>
+      <geometry_group name="fine_collision">
+        <origin rpy="0 0 0" xyz="0 0 0"/>
+        <geometry>
+          <mesh filename="package://herb_description/meshes/bh280/finger1_0.STL"/>
         </geometry>
       </geometry_group>
@@ -169,5 +169,5 @@
       <collision>
         <geometry>
-          <mesh filename="package://herb_description/meshes/finger1_0_collision.STL"/>
+          <mesh filename="package://herb_description/meshes/bh280/finger1_0_collision.STL"/>
         </geometry>
       </collision>
@@ -185,14 +185,14 @@
         <origin xyz="0 0 0" rpy="0 0 0"/>
         <geometry>
-          <mesh filename="package://herb_description/meshes/finger1_1.dae"/>
-        </geometry>
-        <material name="">
-          <color rgba="0.752941176470588 0.752941176470588 0.752941176470588 1"/>
-        </material>
-      </visual>
-      <geometry_group name="fine_collision">
-        <origin rpy="0 0 0" xyz="0 0 0"/>
-        <geometry>
-          <mesh filename="package://herb_description/meshes/finger1_1.STL"/>
+          <mesh filename="package://herb_description/meshes/bh280/finger1_1.dae"/>
+        </geometry>
+        <material name="">
+          <color rgba="0.752941176470588 0.752941176470588 0.752941176470588 1"/>
+        </material>
+      </visual>
+      <geometry_group name="fine_collision">
+        <origin rpy="0 0 0" xyz="0 0 0"/>
+        <geometry>
+          <mesh filename="package://herb_description/meshes/bh280/finger1_1.STL"/>
         </geometry>
       </geometry_group>
@@ -207,5 +207,5 @@
       <collision>
         <geometry>
-          <mesh filename="package://herb_description/meshes/finger1_1_collision.STL"/>
+          <mesh filename="package://herb_description/meshes/bh280/finger1_1_collision.STL"/>
         </geometry>
       </collision>
@@ -222,5 +222,5 @@
         <origin xyz="0 0 0" rpy="0 0 0"/>
         <geometry>
-          <mesh filename="package://herb_description/meshes/finger1_2.dae"/>
+          <mesh filename="package://herb_description/meshes/bh280/finger1_2.dae"/>
         </geometry>
         <material name="">
@@ -231,5 +231,5 @@
         <origin rpy="0 0 0" xyz="0 0 0"/>
         <geometry>
-          <mesh filename="package://herb_description/meshes/finger1_2.STL"/>
+          <mesh filename="package://herb_description/meshes/bh280/finger1_2.STL"/>
         </geometry>
       </geometry_group>
@@ -244,5 +244,5 @@
       <collision>
         <geometry>
-          <mesh filename="package://herb_description/meshes/finger1_2_collision.STL"/>
+          <mesh filename="package://herb_description/meshes/bh280/finger1_2_collision.STL"/>
         </geometry>
       </collision>
@@ -260,14 +260,14 @@
         <origin xyz="0 0 0" rpy="0 0 0"/>
         <geometry>
-          <mesh filename="package://herb_description/meshes/finger2_1.dae"/>
-        </geometry>
-        <material name="">
-          <color rgba="0.752941176470588 0.752941176470588 0.752941176470588 1"/>
-        </material>
-      </visual>
-      <geometry_group name="fine_collision">
-        <origin rpy="0 0 0" xyz="0 0 0"/>
-        <geometry>
-          <mesh filename="package://herb_description/meshes/finger2_1.STL"/>
+          <mesh filename="package://herb_description/meshes/bh280/finger2_1.dae"/>
+        </geometry>
+        <material name="">
+          <color rgba="0.752941176470588 0.752941176470588 0.752941176470588 1"/>
+        </material>
+      </visual>
+      <geometry_group name="fine_collision">
+        <origin rpy="0 0 0" xyz="0 0 0"/>
+        <geometry>
+          <mesh filename="package://herb_description/meshes/bh280/finger2_1.STL"/>
         </geometry>
       </geometry_group>
@@ -282,5 +282,5 @@
       <collision>
         <geometry>
-          <mesh filename="package://herb_description/meshes/finger2_1_collision.STL"/>
+          <mesh filename="package://herb_description/meshes/bh280/finger2_1_collision.STL"/>
         </geometry>
       </collision>
@@ -297,5 +297,5 @@
         <origin xyz="0 0 0" rpy="0 0 0"/>
         <geometry>
-          <mesh filename="package://herb_description/meshes/finger2_2.dae"/>
+          <mesh filename="package://herb_description/meshes/bh280/finger2_2.dae"/>
         </geometry>
         <material name="">
@@ -306,5 +306,5 @@
         <origin rpy="0 0 0" xyz="0 0 0"/>
         <geometry>
-          <mesh filename="package://herb_description/meshes/finger2_2.STL"/>
+          <mesh filename="package://herb_description/meshes/bh280/finger2_2.STL"/>
         </geometry>
       </geometry_group>
@@ -319,5 +319,5 @@
       <collision>
         <geometry>
-          <mesh filename="package://herb_description/meshes/finger2_2_collision.STL"/>
+          <mesh filename="package://herb_description/meshes/bh280/finger2_2_collision.STL"/>
         </geometry>
       </collision>

File: robots/herb.urdf.xacro (robot description, xacro)
@@ -3,4 +3,5 @@
   <xacro:include filename="herb_base.urdf.xacro"/>
   <xacro:include filename="bh280.urdf.xacro"/>
+  <xacro:include filename="bh282.urdf.xacro"/>
   <xacro:include filename="wam.urdf.xacro"/>
   <xacro:include filename="fixed_transforms.urdf.xacro"/>
@@ -8,8 +9,11 @@
        optionally the BH-280 BarrettHand end-effector. -->
   <xacro:macro name="herb_manipulator"
-               params="prefix:=${prefix} bh280:=false">
+               params="prefix:=${prefix} bh280:=false bh282:=false">
     <xacro:wam prefix="${prefix}"/>
     <xacro:if value="${bh280}">
       <xacro:bh280 prefix="${prefix}"/>
+    </xacro:if>
+    <xacro:if value="${bh282}">
+      <xacro:bh282 prefix="${prefix}"/>
     </xacro:if>
     <link name="${prefix}/force_torque">
@@ -37,10 +41,20 @@
       </joint>
     </xacro:if>
+    <xacro:if value="${bh282}">
+      <joint name="${prefix}/hand_mount" type="fixed">
+        <!-- The force/torque sensor is 12 mm thick. -->
+        <origin xyz="0 0 0.012" rpy="0 0 ${pi/2}"/>
+        <parent link="${prefix}/force_torque"/>
+        <child link="${prefix}/hand_base"/>
+      </joint>
+    </xacro:if>
   </xacro:macro>
   <!-- hand arguments should all default to false to make argument passing sane -->
   <xacro:arg name="left_bh280" default="false"/>
   <xacro:arg name="right_bh280" default="false"/>
-  <xacro:herb_manipulator prefix="/left" bh280="$(arg left_bh280)"/>
-  <xacro:herb_manipulator prefix="/right" bh280="$(arg right_bh280)"/>
+  <xacro:arg name="left_bh282" default="false"/>
+  <xacro:arg name="right_bh282" default="false"/>
+  <xacro:herb_manipulator prefix="/left" bh280="$(arg left_bh280)" bh282="$(arg left_bh282)"/>
+  <xacro:herb_manipulator prefix="/right" bh280="$(arg right_bh280)" bh282="$(arg right_bh282)"/>
   <xacro:herb_base prefix=""/>
   <joint name="/left/wam_mount" type="fixed">

File: robots/herb_base.urdf.xacro (robot description, xacro)
@@ -13,5 +13,5 @@
         <origin xyz="0 0 0" rpy="0 0 0"/>
         <geometry>
-          <mesh filename="package://herb_description/meshes/herb_base.dae"/>
+          <mesh filename="package://herb_description/meshes/base/herb_base.dae"/>
         </geometry>
         <material name="">
@@ -21,5 +21,5 @@
       <collision>
         <geometry>
-          <mesh filename="package://herb_description/meshes/herb_base_collision.STL"/>
+          <mesh filename="package://herb_description/meshes/base/herb_base_collision.STL"/>
         </geometry>
       </collision>
@@ -37,5 +37,5 @@
         <origin xyz="0 0 0" rpy="0 0 0"/>
         <geometry>
-          <mesh filename="package://herb_description/meshes/segway_wheel_left.dae"/>
+          <mesh filename="package://herb_description/meshes/segway/segway_wheel_left.dae"/>
         </geometry>
         <material name="">
@@ -45,5 +45,5 @@
       <collision>
         <geometry>
-          <mesh filename="package://herb_description/meshes/segway_wheel_left_collision.STL"/>
+          <mesh filename="package://herb_description/meshes/segway/segway_wheel_left_collision.STL"/>
         </geometry>
       </collision>
@@ -67,5 +67,5 @@
         <origin xyz="0 0 0" rpy="0 0 0"/>
         <geometry>
-          <mesh filename="package://herb_description/meshes/segway_wheel_right.dae"/>
+          <mesh filename="package://herb_description/meshes/segway/segway_wheel_right.dae"/>
         </geometry>
         <material name="">
@@ -75,5 +75,5 @@
       <collision>
         <geometry>
-          <mesh filename="package://herb_description/meshes/segway_wheel_right_collision.STL"/>
+          <mesh filename="package://herb_description/meshes/segway/segway_wheel_right_collision.STL"/>
         </geometry>
       </collision>
@@ -97,5 +97,5 @@
         <origin xyz="0 0 0" rpy="0 0 0"/>
         <geometry>
-          <mesh filename="package://herb_description/meshes/head_wam1.dae"/>
+          <mesh filename="package://herb_description/meshes/head/head_wam1.dae"/>
         </geometry>
         <material name="">
@@ -105,5 +105,5 @@
       <collision>
         <geometry>
-        <mesh filename="package://herb_description/meshes/head_wam1_collision.STL"/></geometry>
+        <mesh filename="package://herb_description/meshes/head/head_wam1_collision.STL"/></geometry>
       </collision>
     </link>
@@ -126,5 +126,5 @@
         <origin xyz="0 0 0" rpy="0 0 0"/>
         <geometry>
-          <mesh filename="package://herb_description/meshes/head_wam2.dae"/>
+          <mesh filename="package://herb_description/meshes/head/head_wam2.dae"/>
         </geometry>
         <material name="">
@@ -134,5 +134,5 @@
       <collision>
         <geometry>
-        <mesh filename="package://herb_description/meshes/head_wam2_collision.STL"/></geometry>
+        <mesh filename="package://herb_description/meshes/head/head_wam2_collision.STL"/></geometry>
       </collision>
     </link>

File: robots/wam.urdf.xacro (robot description, xacro)
@@ -5,5 +5,5 @@
         <origin xyz="0 0 0" rpy="0 0 0"/>
         <geometry>
-          <mesh filename="package://herb_description/meshes/wam_base.dae"/>
+          <mesh filename="package://herb_description/meshes/wam/wam_base.dae"/>
         </geometry>
         <material name="">
@@ -20,5 +20,5 @@
       </inertial>
       <collision>
-        <geometry><mesh filename="package://herb_description/meshes/wam_base_collision.STL"/>
+        <geometry><mesh filename="package://herb_description/meshes/wam/wam_base_collision.STL"/>
         </geometry>
       </collision>
@@ -28,5 +28,5 @@
         <origin xyz="0 0 0" rpy="0 0 0"/>
         <geometry>
-          <mesh filename="package://herb_description/meshes/wam1.dae"/>
+          <mesh filename="package://herb_description/meshes/wam/wam1.dae"/>
         </geometry>
         <material name="">
@@ -44,5 +44,5 @@
       <collision>
         <geometry>
-          <mesh filename="package://herb_description/meshes/wam1_collision.STL"/>
+          <mesh filename="package://herb_description/meshes/wam/wam1_collision.STL"/>
         </geometry>
       </collision>
@@ -60,5 +60,5 @@
         <origin xyz="0 0 0" rpy="0 0 0"/>
         <geometry>
-          <mesh filename="package://herb_description/meshes/wam2.dae"/>
+          <mesh filename="package://herb_description/meshes/wam/wam2.dae"/>
         </geometry>
         <material name="">
@@ -76,5 +76,5 @@
       <collision>
         <geometry>
-          <mesh filename="package://herb_description/meshes/wam2_collision.STL"/>
+          <mesh filename="package://herb_description/meshes/wam/wam2_collision.STL"/>
         </geometry>
       </collision>
@@ -91,5 +91,5 @@
         <origin xyz="0 0 0" rpy="0 0 0"/>
         <geometry>
-          <mesh filename="package://herb_description/meshes/wam3.dae"/>
+          <mesh filename="package://herb_description/meshes/wam/wam3.dae"/>
         </geometry>
         <material name="">
@@ -107,5 +107,5 @@
       <collision>
         <geometry>
-          <mesh filename="package://herb_description/meshes/wam3_collision.STL"/>
+          <mesh filename="package://herb_description/meshes/wam/wam3_collision.STL"/>
         </geometry>
       </collision>
@@ -122,5 +122,5 @@
         <origin xyz="0 0 0" rpy="0 0 0"/>
         <geometry>
-          <mesh filename="package://herb_description/meshes/wam4.dae"/>
+          <mesh filename="package://herb_description/meshes/wam/wam4.dae"/>
         </geometry>
         <material name="">
@@ -138,5 +138,5 @@
       <collision>
         <geometry>
-          <mesh filename="package://herb_description/meshes/wam4_collision.STL"/>
+          <mesh filename="package://herb_description/meshes/wam/wam4_collision.STL"/>
         </geometry>
       </collision>
@@ -153,5 +153,5 @@
         <origin xyz="0 0 0" rpy="0 0 0"/>
         <geometry>
-          <mesh filename="package://herb_description/meshes/wam5.dae"/>
+          <mesh filename="package://herb_description/meshes/wam/wam5.dae"/>
         </geometry>
         <material name="">
@@ -169,5 +169,5 @@
       <collision>
         <geometry>
-          <mesh filename="package://herb_description/meshes/wam5_collision.STL"/>
+          <mesh filename="package://herb_description/meshes/wam/wam5_collision.STL"/>
         </geometry>
       </collision>
@@ -184,5 +184,5 @@
         <origin xyz="0 0 0" rpy="0 0 0"/>
         <geometry>
-          <mesh filename="package://herb_description/meshes/wam6.dae"/>
+          <mesh filename="package://herb_description/meshes/wam/wam6.dae"/>
         </geometry>
         <material name="">
@@ -200,5 +200,5 @@
       <collision>
         <geometry>
-          <mesh filename="package://herb_description/meshes/wam6_collision.STL"/>
+          <mesh filename="package://herb_description/meshes/wam/wam6_collision.STL"/>
         </geometry>
       </collision>
@@ -215,5 +215,5 @@
         <origin xyz="0 0 0" rpy="0 0 0"/>
         <geometry>
-          <mesh filename="package://herb_description/meshes/wam7.dae"/>
+          <mesh filename="package://herb_description/meshes/wam/wam7.dae"/>
         </geometry>
         <material name="">
@@ -231,5 +231,5 @@
       <collision>
         <geometry>
-          <mesh filename="package://herb_description/meshes/wam7_collision.STL"/>
+          <mesh filename="package://herb_description/meshes/wam/wam7_collision.STL"/>
         </geometry>
       </collision>
