Commit message: zero-fixes and add inertia for new bh282 base

File: robots/bh280.urdf.xacro (robot description, xacro)
@@ -22,6 +22,6 @@
         <inertia
             ixx="0.0006986" ixy="2.7577e-007" ixz="-7.8138e-007"
-            iyx="0.0000000" iyy="0.00050354"  iyz="-6.44e-005"
-            izx="0.0000000" izy="0.00000000"  izz="0.00062253"/>
+            iyy="0.00050354"  iyz="-6.44e-005"
+            izz="0.00062253"/>
       </inertial>
       <collision>
@@ -52,6 +52,6 @@
         <inertia
             ixx="2.0672e-005" ixy="2.6024e-007" ixz="6.3481e-006"
-            iyx="0.000000000" iyy="7.4105e-005" iyz="1.7118e-008"
-            izx="0.000000000" izy="0.000000000" izz="6.8207e-005"/>
+            iyy="7.4105e-005" iyz="1.7118e-008"
+            izz="6.8207e-005"/>
       </inertial>
       <collision>
@@ -89,6 +89,6 @@
         <inertia
             ixx="4.8162e-006" ixy="5.7981e-007" ixz="-7.2483e-007"
-            iyx="0.000000000" iyy="4.3317e-005" iyz="-2.6653e-009"
-            izx="0.000000000" izy="0.000000000" izz="4.4441e-005"/>
+            iyy="4.3317e-005" iyz="-2.6653e-009"
+            izz="4.4441e-005"/>
       </inertial>
       <collision>
@@ -126,6 +126,6 @@
         <inertia
             ixx="3.1199e-006" ixy="4.5115e-007" ixz="-2.9813e-007"
-            iyx="0.000000000" iyy="1.6948e-005" iyz="-1.8635e-008"
-            izx="0.000000000" izy="0.000000000" izz="1.5809e-005"/>
+            iyy="1.6948e-005" iyz="-1.8635e-008"
+            izz="1.5809e-005"/>
       </inertial>
       <collision>
@@ -164,6 +164,6 @@
         <inertia
             ixx="2.0672e-005" ixy="2.6024e-007" ixz="6.3481e-006"
-            iyx="0.000000000" iyy="7.4105e-005" iyz="1.7118e-008"
-            izx="0.000000000" izy="0.000000000" izz="6.8207e-005"/>
+            iyy="7.4105e-005" iyz="1.7118e-008"
+            izz="6.8207e-005"/>
       </inertial>
       <collision>
@@ -202,6 +202,6 @@
         <inertia
             ixx="4.8162e-006" ixy="5.7981e-007" ixz="-7.2483e-007"
-            iyx="0.000000000" iyy="4.3317e-005" iyz="-2.6653e-009"
-            izx="0.000000000" izy="0.000000000" izz="4.4441e-005"/>
+            iyy="4.3317e-005" iyz="-2.6653e-009"
+            izz="4.4441e-005"/>
       </inertial>
       <collision>
@@ -239,6 +239,6 @@
         <inertia
             ixx="3.1199e-006" ixy="4.5115e-007" ixz="-2.9813e-007"
-            iyx="0.000000000" iyy="1.6948e-005" iyz="-1.8635e-008"
-            izx="0.000000000" izy="0.000000000" izz="1.5809e-005"/>
+            iyy="1.6948e-005" iyz="-1.8635e-008"
+            izz="1.5809e-005"/>
       </inertial>
       <collision>
@@ -277,6 +277,6 @@
         <inertia
             ixx="4.8162e-006" ixy="5.7981e-007" ixz="-7.2483e-007"
-            iyx="0.000000000" iyy="4.3317e-005" iyz="-2.6653e-009"
-            izx="0.000000000" izy="0.000000000" izz="4.4441e-005"/>
+            iyy="4.3317e-005" iyz="-2.6653e-009"
+            izz="4.4441e-005"/>
       </inertial>
       <collision>
@@ -314,6 +314,6 @@
         <inertia
             ixx="3.1199e-006" ixy="4.5115e-007" ixz="-2.9813e-007"
-            iyx="0.000000000" iyy="1.6948e-005" iyz="-1.8635e-008"
-            izx="0.000000000" izy="0.000000000" izz="1.5809e-005"/>
+            iyy="1.6948e-005" iyz="-1.8635e-008"
+            izz="1.5809e-005"/>
       </inertial>
       <collision>

File: robots/bh282.urdf.xacro (robot description, xacro)
@@ -19,10 +19,10 @@
       </geometry_group>
       <inertial>
-        <origin xyz="5.0019e-005 -0.0044561 0.037268"/>
-        <mass value="0.60858"/>
-        <inertia
-            ixx="0.0006986" ixy="2.7577e-007" ixz="-7.8138e-007"
-            iyx="0.0000000" iyy="0.00050354"  iyz="-6.44e-005"
-            izx="0.0000000" izy="0.00000000"  izz="0.00062253"/>
+        <origin xyz="-2.506e-005 0.034479 -0.0072785"/>
+        <mass value="0.36699"/>
+        <inertia
+            ixx="0.00040811" ixy= "0.00000082" ixz="0.00000048"
+            iyy= "0.00040009" iyz="-0.00002736"
+            izz="0.00022400"/>
       </inertial>
       <collision>
@@ -49,10 +49,11 @@
       </geometry_group>
       <inertial>
-        <origin xyz="5.0019e-005 -0.0044561 0.037268"/>
-        <mass value="0.60858"/>
-        <inertia
-            ixx="0.0006986" ixy="2.7577e-007" ixz="-7.8138e-007"
-            iyx="0.0000000" iyy="0.00050354"  iyz="-6.44e-005"
-            izx="0.0000000" izy="0.00000000"  izz="0.00062253"/>
+        <!-- TODO -->
+        <origin xyz="0 0 0"/>
+        <mass value="0.01"/>
+        <inertia
+            ixx="0.0000001" ixy="0.0000001" ixz="0.0000001"
+            iyy="0.0000001" iyz="0.0000001"
+            izz="0.0000001"/>
       </inertial>
       <collision>
@@ -74,5 +75,5 @@
         </geometry>
         <material name="">
-          <color rgba="0.752941176470588 0.752941176470588 0.752941176470588 1"/>
+          <color rgba="0.75 0.75 0.75 1"/>
         </material>
       </visual>
@@ -88,6 +89,6 @@
         <inertia
             ixx="2.0672e-005" ixy="2.6024e-007" ixz="6.3481e-006"
-            iyx="0.000000000" iyy="7.4105e-005" iyz="1.7118e-008"
-            izx="0.000000000" izy="0.000000000" izz="6.8207e-005"/>
+            iyy="7.4105e-005" iyz="1.7118e-008"
+            izz="6.8207e-005"/>
       </inertial>
       <collision>
@@ -125,6 +126,6 @@
         <inertia
             ixx="4.8162e-006" ixy="5.7981e-007" ixz="-7.2483e-007"
-            iyx="0.000000000" iyy="4.3317e-005" iyz="-2.6653e-009"
-            izx="0.000000000" izy="0.000000000" izz="4.4441e-005"/>
+            iyy="4.3317e-005" iyz="-2.6653e-009"
+            izz="4.4441e-005"/>
       </inertial>
       <collision>
@@ -162,6 +163,6 @@
         <inertia
             ixx="3.1199e-006" ixy="4.5115e-007" ixz="-2.9813e-007"
-            iyx="0.000000000" iyy="1.6948e-005" iyz="-1.8635e-008"
-            izx="0.000000000" izy="0.000000000" izz="1.5809e-005"/>
+            iyy="1.6948e-005" iyz="-1.8635e-008"
+            izz="1.5809e-005"/>
       </inertial>
       <collision>
@@ -200,6 +201,6 @@
         <inertia
             ixx="2.0672e-005" ixy="2.6024e-007" ixz="6.3481e-006"
-            iyx="0.000000000" iyy="7.4105e-005" iyz="1.7118e-008"
-            izx="0.000000000" izy="0.000000000" izz="6.8207e-005"/>
+            iyy="7.4105e-005" iyz="1.7118e-008"
+            izz="6.8207e-005"/>
       </inertial>
       <collision>
@@ -238,6 +239,6 @@
         <inertia
             ixx="4.8162e-006" ixy="5.7981e-007" ixz="-7.2483e-007"
-            iyx="0.000000000" iyy="4.3317e-005" iyz="-2.6653e-009"
-            izx="0.000000000" izy="0.000000000" izz="4.4441e-005"/>
+            iyy="4.3317e-005" iyz="-2.6653e-009"
+            izz="4.4441e-005"/>
       </inertial>
       <collision>
@@ -275,6 +276,6 @@
         <inertia
             ixx="3.1199e-006" ixy="4.5115e-007" ixz="-2.9813e-007"
-            iyx="0.000000000" iyy="1.6948e-005" iyz="-1.8635e-008"
-            izx="0.000000000" izy="0.000000000" izz="1.5809e-005"/>
+            iyy="1.6948e-005" iyz="-1.8635e-008"
+            izz="1.5809e-005"/>
       </inertial>
       <collision>
@@ -313,6 +314,6 @@
         <inertia
             ixx="4.8162e-006" ixy="5.7981e-007" ixz="-7.2483e-007"
-            iyx="0.000000000" iyy="4.3317e-005" iyz="-2.6653e-009"
-            izx="0.000000000" izy="0.000000000" izz="4.4441e-005"/>
+            iyy="4.3317e-005" iyz="-2.6653e-009"
+            izz="4.4441e-005"/>
       </inertial>
       <collision>
@@ -351,6 +352,6 @@
         <inertia
             ixx="3.1199e-006" ixy="4.5115e-007" ixz="-2.9813e-007"
-            iyx="0.000000000" iyy="1.6948e-005" iyz="-1.8635e-008"
-            izx="0.000000000" izy="0.000000000" izz="1.5809e-005"/>
+            iyy="1.6948e-005" iyz="-1.8635e-008"
+            izz="1.5809e-005"/>
       </inertial>
       <collision>
