Commit message: Added the herb_base export.

File: robots/herb.urdf.xacro (robot description, xacro)
@@ -1,4 +1,5 @@
 <robot xmlns:xacro="http://www.ros.org/wiki/xacro" name="herb">
     <xacro:property name="pi" value="3.14159265359"/>
+    <xacro:include filename="herb_base.urdf.xacro"/>
     <xacro:include filename="bh280.urdf.xacro"/>
     <xacro:include filename="wam.urdf.xacro"/>
@@ -16,16 +17,16 @@
     </xacro:macro>
     <xacro:macro name="herb">
+        <xacro:herb_base prefix=""/>
         <xacro:wam_ft_bh280 prefix="/left"/>
         <xacro:wam_ft_bh280 prefix="/right"/>
-        <link name="herb_base"/>
         <joint name="/left/wam_mount" type="fixed">
-            <origin xyz="0.079  0.191 0.905" rpy="0 ${-pi/2} ${pi}"/>
-            <parent link="herb_base"/>
-            <child link="/left/wam0"/>
+            <origin rpy="0 ${-pi/2} ${pi}"/>
+            <parent link="/herb_base"/>
+            <child link="/left/wam_base"/>
         </joint>
         <joint name="/right/wam_mount" type="fixed">
-            <origin xyz="0.079 -0.191 0.905" rpy="0 ${-pi/2} ${pi}"/>
-            <parent link="herb_base"/>
-            <child link="/right/wam0"/>
+            <origin rpy="0 ${-pi/2} ${pi}"/>
+            <parent link="/herb_base"/>
+            <child link="/right/wam_base"/>
         </joint>
     </xacro:macro>

Commit message: add explicit force torque sensor link w/ inertia and mass to herb URDF

File: robots/herb.urdf.xacro (robot description, xacro)
@@ -10,8 +10,23 @@
         <xacro:wam prefix="${prefix}"/>
         <xacro:bh280 prefix="${prefix}"/>
+        <link name="${prefix}/force_torque">
+            <inertial>
+		<origin xyz="0.0002 0 0.0054" rpy="0 0 0" />
+		<mass value="0.133278" />
+		<inertia ixx="0.07551" ixy="-0.0001199" ixz="-0.00007002"
+                                       iyy= "0.07508"   iyz="-0.0000537"
+                                                        izz= "0.1462" />
+	   </inertial>
+        </link>
+        <joint name="${prefix}/force_torque_mount" type="fixed">
+            <!-- difference between URDF wam7 frame and Barrett's wam7 frame is 0.06m -->
+            <origin xyz="0 0 0.06" rpy="0 0 0"/>
+            <parent link="${prefix}/wam7"/>
+            <child link="${prefix}/force_torque"/>
+        </joint>
         <joint name="${prefix}/hand_mount" type="fixed">
             <!-- The force/torque sensor is 12 mm thick. -->
-            <origin xyz="0 0 0.072" rpy="0 0 ${pi/2}"/>
-            <parent link="${prefix}/wam7"/>
+            <origin xyz="0 0 0.012" rpy="0 0 ${pi/2}"/>
+            <parent link="${prefix}/force_torque"/>
             <child link="${prefix}/hand_base"/>
         </joint>

Commit message: Fixed the force/torque inertia tensor.

File: robots/herb.urdf.xacro (robot description, xacro)
@@ -12,10 +12,10 @@
         <link name="${prefix}/force_torque">
             <inertial>
-		<origin xyz="0.0002 0 0.0054" rpy="0 0 0" />
-		<mass value="0.133278" />
-		<inertia ixx="0.07551" ixy="-0.0001199" ixz="-0.00007002"
-                                       iyy= "0.07508"   iyz="-0.0000537"
-                                                        izz= "0.1462" />
-	   </inertial>
+                <origin xyz="0.0002 0 0.0054" rpy="0 0 0"/>
+                <mass value="0.133278"/>
+                <inertia ixx="0.00007551" ixy="-0.0000001199" ixz="-0.0000000700"
+                                          iyy= "0.0000750800" iyz="-0.0000000537"
+                                                              izz= "0.0001462000"/>
+            </inertial>
         </link>
         <joint name="${prefix}/force_torque_mount" type="fixed">

Commit message: set transform for arms on herb3 model

File: robots/herb.urdf.xacro (robot description, xacro)
@@ -59,10 +59,10 @@
   <xacro:herb_base prefix=""/>
   <joint name="/left/wam_mount" type="fixed">
-    <origin xyz="-0.266700 0.332276 0.694588" rpy="0 ${-pi/2} ${pi}"/>
+    <origin xyz="-0.355924 0.005376 -0.357421" rpy="0 -1.57075 -1.57075"/>
     <parent link="herb_frame"/>
     <child link="/left/wam_base"/>
   </joint>
   <joint name="/right/wam_mount" type="fixed">
-    <origin xyz="-0.266700 -0.049121 0.694588" rpy="0 ${-pi/2} ${pi}"/>
+    <origin xyz="0.050805 0.005376 -0.357421" rpy="0 -1.57075 -1.57075"/>
     <parent link="herb_frame"/>
     <child link="/right/wam_base"/>
