Commit message: Added the SRDF file to the Makefile.

File: robots/herb.srdf.xacro (robot description, xacro)
@@ -1,6 +1,6 @@
 <robot xmlns:xacro="http://www.ros.org/wiki/xacro" name="herb">
-    <xacro:macro name="wam_bhd280_manipulator" params="prefix">
+    <xacro:macro name="wam_bh280_manipulator" params="prefix">
         <group name="${prefix}_wam">
-            <chain base_link="/${prefix}/wam_base" tip_link="/${prefix}/wam7">
+            <chain base_link="/${prefix}/wam_base" tip_link="/${prefix}/wam7"/>
         </group>
         <group name="${prefix}_hand">
@@ -16,5 +16,5 @@
         </group>
         <end_effector name="left_hand" group="left_hand"
-                      parent_link="/${prefix}/wam7" parent_group="${prefix}_arm">
+                      parent_link="/${prefix}/wam7" parent_group="${prefix}_arm"/>
         <!-- Disable collisions between the fingers. -->
         <disable_collisions link1="/${prefix}/finger0_0" link2="/${prefix}/finger1_0"/>
@@ -116,5 +116,5 @@
         </group>
         <end_effector name="head_wam" group="head"
-                      parent_link="/herb_base" parent_group="/head/wam2">
+                      parent_link="/herb_base" parent_group="/head/wam2"/>
     </xacro:macro>
     <xacro:wam_bh280_manipulator prefix="left"/>

Commit message: Removed rosrun reference.

File: robots/herb.srdf.xacro (robot description, xacro)
@@ -5,5 +5,5 @@
         </group>
         <group name="${prefix}_hand">
-            <link name="/${prefix}/base_link"/>
+            <link name="/${prefix}/hand_base"/>
             <link name="/${prefix}/finger0_0"/>
             <link name="/${prefix}/finger0_1"/>
@@ -15,5 +15,5 @@
             <link name="/${prefix}/finger2_2"/>
         </group>
-        <end_effector name="left_hand" group="left_hand"
+        <end_effector name="${prefix}_hand" group="${prefix}_hand"
                       parent_link="/${prefix}/wam7" parent_group="${prefix}_arm"/>
         <!-- Disable collisions between the fingers. -->
@@ -47,11 +47,11 @@
         <disable_collisions link1="/${prefix}/finger2_1" link2="/${prefix}/finger2_2"/>
         <!-- Disable collisions between the fingers and the palm. -->
-        <disable_collisions link1="/${prefix}/wam7" link2="/${prefix}/finger1_0"/>
-        <disable_collisions link1="/${prefix}/wam7" link2="/${prefix}/finger0_1"/>
-        <disable_collisions link1="/${prefix}/wam7" link2="/${prefix}/finger0_2"/>
-        <disable_collisions link1="/${prefix}/wam7" link2="/${prefix}/finger1_1"/>
-        <disable_collisions link1="/${prefix}/wam7" link2="/${prefix}/finger1_2"/>
-        <disable_collisions link1="/${prefix}/wam7" link2="/${prefix}/finger2_1"/>
-        <disable_collisions link1="/${prefix}/wam7" link2="/${prefix}/finger2_2"/>
+        <disable_collisions link1="/${prefix}/hand_base" link2="/${prefix}/finger1_0"/>
+        <disable_collisions link1="/${prefix}/hand_base" link2="/${prefix}/finger0_1"/>
+        <disable_collisions link1="/${prefix}/hand_base" link2="/${prefix}/finger0_2"/>
+        <disable_collisions link1="/${prefix}/hand_base" link2="/${prefix}/finger1_1"/>
+        <disable_collisions link1="/${prefix}/hand_base" link2="/${prefix}/finger1_2"/>
+        <disable_collisions link1="/${prefix}/hand_base" link2="/${prefix}/finger2_1"/>
+        <disable_collisions link1="/${prefix}/hand_base" link2="/${prefix}/finger2_2"/>
         <!-- Sphere representation for CHOMP -->
         <link_sphere_approximation link="/${prefix}/wam0">

Commit message: Added missing link from the head manipulator group.

File: robots/herb.srdf.xacro (robot description, xacro)
@@ -106,4 +106,5 @@
     <xacro:macro name="pantilt" params="name">
         <group name="${name}">
+            <link name="/herb_base"/>
             <link name="/${name}/wam1"/>
             <link name="/${name}/wam2"/>

Commit message: Grabbed the latest SRDF file.

File: robots/herb.srdf.xacro (robot description, xacro)
@@ -1,5 +1,5 @@
 <robot xmlns:xacro="http://www.ros.org/wiki/xacro" name="herb">
     <xacro:macro name="wam_bh280_manipulator" params="prefix">
-        <group name="${prefix}_wam">
+        <group name="${prefix}">
             <chain base_link="/${prefix}/wam_base" tip_link="/${prefix}/wam7"/>
         </group>
@@ -16,5 +16,5 @@
         </group>
         <end_effector name="${prefix}_hand" group="${prefix}_hand"
-                      parent_link="/${prefix}/wam7" parent_group="${prefix}_arm"/>
+                      parent_link="/${prefix}/wam7" parent_group="${prefix}"/>
         <!-- Disable collisions between the fingers. -->
         <disable_collisions link1="/${prefix}/finger0_0" link2="/${prefix}/finger1_0"/>
@@ -55,5 +55,5 @@
         <disable_collisions link1="/${prefix}/hand_base" link2="/${prefix}/finger2_2"/>
         <!-- Sphere representation for CHOMP -->
-        <link_sphere_approximation link="/${prefix}/wam0">
+        <link_sphere_approximation link="/${prefix}/wam_base">
             <sphere center="0.0 0.0 0.0" radius="0.15"/>
         </link_sphere_approximation>
@@ -106,4 +106,5 @@
     <xacro:macro name="pantilt" params="name">
         <group name="${name}">
+            <link name="/herb_base"/>
             <link name="/${name}/wam1"/>
             <link name="/${name}/wam2"/>
@@ -115,6 +116,10 @@
             </link_sphere_approximation>
         </group>
-        <end_effector name="head_wam" group="head"
-                      parent_link="/herb_base" parent_group="/head/wam2"/>
+        <!-- Dummy group to make the head look like an end-effector; e.g. to
+             run inverse kinematics. HERB doesn't actually have a gripper on
+             his head (maybe on HERB3?). -->
+        <group name="${name}_hand"/>
+        <end_effector name="head" group="${name}_hand"
+                      parent_link="/${name}/wam2" parent_group="${name}"/>
     </xacro:macro>
     <xacro:wam_bh280_manipulator prefix="left"/>
@@ -125,3 +130,195 @@
     <disable_collisions link1="/left/wam_base" link2="/right/wam_base"/>
     <disable_collisions link1="/left/wam1" link2="/right/wam1"/>
+    <disable_collisions link1="/herb_base" link2="/head/wam2" />
+    <!-- Automatically-generated by the MoveIt setup assistant. -->
+    <!--
+    <disable_collisions link1="/head/wam1" link2="/head/wam2" reason="Adjacent" />
+    <disable_collisions link1="/head/wam1" link2="/herb_base" reason="Adjacent" />
+    <disable_collisions link1="/head/wam1" link2="/left/wam1" reason="Never" />
+    <disable_collisions link1="/head/wam1" link2="/left/wam2" reason="Never" />
+    <disable_collisions link1="/head/wam1" link2="/left/wam_base" reason="Never" />
+    <disable_collisions link1="/head/wam1" link2="/right/wam1" reason="Never" />
+    <disable_collisions link1="/head/wam1" link2="/right/wam2" reason="Never" />
+    <disable_collisions link1="/head/wam1" link2="/right/wam_base" reason="Never" />
+    <disable_collisions link1="/head/wam1" link2="/segway_wheel_left" reason="Never" />
+    <disable_collisions link1="/head/wam1" link2="/segway_wheel_right" reason="Never" />
+    <disable_collisions link1="/head/wam2" link2="/herb_base" reason="Always" />
+    <disable_collisions link1="/head/wam2" link2="/left/wam1" reason="Never" />
+    <disable_collisions link1="/head/wam2" link2="/left/wam2" reason="Never" />
+    <disable_collisions link1="/head/wam2" link2="/left/wam_base" reason="Never" />
+    <disable_collisions link1="/head/wam2" link2="/right/wam1" reason="Never" />
+    <disable_collisions link1="/head/wam2" link2="/right/wam2" reason="Never" />
+    <disable_collisions link1="/head/wam2" link2="/right/wam_base" reason="Never" />
+    <disable_collisions link1="/head/wam2" link2="/segway_wheel_left" reason="Never" />
+    <disable_collisions link1="/head/wam2" link2="/segway_wheel_right" reason="Never" />
+    <disable_collisions link1="/herb_base" link2="/left/wam1" reason="Default" />
+    <disable_collisions link1="/herb_base" link2="/left/wam2" reason="Never" />
+    <disable_collisions link1="/herb_base" link2="/left/wam_base" reason="Adjacent" />
+    <disable_collisions link1="/herb_base" link2="/right/wam1" reason="Default" />
+    <disable_collisions link1="/herb_base" link2="/right/wam2" reason="Never" />
+    <disable_collisions link1="/herb_base" link2="/right/wam_base" reason="Adjacent" />
+    <disable_collisions link1="/herb_base" link2="/segway_wheel_left" reason="Adjacent" />
+    <disable_collisions link1="/herb_base" link2="/segway_wheel_right" reason="Adjacent" />
+    <disable_collisions link1="/left/finger0_0" link2="/left/finger0_1" reason="Adjacent" />
+    <disable_collisions link1="/left/finger0_0" link2="/left/finger0_2" reason="Never" />
+    <disable_collisions link1="/left/finger0_0" link2="/left/finger1_0" reason="Never" />
+    <disable_collisions link1="/left/finger0_0" link2="/left/finger1_1" reason="Never" />
+    <disable_collisions link1="/left/finger0_0" link2="/left/hand_base" reason="Adjacent" />
+    <disable_collisions link1="/left/finger0_0" link2="/left/wam4" reason="Never" />
+    <disable_collisions link1="/left/finger0_0" link2="/left/wam5" reason="Never" />
+    <disable_collisions link1="/left/finger0_0" link2="/left/wam6" reason="Never" />
+    <disable_collisions link1="/left/finger0_0" link2="/left/wam7" reason="Never" />
+    <disable_collisions link1="/left/finger0_1" link2="/left/finger0_2" reason="Adjacent" />
+    <disable_collisions link1="/left/finger0_1" link2="/left/finger1_0" reason="Never" />
+    <disable_collisions link1="/left/finger0_1" link2="/left/finger1_1" reason="Never" />
+    <disable_collisions link1="/left/finger0_1" link2="/left/hand_base" reason="Default" />
+    <disable_collisions link1="/left/finger0_1" link2="/left/wam4" reason="Never" />
+    <disable_collisions link1="/left/finger0_1" link2="/left/wam5" reason="Never" />
+    <disable_collisions link1="/left/finger0_1" link2="/left/wam6" reason="Never" />
+    <disable_collisions link1="/left/finger0_1" link2="/left/wam7" reason="Never" />
+    <disable_collisions link1="/left/finger0_2" link2="/left/wam4" reason="Never" />
+    <disable_collisions link1="/left/finger0_2" link2="/left/wam5" reason="Never" />
+    <disable_collisions link1="/left/finger0_2" link2="/left/wam6" reason="Never" />
+    <disable_collisions link1="/left/finger0_2" link2="/left/wam7" reason="Never" />
+    <disable_collisions link1="/left/finger1_0" link2="/left/finger1_1" reason="Adjacent" />
+    <disable_collisions link1="/left/finger1_0" link2="/left/finger1_2" reason="Never" />
+    <disable_collisions link1="/left/finger1_0" link2="/left/finger2_2" reason="Never" />
+    <disable_collisions link1="/left/finger1_0" link2="/left/hand_base" reason="Adjacent" />
+    <disable_collisions link1="/left/finger1_0" link2="/left/wam4" reason="Never" />
+    <disable_collisions link1="/left/finger1_0" link2="/left/wam5" reason="Never" />
+    <disable_collisions link1="/left/finger1_0" link2="/left/wam6" reason="Never" />
+    <disable_collisions link1="/left/finger1_0" link2="/left/wam7" reason="Never" />
+    <disable_collisions link1="/left/finger1_1" link2="/left/finger1_2" reason="Adjacent" />
+    <disable_collisions link1="/left/finger1_1" link2="/left/hand_base" reason="Default" />
+    <disable_collisions link1="/left/finger1_1" link2="/left/wam4" reason="Never" />
+    <disable_collisions link1="/left/finger1_1" link2="/left/wam5" reason="Never" />
+    <disable_collisions link1="/left/finger1_1" link2="/left/wam6" reason="Never" />
+    <disable_collisions link1="/left/finger1_1" link2="/left/wam7" reason="Never" />
+    <disable_collisions link1="/left/finger1_2" link2="/left/wam4" reason="Never" />
+    <disable_collisions link1="/left/finger1_2" link2="/left/wam5" reason="Never" />
+    <disable_collisions link1="/left/finger1_2" link2="/left/wam6" reason="Never" />
+    <disable_collisions link1="/left/finger1_2" link2="/left/wam7" reason="Never" />
+    <disable_collisions link1="/left/finger2_1" link2="/left/finger2_2" reason="Adjacent" />
+    <disable_collisions link1="/left/finger2_1" link2="/left/hand_base" reason="Adjacent" />
+    <disable_collisions link1="/left/finger2_1" link2="/left/wam4" reason="Never" />
+    <disable_collisions link1="/left/finger2_1" link2="/left/wam5" reason="Never" />
+    <disable_collisions link1="/left/finger2_1" link2="/left/wam6" reason="Never" />
+    <disable_collisions link1="/left/finger2_1" link2="/left/wam7" reason="Never" />
+    <disable_collisions link1="/left/finger2_2" link2="/left/wam4" reason="Never" />
+    <disable_collisions link1="/left/finger2_2" link2="/left/wam5" reason="Never" />
+    <disable_collisions link1="/left/finger2_2" link2="/left/wam6" reason="Never" />
+    <disable_collisions link1="/left/finger2_2" link2="/left/wam7" reason="Never" />
+    <disable_collisions link1="/left/hand_base" link2="/left/wam4" reason="Never" />
+    <disable_collisions link1="/left/hand_base" link2="/left/wam5" reason="Never" />
+    <disable_collisions link1="/left/hand_base" link2="/left/wam6" reason="Never" />
+    <disable_collisions link1="/left/hand_base" link2="/left/wam7" reason="Adjacent" />
+    <disable_collisions link1="/left/wam1" link2="/left/wam2" reason="Adjacent" />
+    <disable_collisions link1="/left/wam1" link2="/left/wam3" reason="Default" />
+    <disable_collisions link1="/left/wam1" link2="/left/wam4" reason="Never" />
+    <disable_collisions link1="/left/wam1" link2="/left/wam5" reason="Never" />
+    <disable_collisions link1="/left/wam1" link2="/left/wam_base" reason="Adjacent" />
+    <disable_collisions link1="/left/wam1" link2="/right/wam2" reason="Never" />
+    <disable_collisions link1="/left/wam1" link2="/right/wam_base" reason="Never" />
+    <disable_collisions link1="/left/wam1" link2="/segway_wheel_left" reason="Never" />
+    <disable_collisions link1="/left/wam1" link2="/segway_wheel_right" reason="Never" />
+    <disable_collisions link1="/left/wam2" link2="/left/wam3" reason="Adjacent" />
+    <disable_collisions link1="/left/wam2" link2="/left/wam4" reason="Never" />
+    <disable_collisions link1="/left/wam2" link2="/left/wam5" reason="Never" />
+    <disable_collisions link1="/left/wam2" link2="/left/wam6" reason="Never" />
+    <disable_collisions link1="/left/wam2" link2="/left/wam7" reason="Never" />
+    <disable_collisions link1="/left/wam2" link2="/left/wam_base" reason="Never" />
+    <disable_collisions link1="/left/wam2" link2="/right/wam1" reason="Never" />
+    <disable_collisions link1="/left/wam2" link2="/right/wam2" reason="Never" />
+    <disable_collisions link1="/left/wam2" link2="/right/wam_base" reason="Never" />
+    <disable_collisions link1="/left/wam2" link2="/segway_wheel_left" reason="Never" />
+    <disable_collisions link1="/left/wam2" link2="/segway_wheel_right" reason="Never" />
+    <disable_collisions link1="/left/wam3" link2="/left/wam4" reason="Adjacent" />
+    <disable_collisions link1="/left/wam3" link2="/left/wam_base" reason="Never" />
+    <disable_collisions link1="/left/wam4" link2="/left/wam5" reason="Adjacent" />
+    <disable_collisions link1="/left/wam4" link2="/left/wam6" reason="Default" />
+    <disable_collisions link1="/left/wam5" link2="/left/wam6" reason="Adjacent" />
+    <disable_collisions link1="/left/wam6" link2="/left/wam7" reason="Adjacent" />
+    <disable_collisions link1="/left/wam_base" link2="/right/wam1" reason="Never" />
+    <disable_collisions link1="/left/wam_base" link2="/right/wam2" reason="Never" />
+    <disable_collisions link1="/left/wam_base" link2="/right/wam_base" reason="Never" />
+    <disable_collisions link1="/left/wam_base" link2="/segway_wheel_left" reason="Never" />
+    <disable_collisions link1="/left/wam_base" link2="/segway_wheel_right" reason="Never" />
+    <disable_collisions link1="/right/finger0_0" link2="/right/finger0_1" reason="Adjacent" />
+    <disable_collisions link1="/right/finger0_0" link2="/right/finger0_2" reason="Never" />
+    <disable_collisions link1="/right/finger0_0" link2="/right/finger1_0" reason="Never" />
+    <disable_collisions link1="/right/finger0_0" link2="/right/finger1_1" reason="Never" />
+    <disable_collisions link1="/right/finger0_0" link2="/right/hand_base" reason="Adjacent" />
+    <disable_collisions link1="/right/finger0_0" link2="/right/wam4" reason="Never" />
+    <disable_collisions link1="/right/finger0_0" link2="/right/wam5" reason="Never" />
+    <disable_collisions link1="/right/finger0_0" link2="/right/wam6" reason="Never" />
+    <disable_collisions link1="/right/finger0_0" link2="/right/wam7" reason="Never" />
+    <disable_collisions link1="/right/finger0_1" link2="/right/finger0_2" reason="Adjacent" />
+    <disable_collisions link1="/right/finger0_1" link2="/right/finger1_0" reason="Never" />
+    <disable_collisions link1="/right/finger0_1" link2="/right/finger1_1" reason="Never" />
+    <disable_collisions link1="/right/finger0_1" link2="/right/hand_base" reason="Default" />
+    <disable_collisions link1="/right/finger0_1" link2="/right/wam4" reason="Never" />
+    <disable_collisions link1="/right/finger0_1" link2="/right/wam5" reason="Never" />
+    <disable_collisions link1="/right/finger0_1" link2="/right/wam6" reason="Never" />
+    <disable_collisions link1="/right/finger0_1" link2="/right/wam7" reason="Never" />
+    <disable_collisions link1="/right/finger0_2" link2="/right/wam4" reason="Never" />
+    <disable_collisions link1="/right/finger0_2" link2="/right/wam5" reason="Never" />
+    <disable_collisions link1="/right/finger0_2" link2="/right/wam6" reason="Never" />
+    <disable_collisions link1="/right/finger0_2" link2="/right/wam7" reason="Never" />
+    <disable_collisions link1="/right/finger1_0" link2="/right/finger1_1" reason="Adjacent" />
+    <disable_collisions link1="/right/finger1_0" link2="/right/finger1_2" reason="Never" />
+    <disable_collisions link1="/right/finger1_0" link2="/right/finger2_2" reason="Never" />
+    <disable_collisions link1="/right/finger1_0" link2="/right/hand_base" reason="Adjacent" />
+    <disable_collisions link1="/right/finger1_0" link2="/right/wam4" reason="Never" />
+    <disable_collisions link1="/right/finger1_0" link2="/right/wam5" reason="Never" />
+    <disable_collisions link1="/right/finger1_0" link2="/right/wam6" reason="Never" />
+    <disable_collisions link1="/right/finger1_0" link2="/right/wam7" reason="Never" />
+    <disable_collisions link1="/right/finger1_1" link2="/right/finger1_2" reason="Adjacent" />
+    <disable_collisions link1="/right/finger1_1" link2="/right/hand_base" reason="Default" />
+    <disable_collisions link1="/right/finger1_1" link2="/right/wam4" reason="Never" />
+    <disable_collisions link1="/right/finger1_1" link2="/right/wam5" reason="Never" />
+    <disable_collisions link1="/right/finger1_1" link2="/right/wam6" reason="Never" />
+    <disable_collisions link1="/right/finger1_1" link2="/right/wam7" reason="Never" />
+    <disable_collisions link1="/right/finger1_2" link2="/right/wam4" reason="Never" />
+    <disable_collisions link1="/right/finger1_2" link2="/right/wam5" reason="Never" />
+    <disable_collisions link1="/right/finger1_2" link2="/right/wam6" reason="Never" />
+    <disable_collisions link1="/right/finger1_2" link2="/right/wam7" reason="Never" />
+    <disable_collisions link1="/right/finger2_1" link2="/right/finger2_2" reason="Adjacent" />
+    <disable_collisions link1="/right/finger2_1" link2="/right/hand_base" reason="Adjacent" />
+    <disable_collisions link1="/right/finger2_1" link2="/right/wam4" reason="Never" />
+    <disable_collisions link1="/right/finger2_1" link2="/right/wam5" reason="Never" />
+    <disable_collisions link1="/right/finger2_1" link2="/right/wam6" reason="Never" />
+    <disable_collisions link1="/right/finger2_1" link2="/right/wam7" reason="Never" />
+    <disable_collisions link1="/right/finger2_2" link2="/right/wam4" reason="Never" />
+    <disable_collisions link1="/right/finger2_2" link2="/right/wam5" reason="Never" />
+    <disable_collisions link1="/right/finger2_2" link2="/right/wam6" reason="Never" />
+    <disable_collisions link1="/right/finger2_2" link2="/right/wam7" reason="Never" />
+    <disable_collisions link1="/right/hand_base" link2="/right/wam4" reason="Never" />
+    <disable_collisions link1="/right/hand_base" link2="/right/wam5" reason="Never" />
+    <disable_collisions link1="/right/hand_base" link2="/right/wam6" reason="Never" />
+    <disable_collisions link1="/right/hand_base" link2="/right/wam7" reason="Adjacent" />
+    <disable_collisions link1="/right/wam1" link2="/right/wam2" reason="Adjacent" />
+    <disable_collisions link1="/right/wam1" link2="/right/wam3" reason="Default" />
+    <disable_collisions link1="/right/wam1" link2="/right/wam4" reason="Never" />
+    <disable_collisions link1="/right/wam1" link2="/right/wam5" reason="Never" />
+    <disable_collisions link1="/right/wam1" link2="/right/wam_base" reason="Adjacent" />
+    <disable_collisions link1="/right/wam1" link2="/segway_wheel_left" reason="Never" />
+    <disable_collisions link1="/right/wam1" link2="/segway_wheel_right" reason="Never" />
+    <disable_collisions link1="/right/wam2" link2="/right/wam3" reason="Adjacent" />
+    <disable_collisions link1="/right/wam2" link2="/right/wam4" reason="Never" />
+    <disable_collisions link1="/right/wam2" link2="/right/wam5" reason="Never" />
+    <disable_collisions link1="/right/wam2" link2="/right/wam6" reason="Never" />
+    <disable_collisions link1="/right/wam2" link2="/right/wam7" reason="Never" />
+    <disable_collisions link1="/right/wam2" link2="/right/wam_base" reason="Never" />
+    <disable_collisions link1="/right/wam2" link2="/segway_wheel_left" reason="Never" />
+    <disable_collisions link1="/right/wam2" link2="/segway_wheel_right" reason="Never" />
+    <disable_collisions link1="/right/wam3" link2="/right/wam4" reason="Adjacent" />
+    <disable_collisions link1="/right/wam3" link2="/right/wam_base" reason="Never" />
+    <disable_collisions link1="/right/wam4" link2="/right/wam5" reason="Adjacent" />
+    <disable_collisions link1="/right/wam4" link2="/right/wam6" reason="Default" />
+    <disable_collisions link1="/right/wam5" link2="/right/wam6" reason="Adjacent" />
+    <disable_collisions link1="/right/wam6" link2="/right/wam7" reason="Adjacent" />
+    <disable_collisions link1="/right/wam_base" link2="/segway_wheel_left" reason="Never" />
+    <disable_collisions link1="/right/wam_base" link2="/segway_wheel_right" reason="Never" />
+    <disable_collisions link1="/segway_wheel_left" link2="/segway_wheel_right" reason="Never" />
+    -->
 </robot>
