Commit message: optionally build multiple herb models
models without either hand and in the future potentially different hand combinations

File: robots/herb.urdf.xacro (robot description, xacro)
@@ -1,51 +1,56 @@
 <robot xmlns:xacro="http://www.ros.org/wiki/xacro" name="herb">
-    <xacro:property name="pi" value="3.14159265359"/>
-    <xacro:include filename="herb_base.urdf.xacro"/>
-    <xacro:include filename="bh280.urdf.xacro"/>
-    <xacro:include filename="wam.urdf.xacro"/>
-    <xacro:include filename="fixed_transforms.urdf.xacro"/>
-    <!-- 7 DOF Barrett WAM equipped with the Barrett force/torque sensor and
-         the BH-280 BarrettHand end-effector. -->
-    <xacro:macro name="wam_ft_bh280" params="prefix">
-        <xacro:wam prefix="${prefix}"/>
-        <xacro:bh280 prefix="${prefix}"/>
-        <link name="${prefix}/force_torque">
-            <inertial>
-                <origin xyz="0.0002 0 0.0054" rpy="0 0 0"/>
-                <mass value="0.133278"/>
-                <inertia ixx="0.00007551" ixy="-0.0000001199" ixz="-0.0000000700"
-                                          iyy= "0.0000750800" iyz="-0.0000000537"
-                                                              izz= "0.0001462000"/>
-            </inertial>
-        </link>
-        <joint name="${prefix}/force_torque_mount" type="fixed">
-            <!-- difference between URDF wam7 frame and Barrett's wam7 frame is 0.06m -->
-            <origin xyz="0 0 0.06" rpy="0 0 0"/>
-            <parent link="${prefix}/wam7"/>
-            <child link="${prefix}/force_torque"/>
-        </joint>
-        <joint name="${prefix}/hand_mount" type="fixed">
-            <!-- The force/torque sensor is 12 mm thick. -->
-            <origin xyz="0 0 0.012" rpy="0 0 ${pi/2}"/>
-            <parent link="${prefix}/force_torque"/>
-            <child link="${prefix}/hand_base"/>
-        </joint>
-    </xacro:macro>
-    <xacro:macro name="herb">
-        <xacro:wam_ft_bh280 prefix="/left"/>
-        <xacro:wam_ft_bh280 prefix="/right"/>
-        <xacro:herb_base prefix=""/>
-        <joint name="/left/wam_mount" type="fixed">
-            <origin xyz="-0.266700 0.332276 0.694588" rpy="0 ${-pi/2} ${pi}"/>
-            <parent link="/herb_base"/>
-            <child link="/left/wam_base"/>
-        </joint>
-        <joint name="/right/wam_mount" type="fixed">
-            <origin xyz="-0.266700 -0.049121 0.694588" rpy="0 ${-pi/2} ${pi}"/>
-            <parent link="/herb_base"/>
-            <child link="/right/wam_base"/>
-        </joint>
-        <xacro:fixed_transforms/>
-    </xacro:macro>
-    <xacro:herb/>
+  <xacro:property name="pi" value="3.14159265359"/>
+  <xacro:include filename="herb_base.urdf.xacro"/>
+  <xacro:include filename="bh280.urdf.xacro"/>
+  <xacro:include filename="wam.urdf.xacro"/>
+  <xacro:include filename="fixed_transforms.urdf.xacro"/>
+  <!-- 7 DOF Barrett WAM equipped with the Barrett force/torque sensor and
+       optionally the BH-280 BarrettHand end-effector. -->
+  <xacro:macro name="herb_manipulator"
+               params="prefix:=${prefix} bh280:=false">
+    <xacro:wam prefix="${prefix}"/>
+    <xacro:if value="${bh280}">
+      <xacro:bh280 prefix="${prefix}"/>
+    </xacro:if>
+    <link name="${prefix}/force_torque">
+      <inertial>
+        <origin xyz="0.0002 0 0.0054" rpy="0 0 0"/>
+        <mass value="0.133278"/>
+        <inertia ixx="0.00007551" ixy="-0.0000001199" ixz="-0.0000000700"
+                 iyy= "0.0000750800" iyz="-0.0000000537"
+                 izz= "0.0001462000"/>
+      </inertial>
+    </link>
+    <joint name="${prefix}/force_torque_mount" type="fixed">
+      <!-- difference between URDF wam7 frame and Barrett's wam7 frame is 0.06m -->
+      <origin xyz="0 0 0.06" rpy="0 0 0"/>
+      <parent link="${prefix}/wam7"/>
+      <child link="${prefix}/force_torque"/>
+    </joint>
+    <!-- TODO: where should force/torque thickness go if no hand? -->
+    <xacro:if value="${bh280}">
+      <joint name="${prefix}/hand_mount" type="fixed">
+        <!-- The force/torque sensor is 12 mm thick. -->
+        <origin xyz="0 0 0.012" rpy="0 0 ${pi/2}"/>
+        <parent link="${prefix}/force_torque"/>
+        <child link="${prefix}/hand_base"/>
+      </joint>
+    </xacro:if>
+  </xacro:macro>
+  <xacro:arg name="left_bh280" default="false"/>
+  <xacro:arg name="right_bh280" default="false"/>
+  <xacro:herb_manipulator prefix="/left" bh280="$(arg left_bh280)"/>
+  <xacro:herb_manipulator prefix="/right" bh280="$(arg right_bh280)"/>
+  <xacro:herb_base prefix=""/>
+  <joint name="/left/wam_mount" type="fixed">
+    <origin xyz="-0.266700 0.332276 0.694588" rpy="0 ${-pi/2} ${pi}"/>
+    <parent link="/herb_base"/>
+    <child link="/left/wam_base"/>
+  </joint>
+  <joint name="/right/wam_mount" type="fixed">
+    <origin xyz="-0.266700 -0.049121 0.694588" rpy="0 ${-pi/2} ${pi}"/>
+    <parent link="/herb_base"/>
+    <child link="/right/wam_base"/>
+  </joint>
+  <xacro:fixed_transforms/>
 </robot>

Commit message: add dummy endeffector when no hand present

File: robots/herb.srdf.xacro (robot description, xacro)
@@ -40,4 +40,9 @@
       <sphere center="0 0 0" radius="0"/>
     </link_sphere_approximation>
+  </xacro:macro>
+  <xacro:macro name="empty_endeffector" params="prefix:=${prefix}">
+    <group name="${prefix}_hand"/>
+    <end_effector name="${prefix}_hand" group="${prefix}_hand"
+                  parent_link="/${prefix}/wam7" parent_group="${prefix}"/>
   </xacro:macro>
   <xacro:macro name="barretthand_endeffector" params="prefix:=${prefix}">
@@ -144,7 +149,13 @@
     <xacro:barretthand_endeffector prefix="left"/>
   </xacro:if>
+  <xacro:unless value="$(arg left_hand)">
+    <xacro:empty_endeffector prefix="left"/>
+  </xacro:unless>
   <xacro:if value="$(arg right_hand)">
     <xacro:barretthand_endeffector prefix="right"/>
   </xacro:if>
+  <xacro:unless value="$(arg right_hand)">
+    <xacro:empty_endeffector prefix="right"/>
+  </xacro:unless>
   <xacro:pantilt name="head"/>
   <passive_joint name="/segway_wheel_left"/>

Commit message: fix leading bytes in STLs exported from solidworks

File: robots/herb.srdf.xacro (robot description, xacro)
@@ -134,23 +134,23 @@
     </link_sphere_approximation>
   </xacro:macro>
-  <xacro:macro name="pantilt" params="name">
-    <group name="${name}">
-      <link name="/herb_base"/>
-      <link name="/${name}/wam1"/>
-      <link name="/${name}/wam2"/>
-      <link_sphere_approximation link="/${name}/wam1">
-        <sphere center="0 0 0" radius="0.20"/>
-      </link_sphere_approximation>
-      <link_sphere_approximation link="/${name}/wam2">
-        <sphere center="0 0 0" radius="0"/>
-      </link_sphere_approximation>
-    </group>
-    <!-- Dummy group to make the head look like an end-effector; e.g. to
-         run inverse kinematics. HERB doesn't actually have a gripper on
-         his head (maybe on HERB3?). -->
-    <group name="${name}_hand"/>
-    <end_effector name="head" group="${name}_hand"
-                  parent_link="/${name}/wam2" parent_group="${name}"/>
-  </xacro:macro>
+  <!-- <xacro:macro name="pantilt" params="name"> -->
+  <!--   <group name="${name}"> -->
+  <!--     <link name="/herb_base"/> -->
+  <!--     <link name="/${name}/wam1"/> -->
+  <!--     <link name="/${name}/wam2"/> -->
+  <!--     <link_sphere_approximation link="/${name}/wam1"> -->
+  <!--       <sphere center="0 0 0" radius="0.20"/> -->
+  <!--     </link_sphere_approximation> -->
+  <!--     <link_sphere_approximation link="/${name}/wam2"> -->
+  <!--       <sphere center="0 0 0" radius="0"/> -->
+  <!--     </link_sphere_approximation> -->
+  <!--   </group> -->
+  <!--   <!-\- Dummy group to make the head look like an end-effector; e.g. to -->
+  <!--        run inverse kinematics. HERB doesn't actually have a gripper on -->
+  <!--        his head (maybe on HERB3?). -\-> -->
+  <!--   <group name="${name}_hand"/> -->
+  <!--   <end_effector name="head" group="${name}_hand" -->
+  <!--                 parent_link="/${name}/wam2" parent_group="${name}"/> -->
+  <!-- </xacro:macro> -->
   <!-- hand arguments should all default to false to make argument passing sane -->
   <!-- NOTE: if we use kinematically distinct hands from the BarrettHand
@@ -174,9 +174,7 @@
     <xacro:empty_endeffector prefix="right"/>
   </xacro:unless>
-  <xacro:pantilt name="head"/>
-  <passive_joint name="/segway_wheel_left"/>
-  <passive_joint name="/segway_wheel_right"/>
+  <!-- <xacro:pantilt name="head"/> -->
   <disable_collisions link1="/left/wam_base" link2="/right/wam_base"/>
   <disable_collisions link1="/left/wam1" link2="/right/wam1"/>
-  <disable_collisions link1="/herb_base" link2="/head/wam2" />
+  <!-- <disable_collisions link1="/herb_base" link2="/head/wam2" /> -->
 </robot>

Commit message: Weiss gripper (#53)
* added initial weiss gripper implimentation

* integrated weiss gripper

* improved wsg50 integration

* improved wsg50 integration

* corrected TODO statement

* Build all possible HERB models.

File: robots/herb.srdf.xacro (robot description, xacro)
@@ -136,4 +136,25 @@
     </link_sphere_approximation>
   </xacro:macro>
+  <xacro:macro name="wsg50_endeffector" params="prefix:=${prefix}">
+    <group name="${prefix}_hand">
+      <link name="/${prefix}/hand_base"/>
+      <link name="/${prefix}/left_finger_mount"/>
+      <link name="/${prefix}/left_finger"/>
+      <link name="/${prefix}/right_finger_mount"/>
+      <link name="/${prefix}/right_finger"/>
+    </group>
+    <!-- Disable collisions between the fingers. -->
+    <disable_collisions link1="/${prefix}/left_finger_mount" link2="/${prefix}/left_finger"/>
+    <disable_collisions link1="/${prefix}/left_finger_mount" link2="/${prefix}/right_finger_mount"/>
+    <disable_collisions link1="/${prefix}/left_finger_mount" link2="/${prefix}/right_finger"/>
+    <disable_collisions link1="/${prefix}/left_finger" link2="/${prefix}/right_finger_mount"/>
+    <disable_collisions link1="/${prefix}/left_finger" link2="/${prefix}/right_finger"/>
+    <disable_collisions link1="/${prefix}/right_finger_mount" link2="/${prefix}/right_finger"/>
+    <!-- Disable collisions between the fingers and the hand base. -->
+    <disable_collisions link1="/${prefix}/hand_base" link2="/${prefix}/left_finger_mount"/>
+    <disable_collisions link1="/${prefix}/hand_base" link2="/${prefix}/left_finger"/>
+    <disable_collisions link1="/${prefix}/hand_base" link2="/${prefix}/right_finger_mount"/>
+    <disable_collisions link1="/${prefix}/hand_base" link2="/${prefix}/right_finger"/>
+  </xacro:macro>
   <!-- <xacro:macro name="pantilt" params="name"> -->
   <!--   <group name="${name}"> -->
@@ -158,22 +179,36 @@
   <!-- NOTE: if we use kinematically distinct hands from the BarrettHand
        we will need more fine-grained arguments -->
-  <xacro:arg name="left_hand" default="false"/>
-  <xacro:arg name="right_hand" default="false"/>
+  <xacro:property name="left_none" value="true"/>
+  <xacro:property name="right_none" value="true"/>
+  <xacro:arg name="left_barrett" default="false"/>
+  <xacro:arg name="right_barrett" default="false"/>
+  <xacro:arg name="left_wsg50" default="false"/>
+  <xacro:arg name="right_wsg50" default="false"/>
   <xacro:arg name="left_perception" default="false"/>
   <xacro:arg name="right_perception" default="false"/>
   <xacro:wam_manipulator prefix="left"/>
   <xacro:wam_manipulator prefix="right"/>
-  <xacro:if value="$(arg left_hand)">
+  <xacro:if value="$(arg left_barrett)">
     <xacro:barretthand_endeffector prefix="left" perception="$(arg left_perception)"/>
-  </xacro:if>
-  <xacro:unless value="$(arg left_hand)">
+    <xacro:property name="left_none" value="false"/>
+  </xacro:if>
+  <xacro:if value="$(arg left_wsg50)">
+    <xacro:wsg50_endeffector prefix="left"/>
+    <xacro:property name="left_none" value="false"/>
+  </xacro:if>
+  <xacro:if value="${left_none == 'true'}">
     <xacro:empty_endeffector prefix="left"/>
-  </xacro:unless>
-  <xacro:if value="$(arg right_hand)">
+  </xacro:if>
+  <xacro:if value="$(arg right_barrett)">
     <xacro:barretthand_endeffector prefix="right" perception="$(arg right_perception)"/>
-  </xacro:if>
-  <xacro:unless value="$(arg right_hand)">
+    <xacro:property name="right_none" value="false"/>
+  </xacro:if>
+  <xacro:if value="$(arg right_wsg50)">
+    <xacro:wsg50_endeffector prefix="right"/>
+    <xacro:property name="right_none" value="false"/>
+  </xacro:if>
+  <xacro:if value="${right_none == 'true'}">
     <xacro:empty_endeffector prefix="right"/>
-  </xacro:unless>
+  </xacro:if>
   <!-- <xacro:pantilt name="head"/> -->
   <disable_collisions link1="/left/wam_base" link2="/right/wam_base"/>

File: robots/herb.urdf.xacro (robot description, xacro)
@@ -3,4 +3,5 @@
   <xacro:include filename="bh280.urdf.xacro"/>
   <xacro:include filename="bh282.urdf.xacro"/>
+  <xacro:include filename="wsg50.urdf.xacro"/>
   <xacro:include filename="wam.urdf.xacro"/>
   <xacro:include filename="fixed_transforms.urdf.xacro"/>
@@ -8,5 +9,5 @@
        optionally the BH-280 BarrettHand end-effector. -->
   <xacro:macro name="herb_manipulator"
-               params="prefix:=${prefix} bh280:=false bh282:=false">
+               params="prefix:=${prefix} bh280:=false bh282:=false wsg50:=false">
     <xacro:wam prefix="${prefix}"/>
     <xacro:if value="${bh280}">
@@ -15,4 +16,7 @@
     <xacro:if value="${bh282}">
       <xacro:bh282 prefix="${prefix}"/>
+    </xacro:if>
+    <xacro:if value="${wsg50}">
+      <xacro:wsg50 prefix="${prefix}"/>
     </xacro:if>
     <link name="${prefix}/force_torque">
@@ -48,4 +52,12 @@
       </joint>
     </xacro:if>
+  <xacro:if value="${wsg50}">
+      <joint name="${prefix}/hand_mount" type="fixed">
+        <!-- The force/torque sensor is 12 mm thick. -->
+        <origin xyz="0 0 0.012" rpy="0 0 ${pi/2}"/>
+        <parent link="${prefix}/force_torque"/>
+        <child link="${prefix}/hand_base"/>
+      </joint>
+    </xacro:if>
   </xacro:macro>
   <!-- hand arguments should all default to false to make argument passing sane -->
@@ -54,6 +66,8 @@
   <xacro:arg name="left_bh282" default="false"/>
   <xacro:arg name="right_bh282" default="false"/>
-  <xacro:herb_manipulator prefix="/left" bh280="$(arg left_bh280)" bh282="$(arg left_bh282)"/>
-  <xacro:herb_manipulator prefix="/right" bh280="$(arg right_bh280)" bh282="$(arg right_bh282)"/>
+  <xacro:arg name="left_wsg50" default="false"/>
+  <xacro:arg name="right_wsg50" default="false"/>
+  <xacro:herb_manipulator prefix="/left" bh280="$(arg left_bh280)" bh282="$(arg left_bh282)" wsg50="$(arg left_wsg50)"/>
+  <xacro:herb_manipulator prefix="/right" bh280="$(arg right_bh280)" bh282="$(arg right_bh282)" wsg50="$(arg right_wsg50)"/>
   <xacro:herb_base prefix=""/>
   <joint name="/left/wam_mount" type="fixed">
