Commit message: add perception palm to srdf. use collada models

File: robots/bh282.urdf.xacro (robot description, xacro)
@@ -6,14 +6,14 @@
         <origin xyz="-0.112 -0.056 -0.023" rpy="0 0 0"/>
         <geometry>
-          <mesh filename="package://herb_description/meshes/bh282/hand_base.stl"/>
-        </geometry>
-        <material name="">
-          <color rgba="0.752941176470588 0.752941176470588 0.752941176470588 1"/>
-        </material>
-      </visual>
-      <geometry_group name="fine_collision">
-        <origin rpy="0 0 0" xyz="0 0 0"/>
-        <geometry>
-          <mesh filename="package://herb_description/meshes/bh282/hand_base.stl"/>
+          <mesh filename="package://herb_description/meshes/bh282/hand_base.dae"/>
+        </geometry>
+        <material name="">
+          <color rgba="0.75 0.75 0.75 1"/>
+        </material>
+      </visual>
+      <geometry_group name="fine_collision">
+        <origin rpy="0 0 0" xyz="0 0 0"/>
+        <geometry>
+          <mesh filename="package://herb_description/meshes/bh282/hand_base.dae"/>
         </geometry>
       </geometry_group>
@@ -28,22 +28,22 @@
       <collision>
         <geometry>
-          <mesh filename="package://herb_description/meshes/bh282/hand_base.stl"/>
-        </geometry>
-      </collision>
-    </link>
-    <link name="${prefix}/palm">
+          <mesh filename="package://herb_description/meshes/bh282/hand_base.dae"/>
+        </geometry>
+      </collision>
+    </link>
+    <link name="${prefix}/perception_palm">
       <visual>
         <origin xyz="-0.112 -0.056 -0.023" rpy="0 0 0"/>
         <geometry>
-          <mesh filename="package://herb_description/meshes/bh282/perception_palm.stl"/>
-        </geometry>
-        <material name="">
-          <color rgba="0.752941176470588 0.752941176470588 0.752941176470588 1"/>
-        </material>
-      </visual>
-      <geometry_group name="fine_collision">
-        <origin rpy="0 0 0" xyz="0 0 0"/>
-        <geometry>
-          <mesh filename="package://herb_description/meshes/bh282/perception_palm.stl"/>
+          <mesh filename="package://herb_description/meshes/bh282/perception_palm.dae"/>
+        </geometry>
+        <material name="">
+          <color rgba="0.75 0.75 0.75 1"/>
+        </material>
+      </visual>
+      <geometry_group name="fine_collision">
+        <origin rpy="0 0 0" xyz="0 0 0"/>
+        <geometry>
+          <mesh filename="package://herb_description/meshes/bh282/perception_palm.dae"/>
         </geometry>
       </geometry_group>
@@ -58,12 +58,12 @@
       <collision>
         <geometry>
-          <mesh filename="package://herb_description/meshes/bh282/hand_base.stl"/>
-        </geometry>
-      </collision>
-    </link>
-    <joint name="${prefix}/palm_mount" type="fixed">
+          <mesh filename="package://herb_description/meshes/bh282/perception_palm.dae"/>
+        </geometry>
+      </collision>
+    </link>
+    <joint name="${prefix}/perception_palm_mount" type="fixed">
         <origin xyz="0 0 0" rpy="0 0 0"/>
         <parent link="${prefix}/hand_base"/>
-        <child link="${prefix}/palm"/>
+        <child link="${prefix}/perception_palm"/>
     </joint>
     <link name="${prefix}/finger0_0">

File: robots/herb.srdf.xacro (robot description, xacro)
@@ -46,5 +46,5 @@
                   parent_link="/${prefix}/wam7" parent_group="${prefix}"/>
   </xacro:macro>
-  <xacro:macro name="barretthand_endeffector" params="prefix:=${prefix}">
+  <xacro:macro name="barretthand_endeffector" params="prefix:=${prefix} perception:=false">
     <!-- Must be included AFTER wam_manipulator -->
     <group name="${prefix}_hand">
@@ -58,4 +58,7 @@
       <link name="/${prefix}/finger2_1"/>
       <link name="/${prefix}/finger2_2"/>
+      <xacro:if value="${perception}">
+        <link name="/${prefix}/perception_palm"/>
+      </xacro:if>
     </group>
     <end_effector name="${prefix}_hand" group="${prefix}_hand"
@@ -90,5 +93,5 @@
     <disable_collisions link1="/${prefix}/finger1_2" link2="/${prefix}/finger2_2"/>
     <disable_collisions link1="/${prefix}/finger2_1" link2="/${prefix}/finger2_2"/>
-    <!-- Disable collisions between the fingers and the palm. -->
+    <!-- Disable collisions between the fingers and the hand base. -->
     <disable_collisions link1="/${prefix}/hand_base" link2="/${prefix}/finger1_0"/>
     <disable_collisions link1="/${prefix}/hand_base" link2="/${prefix}/finger0_1"/>
@@ -98,4 +101,15 @@
     <disable_collisions link1="/${prefix}/hand_base" link2="/${prefix}/finger2_1"/>
     <disable_collisions link1="/${prefix}/hand_base" link2="/${prefix}/finger2_2"/>
+    <xacro:if value="${perception}">
+      <!-- Disable collisions between the fingers and the perception palm. -->
+      <disable_collisions link1="/${prefix}/hand_base" link2="/${prefix}/perception_palm"/>
+      <disable_collisions link1="/${prefix}/perception_palm" link2="/${prefix}/finger1_0"/>
+      <disable_collisions link1="/${prefix}/perception_palm" link2="/${prefix}/finger0_1"/>
+      <disable_collisions link1="/${prefix}/perception_palm" link2="/${prefix}/finger0_2"/>
+      <disable_collisions link1="/${prefix}/perception_palm" link2="/${prefix}/finger1_1"/>
+      <disable_collisions link1="/${prefix}/perception_palm" link2="/${prefix}/finger1_2"/>
+      <disable_collisions link1="/${prefix}/perception_palm" link2="/${prefix}/finger2_1"/>
+      <disable_collisions link1="/${prefix}/perception_palm" link2="/${prefix}/finger2_2"/>
+    </xacro:if>
     <!-- Disable collisions between palm and WAM end link -->
     <disable_collisions link1="/${prefix}/wam6" link2="/${prefix}/hand_base"/>
@@ -144,8 +158,10 @@
   <xacro:arg name="left_hand" default="false"/>
   <xacro:arg name="right_hand" default="false"/>
+  <xacro:arg name="left_perception" default="false"/>
+  <xacro:arg name="right_perception" default="false"/>
   <xacro:wam_manipulator prefix="left"/>
   <xacro:wam_manipulator prefix="right"/>
   <xacro:if value="$(arg left_hand)">
-    <xacro:barretthand_endeffector prefix="left"/>
+    <xacro:barretthand_endeffector prefix="left" perception="$(arg left_perception)"/>
   </xacro:if>
   <xacro:unless value="$(arg left_hand)">
@@ -153,5 +169,5 @@
   </xacro:unless>
   <xacro:if value="$(arg right_hand)">
-    <xacro:barretthand_endeffector prefix="right"/>
+    <xacro:barretthand_endeffector prefix="right" perception="$(arg right_perception)"/>
   </xacro:if>
   <xacro:unless value="$(arg right_hand)">

Commit message: [UBT 16.04] for xacro builds, add inorder option and remove deps and args arguments (#47)
* for xacro builds, add inorder option and remove deps and args arguments

* fix CMakeLists, remove redundant definitions of pi

File: robots/bh282.urdf.xacro (robot description, xacro)
@@ -1,4 +1,3 @@
 <robot xmlns:xacro="http://www.ros.org/wiki/xacro" name="bh282">
-  <xacro:property name="pi" value="3.14159265359"/>
   <xacro:macro name="bh282" params="prefix">
     <link name="${prefix}/hand_base">

File: robots/herb.urdf.xacro (robot description, xacro)
@@ -1,4 +1,3 @@
 <robot xmlns:xacro="http://www.ros.org/wiki/xacro" name="herb">
-  <xacro:property name="pi" value="3.14159265359"/>
   <xacro:include filename="herb_base.urdf.xacro"/>
   <xacro:include filename="bh280.urdf.xacro"/>

File: robots/wam_bh280_standalone.urdf.xacro (robot description, xacro)
@@ -1,5 +1,4 @@
 <robot xmlns:xacro="http://www.ros.org/wiki/xacro" name="wam">
     <xacro:property name="prefix" value=""/>
-    <xacro:property name="pi" value="3.14159265359"/>
     <xacro:include filename="bh280.urdf.xacro"/>
     <xacro:include filename="wam.urdf.xacro"/>

File: robots/wam_bh282_standalone.urdf.xacro (robot description, xacro)
@@ -1,5 +1,4 @@
 <robot xmlns:xacro="http://www.ros.org/wiki/xacro" name="wam">
     <xacro:property name="prefix" value=""/>
-    <xacro:property name="pi" value="3.14159265359"/>
     <xacro:include filename="bh282.urdf.xacro"/>
     <xacro:include filename="wam.urdf.xacro"/>

Commit message: Correction for collision model of hand (#54)
* set origin for collision model as well

* similar fix for the fingers

File: robots/bh282.urdf.xacro (robot description, xacro)
@@ -26,4 +26,5 @@
       </inertial>
       <collision>
+        <origin xyz="-0.112 -0.056 -0.023"/>
         <geometry>
           <mesh filename="package://herb_description/meshes/bh282/hand_base.dae"/>
@@ -56,4 +57,5 @@
       </inertial>
       <collision>
+        <origin xyz="-0.112 -0.056 -0.023"/>
         <geometry>
           <mesh filename="package://herb_description/meshes/bh282/perception_palm.dae"/>
@@ -91,4 +93,5 @@
       </inertial>
       <collision>
+        <origin xyz="0 0 -0.029" rpy="0 0 0"/>
         <geometry>
           <mesh filename="package://herb_description/meshes/bh280/finger0_0_collision.STL"/>
@@ -203,4 +206,5 @@
       </inertial>
       <collision>
+        <origin xyz="0 0 -0.029" rpy="0 0 0"/>
         <geometry>
           <mesh filename="package://herb_description/meshes/bh280/finger1_0_collision.STL"/>

Commit message: mass checks plus realsense things

File: robots/bh282.urdf.xacro (robot description, xacro)
@@ -19,5 +19,5 @@
       <inertial>
         <origin xyz="5.0019e-005 -0.0044561 0.037268"/>
-        <mass value="0.60858"/>
+        <mass value="0.36699"/>
         <inertia
             ixx="0.0006986" ixy="2.7577e-007" ixz="-7.8138e-007"
@@ -49,5 +49,5 @@
       <inertial>
         <origin xyz="5.0019e-005 -0.0044561 0.037268"/>
-        <mass value="0.60858"/>
+        <mass value="0.05"/>
         <inertia
             ixx="0.0006986" ixy="2.7577e-007" ixz="-7.8138e-007"

File: robots/herb_base.urdf.xacro (robot description, xacro)
@@ -334,5 +334,5 @@
         <origin
             xyz="0 0 0"
-            rpy="0 3.1415926 0" />
+            rpy="1.5707963 3.1415926 0" />
         <geometry>
           <mesh
@@ -353,12 +353,12 @@
       </link>
     <joint
-        name="crl_head_to_realsense"
-        type="fixed">
-      <parent
-          link="crl_head" />
+        name="neck_tilt_to_realsense"
+        type="fixed">
+      <parent
+          link="neck_tilt" />
       <child
           link="camera_link" />
       <origin
-          xyz="0.008 -0.1690163 -0.0765607"
+          xyz="0 -0.150963 -0.1015607"
           rpy="0 1.5707 1.5707" />
     </joint>
