Commit message: Adding artificial base link

File: robots/herb_base.urdf.xacro (robot description, xacro)
@@ -1,4 +1,20 @@
 <robot xmlns:xacro="http://www.ros.org/wiki/xacro" name="herb_base">
   <xacro:macro name="herb_base" params="prefix">
+    <link name="herb_base_link">
+      <inertial>
+        <origin
+            xyz="0 0 0"
+            rpy="0 0 0" />
+        <mass
+            value="0.1" />
+        <inertia
+            ixx="1"
+            ixy="0"
+            ixz="0"
+            iyy="1"
+            iyz="0"
+            izz="1" />
+      </inertial>
+    </link>
     <link
         name="herb_frame">
@@ -42,4 +58,15 @@
       </collision>
     </link>
+    <joint
+        name="root_to_frame"
+        type="fixed">
+      <origin
+          xyz="0 0 1.05"
+          rpy="0 0 -1.57075" />
+      <parent
+          link="herb_base_link" />
+      <child
+          link="herb_frame" />
+    </joint>
     <link
         name="neobotix_base">

Commit message: Changed herb_base_link to base_footprint

File: robots/herb_base.urdf.xacro (robot description, xacro)
@@ -1,5 +1,5 @@
 <robot xmlns:xacro="http://www.ros.org/wiki/xacro" name="herb_base">
   <xacro:macro name="herb_base" params="prefix">
-    <link name="herb_base_link">
+    <link name="base_footprint">
       <inertial>
         <origin
@@ -65,5 +65,5 @@
           rpy="0 0 -1.57075" />
       <parent
-          link="herb_base_link" />
+          link="base_footprint" />
       <child
           link="herb_frame" />

Commit message: Updated stl and urdf to reflect taller herb frame

File: robots/herb_base.urdf.xacro (robot description, xacro)
@@ -25,12 +25,12 @@
             rpy="0 0 0" />
         <mass
-            value="75.88" />
-        <inertia
-            ixx="11.92524"
-            ixy="0.00418"
-            ixz="0.00448"
-            iyy="4.13145"
-            iyz="2.60056"
-            izz="10.77706" />
+            value="106.25" />
+        <inertia
+            ixx="22.3955"
+            ixy="-0.2746"
+            ixz="-0.0999"
+            iyy="5.9126"
+            iyz="5.1995"
+            izz="20.4410" />
       </inertial>
       <visual>
@@ -74,5 +74,5 @@
       <inertial>
         <origin
-            xyz="0 -0.074086 -1.040385"
+            xyz="0 -0.074086 -1.101244"
             rpy="0 0 0" />
         <mass
@@ -114,5 +114,5 @@
         type="fixed">
       <origin
-          xyz="0 -0.074086 -1.040385"
+          xyz="0 -0.074086 -1.101244"
           rpy="0 0 3.141592" />
       <parent
@@ -167,10 +167,10 @@
       <axis
           xyz="0 0 1" />
-      <!--velocity is arbitrary; check against real values-->
+      <!--velocity dimensions assumed to be rad/s-->
       <limit
-          effort="4.0"
+          effort="2.0"
           lower="-1.57075"
           upper="1.57075"
-          velocity="1" />
+          velocity="6.28319" />
       <origin
           xyz="0 0.124900 0.050806"
@@ -226,10 +226,10 @@
       <axis
           xyz="1 0 0" />
-      <!--velocity is arbitrary; check against real values-->
+      <!--velocity dimensions assumed to be rad/s-->
       <limit
-          effort="24.0"
+          effort="12.0"
           lower="-1.57075"
           upper="1.57075"
-          velocity="1" />
+          velocity="4.18879" />
       <origin
           xyz="0 0 -0.0919"

Commit message: added extra link to multisense frame

File: robots/herb_base.urdf.xacro (robot description, xacro)
@@ -234,5 +234,5 @@
       <origin
           xyz="0 0 -0.0919"
-          rpy="0 0 0" />
+          rpy="-0.698132 0 0" />
       <parent
           link="neck_pan" />
@@ -241,5 +241,5 @@
     </joint>
     <link
-        name="multisense/head">
+        name="crl_head">
       <!--check inertias and mass-->
       <inertial>
@@ -287,8 +287,35 @@
           link="neck_tilt" />
       <child
+          link="crl_head" />
+      <origin
+          xyz="-0.003895 -0.0575 -0.236"
+          rpy="-1.57075 0 0" />
+    </joint>
+    <link name="multisense/head">
+      <inertial>
+        <origin
+            xyz="0 0 0"
+            rpy="0 0 0" />
+        <mass
+            value="0.1" />
+        <inertia
+            ixx="1"
+            ixy="0"
+            ixz="0"
+            iyy="1"
+            iyz="0"
+            izz="1" />
+      </inertial>
+    </link>
+    <joint
+        name="crl_head_to_multisenseframe"
+        type="fixed">
+      <parent
+          link="crl_head" />
+      <child
           link="multisense/head" />
       <origin
-          xyz="-0.003895 -0.0575 -0.236"
-          rpy="0 3.14159 1.5707" />
+          xyz="0 0 0"
+          rpy="0 1.5707 1.5707" />
     </joint>
     <link
@@ -336,5 +363,5 @@
         type="fixed">
       <parent
-          link="multisense/head" />
+          link="crl_head" />
       <child
           link="kinect" />

Commit message: changing meshes and urdf

File: robots/herb_base.urdf.xacro (robot description, xacro)
@@ -241,5 +241,5 @@
     </joint>
     <link
-        name="crl_head">
+        name="multisense/head">
       <!--check inertias and mass-->
       <inertial>
@@ -287,35 +287,8 @@
           link="neck_tilt" />
       <child
-          link="crl_head" />
-      <origin
-          xyz="-0.003895 -0.0575 -0.236"
+          link="multisense/head" />
+      <origin
+          xyz="0.11446 0.00 -0.148915"
           rpy="-1.57075 0 0" />
-    </joint>
-    <link name="multisense/head">
-      <inertial>
-        <origin
-            xyz="0 0 0"
-            rpy="0 0 0" />
-        <mass
-            value="0.1" />
-        <inertia
-            ixx="1"
-            ixy="0"
-            ixz="0"
-            iyy="1"
-            iyz="0"
-            izz="1" />
-      </inertial>
-    </link>
-    <joint
-        name="crl_head_to_multisenseframe"
-        type="fixed">
-      <parent
-          link="crl_head" />
-      <child
-          link="multisense/head" />
-      <origin
-          xyz="0 -0.056 -0.086"
-          rpy="0 1.5707 1.5707" />
     </joint>
     <link
@@ -360,12 +333,12 @@
     </link>
     <joint
-        name="crl_head_to_kinect"
-        type="fixed">
-      <parent
-          link="crl_head" />
+        name="tilt_neck_to_kinect"
+        type="fixed">
+      <parent
+          link="neck_tilt" />
       <child
           link="kinect" />
       <origin
-          xyz="-0.003895 -0.170163 0.017938"
+          xyz="0.039918 0.0 0.066119"
           rpy="0 1.57075 0" />
     </joint>

Commit message: test/no_multisense

File: robots/herb_base.urdf.xacro (robot description, xacro)
@@ -292,82 +292,4 @@
           rpy="-1.57075 0 0" />
     </joint>
-    <link name="multisense/head">
-      <inertial>
-        <origin
-            xyz="0 0 0"
-            rpy="0 0 0" />
-        <mass
-            value="0.1" />
-        <inertia
-            ixx="1"
-            ixy="0"
-            ixz="0"
-            iyy="1"
-            iyz="0"
-            izz="1" />
-      </inertial>
-    </link>
-    <joint
-        name="crl_head_to_multisenseframe"
-        type="fixed">
-      <parent
-          link="crl_head" />
-      <child
-          link="multisense/head" />
-      <origin
-          xyz="0 -0.086 -0.056"
-          rpy="0 1.5707 1.5707" />
-    </joint>
-    <link
-        name="head/kinect2_link">
-      <inertial>
-        <origin
-            xyz="0.001778 0.164443 0.209049"
-            rpy="0 0 0" />
-        <mass
-            value="0.63"/>
-        <inertia
-            ixx="0.00272"
-            ixy="0.00036"
-            ixz="-0.00002"
-            iyy="0.00258"
-            iyz="-0.00001"
-            izz="0.00145" />
-      </inertial>
-      <visual>
-        <origin
-            xyz="0 0 0"
-            rpy="0 0 0" />
-        <geometry>
-          <mesh
-              filename="package://herb_description/meshes/head/herb_kinect.STL" />
-        </geometry>
-        <material
-            name="">
-          <color
-              rgba="0 0 0 1" />
-        </material>
-      </visual>
-      <collision>
-        <origin
-            xyz="-0.039543 -0.065 0"
-            rpy="1.57075 1.57075 1.57075" />
-        <geometry>
-          <mesh
-              filename="package://herb_description/meshes/head/herb_kinect_collision.STL" />
-        </geometry>
-      </collision>
-    </link>
-    <joint
-        name="crl_head_to_kinect"
-        type="fixed">
-      <parent
-          link="crl_head" />
-      <child
-          link="head/kinect2_link" />
-      <origin
-          xyz="-0.003895 -0.170163 0.017938"
-          rpy="3.14159 0 0" />
-    </joint>
   </xacro:macro>
 </robot>

Commit message: Adding fake links and joints to correct self-collision

File: robots/herb_base.urdf.xacro (robot description, xacro)
@@ -320,5 +320,5 @@
     </joint>
     <link
-        name="head/kinect2_link">
+        name="kinect2_fake_link">
       <inertial>
         <origin
@@ -365,8 +365,35 @@
           link="crl_head" />
       <child
-          link="head/kinect2_link" />
+          link="kinect2_fake_link" />
       <origin
           xyz="-0.003895 -0.170163 0.017938"
-          rpy="3.14159 0 0" />
+          rpy="0 1.57075 0" />
+    </joint>
+    <link name="head/kinect2_link">
+      <inertial>
+        <origin
+            xyz="0 0 0"
+            rpy="0 0 0" />
+        <mass
+            value="0.001" />
+        <inertia
+            ixx="1"
+            ixy="0"
+            ixz="0"
+            iyy="1"
+            iyz="0"
+            izz="1" />
+      </inertial>
+    </link>
+    <joint
+      name="kinect2_fake_joint"
+      type="fixed">
+      <parent
+        link="kinect2_fake_link"/>
+      <child
+        link="head/kinect2_link" />
+      <origin
+        xyz="0 0 0"
+        rpy="3.14159 -1.57075 0"/>
     </joint>
   </xacro:macro>

Commit message: replace the kinect with realsense, and aligned the position

File: robots/herb_base.urdf.xacro (robot description, xacro)
@@ -320,5 +320,5 @@
     </joint>
     <link
-        name="head/kinect2_link">
+        name="head/realsense_link">
       <inertial>
         <origin
@@ -326,5 +326,5 @@
             rpy="0 0 0" />
         <mass
-            value="0.63"/>
+            value="0.79"/>
         <inertia
             ixx="0.00272"
@@ -337,9 +337,9 @@
       <visual>
         <origin
-            xyz="0 0 0"
-            rpy="0 0 0" />
-        <geometry>
-          <mesh
-              filename="package://herb_description/meshes/head/herb_kinect.STL" />
+            xyz="0 -0.0125 -0.045"
+            rpy="4.7123889 4.7123889 0" />
+        <geometry>
+          <mesh
+              filename="package://herb_description/meshes/head/herb_realsense.STL" scale="0.001 0.001 0.001" />
         </geometry>
         <material
@@ -351,9 +351,9 @@
       <collision>
         <origin
-            xyz="-0.039543 -0.065 0"
-            rpy="1.57075 1.57075 1.57075" />
-        <geometry>
-          <mesh
-              filename="package://herb_description/meshes/head/herb_kinect_collision.STL" />
+            xyz="0 -0.0125 -0.045"
+            rpy="0 0 0" />
+        <geometry>
+          <mesh
+              filename="package://herb_description/meshes/head/herb_realsense_collision.STL" scale="0.001 0.001 0.001" />
         </geometry>
       </collision>
@@ -365,8 +365,8 @@
           link="crl_head" />
       <child
-          link="head/kinect2_link" />
-      <origin
-          xyz="-0.003895 -0.170163 0.017938"
-          rpy="0 1.57075 0" />
+          link="head/realsense_link" />
+      <origin
+          xyz="0 -0.170163 0.017938"
+          rpy="0 1.5707 0" />
     </joint>
   </xacro:macro>

Commit message: fix the realsense linking issue

File: robots/herb_base.urdf.xacro (robot description, xacro)
@@ -319,27 +319,23 @@
           rpy="0 1.5707 1.5707" />
     </joint>
-    <link
-        name="head/realsense_link">
-      <inertial>
-        <origin
-            xyz="0.001778 0.164443 0.209049"
-            rpy="0 0 0" />
-        <mass
+        <xacro:property name="d435_cam_width" value="0.090"/>
+    <xacro:property name="d435_cam_height" value="0.025"/>
+    <xacro:property name="d435_cam_depth" value="0.02505"/>
+    <xacro:property name="M_PI" value="3.1415926535897931" />
+    <xacro:property name="d435_cam_mount_from_center_offset" value="0.0149"/>
+    <xacro:property name="d435_cam_depth_py" value="0.0175"/>
+    <link
+        name="camera_link">
+        <origin xyz="${d435_cam_mount_from_center_offset} ${-d435_cam_depth_py} 0" rpy="0 0 0"/>
+	<mass
             value="0.79"/>
-        <inertia
-            ixx="0.00272"
-            ixy="0.00036"
-            ixz="-0.00002"
-            iyy="0.00258"
-            iyz="-0.00001"
-            izz="0.00145" />
-      </inertial>
-      <visual>
-        <origin
-            xyz="0 -0.0125 -0.045"
-            rpy="4.7123889 4.7123889 0" />
-        <geometry>
-          <mesh
-              filename="package://herb_description/meshes/head/herb_realsense.STL" scale="0.001 0.001 0.001" />
+      <inertia ixx="0.003881243" ixy="0.0" ixz="0.0" iyy="0.000498940" iyz="0.0" izz="0.003879257" />
+	<visual>
+        <origin
+            xyz="0 0 0"
+            rpy="3.1415926 0 1.5707" />
+        <geometry>
+          <mesh
+              filename="package://herb_description/meshes/head/realsense.dae" />
         </geometry>
         <material
@@ -349,24 +345,21 @@
         </material>
       </visual>
-      <collision>
-        <origin
-            xyz="0 -0.0125 -0.045"
-            rpy="0 0 0" />
-        <geometry>
-          <mesh
-              filename="package://herb_description/meshes/head/herb_realsense_collision.STL" scale="0.001 0.001 0.001" />
-        </geometry>
-      </collision>
-    </link>
-    <joint
-        name="crl_head_to_kinect"
+    	<collision>
+        <origin xyz="0 ${-d435_cam_depth_py} 0" rpy="0 0 0"/>
+        <geometry>
+        <box size="${d435_cam_depth} ${d435_cam_width} ${d435_cam_height}"/>
+        </geometry>
+      </collision>
+      </link>
+    <joint
+        name="crl_head_to_realsense"
         type="fixed">
       <parent
           link="crl_head" />
       <child
-          link="head/realsense_link" />
+          link="camera_link" />
       <origin
           xyz="0 -0.170163 -0.0323"
-          rpy="0 1.5707 0" />
+          rpy="0 0 1.5707" />
     </joint>
   </xacro:macro>

Commit message: change the rotation of the realsense

File: robots/herb_base.urdf.xacro (robot description, xacro)
@@ -334,5 +334,5 @@
         <origin
             xyz="0 0 0"
-            rpy="3.1415926 0 1.5707" />
+            rpy="0 0 0" />
         <geometry>
           <mesh
@@ -346,5 +346,5 @@
       </visual>
     	<collision>
-        <origin xyz="0 ${-d435_cam_depth_py} 0" rpy="0 0 0"/>
+        <origin xyz="0 0 0" rpy="0 0 0"/>
         <geometry>
         <box size="${d435_cam_depth} ${d435_cam_width} ${d435_cam_height}"/>

Commit message: replace kinect with realsense

File: robots/herb_base.urdf.xacro (robot description, xacro)
@@ -319,27 +319,23 @@
           rpy="0 1.5707 1.5707" />
     </joint>
-    <link
-        name="head/kinect2_link">
-      <inertial>
-        <origin
-            xyz="0.001778 0.164443 0.209049"
-            rpy="0 0 0" />
-        <mass
-            value="0.63"/>
-        <inertia
-            ixx="0.00272"
-            ixy="0.00036"
-            ixz="-0.00002"
-            iyy="0.00258"
-            iyz="-0.00001"
-            izz="0.00145" />
-      </inertial>
-      <visual>
-        <origin
-            xyz="0 0 0"
-            rpy="0 0 0" />
-        <geometry>
-          <mesh
-              filename="package://herb_description/meshes/head/herb_kinect.STL" />
+    <xacro:property name="d435_cam_width" value="0.090"/>
+    <xacro:property name="d435_cam_height" value="0.025"/>
+    <xacro:property name="d435_cam_depth" value="0.02505"/>
+    <xacro:property name="M_PI" value="3.1415926535897931" />
+    <xacro:property name="d435_cam_mount_from_center_offset" value="0.0149"/>
+    <xacro:property name="d435_cam_depth_py" value="0.0175"/>
+    <link
+        name="camera_link">
+        <origin xyz="${d435_cam_mount_from_center_offset} ${-d435_cam_depth_py} 0" rpy="0 0 0"/>
+  <mass
+            value="0.79"/>
+      <inertia ixx="0.003881243" ixy="0.0" ixz="0.0" iyy="0.000498940" iyz="0.0" izz="0.003879257" />
+  <visual>
+        <origin
+            xyz="0 0 0"
+            rpy="0 3.1415926 0" />
+        <geometry>
+          <mesh
+              filename="package://herb_description/meshes/head/realsense.dae" />
         </geometry>
         <material
@@ -350,23 +346,20 @@
       </visual>
       <collision>
-        <origin
-            xyz="-0.039543 -0.065 0"
-            rpy="1.57075 1.57075 1.57075" />
-        <geometry>
-          <mesh
-              filename="package://herb_description/meshes/head/herb_kinect_collision.STL" />
-        </geometry>
-      </collision>
-    </link>
-    <joint
-        name="crl_head_to_kinect"
+        <origin xyz="0 0 0" rpy="0 0 0"/>
+        <geometry>
+        <box size="${d435_cam_depth} ${d435_cam_width} ${d435_cam_height}"/>
+        </geometry>
+      </collision>
+      </link>
+    <joint
+        name="crl_head_to_realsense"
         type="fixed">
       <parent
           link="crl_head" />
       <child
-          link="head/kinect2_link" />
-      <origin
-          xyz="-0.003895 -0.170163 0.017938"
-          rpy="0 1.57075 0" />
+          link="camera_link" />
+      <origin
+          xyz="0.008 -0.1690163 -0.0765607"
+          rpy="0 1.5707 1.5707" />
     </joint>
   </xacro:macro>

Commit message: remove unnecessary things

File: robots/herb_base.urdf.xacro (robot description, xacro)
@@ -325,39 +325,19 @@
     <xacro:property name="d435_cam_mount_from_center_offset" value="0.0149"/>
     <xacro:property name="d435_cam_depth_py" value="0.0175"/>
-    <link
-        name="camera_link">
-        <origin xyz="${d435_cam_mount_from_center_offset} ${-d435_cam_depth_py} 0" rpy="0 0 0"/>
-  <mass
-            value="0.79"/>
-      <inertia ixx="0.003881243" ixy="0.0" ixz="0.0" iyy="0.000498940" iyz="0.0" izz="0.003879257" />
-  <visual>
-        <origin
-            xyz="0 0 0"
-            rpy="0 3.1415926 0" />
-        <geometry>
-          <mesh
-              filename="package://herb_description/meshes/head/realsense.dae" />
-        </geometry>
-        <material
-            name="">
-          <color
-              rgba="0.25 0.25 0.25 1" />
-        </material>
-      </visual>
-      <collision>
-        <origin xyz="0 0 0" rpy="0 0 0"/>
-        <geometry>
-        <box size="${d435_cam_depth} ${d435_cam_width} ${d435_cam_height}"/>
-        </geometry>
-      </collision>
-      </link>
+    <link name="camera_link">
+      <inertial>
+        <origin
+            xyz="${d435_cam_mount_from_center_offset} ${-d435_cam_depth_py} 0"
+            rpy="0 0 0"/>
+      </inertial>
+    </link>
     <joint
         name="crl_head_to_realsense"
         type="fixed">
-      <parent
+        <parent
           link="crl_head" />
-      <child
+        <child
           link="camera_link" />
-      <origin
+        <origin
           xyz="0.008 -0.1690163 -0.0765607"
           rpy="0 1.5707 1.5707" />

Commit message: add camera_link

File: robots/herb_base.urdf.xacro (robot description, xacro)
@@ -164,13 +164,13 @@
     <joint
         name="frame_to_neck_pan"
-        type="revolute">
+        type="fixed">
       <axis
-          xyz="0 0 -1" />
-      <!--pan (swivel) velocity limit of 360 degrees/s-->
+          xyz="0 0 1" />
+      <!--velocity dimensions assumed to be rad/s-->
       <limit
           effort="2.0"
-          lower="-0.78539"
-          upper="0.78539"
-          velocity="6.28318" />
+          lower="-1.57075"
+          upper="1.57075"
+          velocity="6.28319" />
       <origin
           xyz="0 0.124900 0.050806"
@@ -222,17 +222,17 @@
     </link>
     <joint
-        name="neck_pan_to_neck_tilt"
-        type="revolute">
+        name="pan_neck_to_tilt_neck"
+        type="fixed">
       <axis
-          xyz="-1 0 0" />
-      <!--tilt velocity limit of 240 degrees/s-->
+          xyz="1 0 0" />
+      <!--velocity dimensions assumed to be rad/s-->
       <limit
           effort="12.0"
-          lower="-0.78539"
-          upper="0.78539"
+          lower="-1.57075"
+          upper="1.57075"
           velocity="4.18879" />
       <origin
           xyz="0 0 -0.0919"
-          rpy="0 0 0" />
+          rpy="-0.523598 0 0" />
       <parent
           link="neck_pan" />
@@ -282,5 +282,5 @@
     </link>
     <joint
-        name="neck_tilt_to_crl_head"
+        name="tilt_neck_to_crl_head"
         type="fixed">
       <parent
@@ -319,5 +319,5 @@
           rpy="0 1.5707 1.5707" />
     </joint>
-    <xacro:property name="d435_cam_width" value="0.090"/>
+        <xacro:property name="d435_cam_width" value="0.090"/>
     <xacro:property name="d435_cam_height" value="0.025"/>
     <xacro:property name="d435_cam_depth" value="0.02505"/>
@@ -325,19 +325,39 @@
     <xacro:property name="d435_cam_mount_from_center_offset" value="0.0149"/>
     <xacro:property name="d435_cam_depth_py" value="0.0175"/>
-    <link name="camera_link">
-      <inertial>
-        <origin
-            xyz="${d435_cam_mount_from_center_offset} ${-d435_cam_depth_py} 0"
-            rpy="0 0 0"/>
-      </inertial>
-    </link>
+    <link
+        name="camera_link">
+        <origin xyz="${d435_cam_mount_from_center_offset} ${-d435_cam_depth_py} 0" rpy="0 0 0"/>
+	<mass
+            value="0.79"/>
+      <inertia ixx="0.003881243" ixy="0.0" ixz="0.0" iyy="0.000498940" iyz="0.0" izz="0.003879257" />
+	<visual>
+        <origin
+            xyz="0 0 0"
+            rpy="0 3.1415926 0" />
+        <geometry>
+          <mesh
+              filename="package://herb_description/meshes/head/realsense.dae" />
+        </geometry>
+        <material
+            name="">
+          <color
+              rgba="0.25 0.25 0.25 1" />
+        </material>
+      </visual>
+    	<collision>
+        <origin xyz="0 0 0" rpy="0 0 0"/>
+        <geometry>
+        <box size="${d435_cam_depth} ${d435_cam_width} ${d435_cam_height}"/>
+        </geometry>
+      </collision>
+      </link>
     <joint
         name="crl_head_to_realsense"
         type="fixed">
-        <parent
+      <parent
           link="crl_head" />
-        <child
+      <child
           link="camera_link" />
-        <origin
+      <origin
           xyz="0.008 -0.1690163 -0.0765607"
           rpy="0 1.5707 1.5707" />
