Commit message: Add Realsense camera to herb description (#60)
* Add realsense

* adjust neck tilt

File: robots/herb_base.urdf.xacro (robot description, xacro)
@@ -234,5 +234,5 @@
       <origin
           xyz="0 0 -0.0919"
-          rpy="0 0 0" />
+          rpy="-0.523598 0 0" />
       <parent
           link="neck_pan" />
@@ -370,4 +370,43 @@
           rpy="0 1.57075 0" />
     </joint>
+    <xacro:property name="d435_cam_width" value="0.090"/>
+    <xacro:property name="d435_cam_height" value="0.025"/>
+    <xacro:property name="d435_cam_depth" value="0.02505"/>
+    <xacro:property name="M_PI" value="3.1415926535897931" />
+    <xacro:property name="d435_cam_mount_from_center_offset" value="0.0149"/>
+    <xacro:property name="d435_cam_depth_py" value="0.0175"/>
+    <link
+      name="camera_link">
+      <origin xyz="${d435_cam_mount_from_center_offset} ${-d435_cam_depth_py} 0" rpy="0 0 0"/>
+      <mass value="0.79"/>
+      <inertia ixx="0.003881243" ixy="0.0" ixz="0.0" iyy="0.000498940" iyz="0.0" izz="0.003879257" />
+      <visual>
+        <origin
+          xyz="0 0 0"
+          rpy="0 3.1415926 0" />
+        <geometry>
+          <mesh
+            filename="package://herb_description/meshes/head/realsense.dae" />
+        </geometry>
+        <material name="">
+          <color rgba="0.25 0.25 0.25 1" />
+        </material>
+      </visual>
+      <collision>
+        <origin xyz="0 0 0" rpy="0 0 0"/>
+        <geometry>
+          <box size="${d435_cam_depth} ${d435_cam_width} ${d435_cam_height}"/>
+        </geometry>
+      </collision>
+    </link>
+    <joint
+      name="crl_head_to_realsense"
+      type="fixed">
+      <parent link="crl_head" />
+      <child link="camera_link" />
+      <origin
+        xyz="0.008 -0.1690163 -0.0765607"
+        rpy="0 1.5707 1.5707" />
+    </joint>
   </xacro:macro>
 </robot>
