Commit message: Adding changes on herb0

File: robots/fixed_transforms.urdf.xacro (robot description, xacro)
@@ -2,51 +2,133 @@
     <!-- Fixed Transforms -->
     <xacro:macro name="fixed_transforms">
-        <link name="head/kinect2/rgb">
-            <inertial>
-                <origin
-                    xyz="0. 0. 0."
-                    rpy="0. 0. 0." />
-                <mass value="0." />
-                <inertia
-                    ixx="0."
-                    ixy="0."
-                    ixz="0."
-                    iyy="0."
-                    iyz="0."
-                    izz="0." />
-            </inertial>
+        <!-- LEFT WAM -->
+        <!--
+        <link name="left/wam_base" />
+        <joint
+            name="left/wam_base"
+            type="fixed">
+            <origin
+                xyz="-.267 .331 0.685"
+                rpy="3.1416 -1.570796 0." />
+            <parent link="/herb_base" />
+            <child link="left/wam_base" />
+        </joint>
+        -->
+        <link name="/left/wam0" />
+        <joint
+            name="/left/wam0"
+            type="fixed">
+            <origin
+                xyz="0.22 0.14 .346"
+                rpy="0. 0. 0." />
+            <parent link="/left/wam_base" />
+            <child link="/left/wam0" />
+        </joint>
+        <!-- RIGHT WAM -->
+        <link name="/right/wam0" />
+        <joint
+            name="/right/wam0"
+            type="fixed">
+            <origin
+                xyz="0.22 0.14 .346"
+                rpy="0. 0. 0." />
+            <parent link="/right/wam_base" />
+            <child link="/right/wam0" />
+        </joint>
+        <!-- HEAD -->
+        <link name="/head/wam0" />
+        <joint
+            name="/head/wam0"
+            type="fixed">
+            <origin
+                xyz="-0.21908  0.0  1.27298"
+                rpy="0. 0. 0." />
+            <parent link="/herb_base" />
+            <child link="/head/wam0" />
+        </joint>
+        <!-- CAMERAS -->
+        <link name="/head/kinect2/rgb" />
+        <joint
+            name="/head/kinect2/rgb"
+            type="fixed">
+            <origin
+                xyz="0.15837 0.03257 0.09936"
+                rpy="2.84962 -1.5510 0.22398" />
+            <parent link="/head/wam2" />
+            <child link="/head/kinect2/rgb" />
+        </joint>
+        <link name="/head/kinect2/depth">
         </link>
         <joint
-            name="head/kinect2/rgb"
-            type="fixed">
-            <origin
-                xyz="0.11838 0.10257 0.01936"
-                rpy="2.84962 -1.5510 0.22398" />
-            <parent link="head/wam2" />
-            <child link="head/kinect/rgb" />
-        </joint>
-        <link name="head/kinect2/depth">
-            <inertial>
-                <origin
-                    xyz="0. 0. 0."
-                    rpy="0. 0. 0." />
-                <mass value="0." />
-                <inertia
-                    ixx="0."
-                    ixy="0."
-                    ixz="0."
-                    iyy="0."
-                    iyz="0."
-                    izz="0." />
-            </inertial>
-        </link>
-        <joint
-            name="head/kinect2/depth"
+            name="/head/kinect2/depth"
             type="fixed">
             <origin
                 xyz="-0.052 0. 0."
                 rpy="0. 0. 0." />
-            <parent link="head/kinect/rgb" />
-            <child link="head/kinect/depth" />
+            <parent link="/head/kinect2/rgb" />
+            <child link="/head/kinect2/depth" />
+        </joint>
+        <link name="/stargazer_lens" />
+        <joint
+            name="/stargazer_lens"
+            type="fixed">
+            <origin
+                xyz="-0.3024 0.2068 1.0258"
+                rpy="0. 0. 0." />
+            <parent link="/herb_base" />
+            <child link="/stargazer_lens" />
+        </joint>
+       <!-- HOKUYO -->
+       <link name="/base_hokuyo_front"/>
+       <link name="/base_hokuyo_right"/>
+       <link name="/base_hokuyo_left"/>
+       <joint
+             name="/base_hokuyo_left"
+             type="fixed">
+             <origin
+                  xyz = "-0.28613688816430005 0.25414007607683997 0.0811784"
+                  rpy = "2.0320379447076999 0 3.1416"/>
+             <parent link="/herb_base"/>
+             <child link="/base_hokuyo_left"/>
+       </joint>
+       <joint
+             name="/base_hokuyo_right"
+             type="fixed">
+             <origin
+                  xyz = "-0.32942801046380998 -0.31715770603423998 0.0811784"
+                  rpy = "-2.10565775700533 0 3.1416"/>
+             <parent link="/herb_base"/>
+             <child link="/base_hokuyo_right"/>
+       </joint>
+       <joint
+             name="/base_hokuyo_front"
+             type="fixed">
+             <origin
+                  xyz = "0.219 0 0.072"
+                  rpy = "0 0 3.1416"/>
+             <parent link="/herb_base"/>
+             <child link="/base_hokuyo_front"/>
+       </joint>
+        <!-- SEGWAY -->
+        <link name="/base_link"/>
+        <joint
+             name="/base_link"
+             type="fixed">
+             <origin
+                 xyz="0 0 0"
+                 rpy="0 0 0"/>
+             <parent link="/herb_base"/>
+             <child link="/base_link"/>
+        </joint>
+        <!-- CASTER WHEEL -->
+        <link name="/caster_contact" />
+        <joint
+            name="/caster_contact"
+            type="fixed">
+            <origin
+                xyz="-0.3175 0. 0."
+                rpy="0. 0. 0." />
+            <parent link="/herb_base" />
+            <child link="/caster_contact" />
         </joint>
     </xacro:macro>

Commit message: adding new kinect2 frames, possibly not correct yet

File: robots/fixed_transforms.urdf.xacro (robot description, xacro)
@@ -48,4 +48,11 @@
         </joint>
         <!-- CAMERAS -->
+        <joint
+            name="/head/kinect2_link"
+            type="fixed>
+            <origin
+                xyz="0.15837 0.03257 0.09936"
+                rpy="2.84962 -1.5510 0.22398" />
+        </joint>
         <link name="/head/kinect2/rgb" />
         <joint

Commit message: Adding proper joint and link for new kinect2_bridge (from the iai_kinect2 project)

File: robots/fixed_transforms.urdf.xacro (robot description, xacro)
@@ -48,4 +48,5 @@
         </joint>
         <!-- CAMERAS -->
+        <link name="/head/kinect2_link" />
         <joint
             name="/head/kinect2_link"
@@ -53,26 +54,7 @@
             <origin
                 xyz="0.15837 0.03257 0.09936"
-                rpy="2.84962 -1.5510 0.22398" />
-        </joint>
-        <link name="/head/kinect2/rgb" />
-        <joint
-            name="/head/kinect2/rgb"
-            type="fixed">
-            <origin
-                xyz="0.15837 0.03257 0.09936"
-                rpy="2.84962 -1.5510 0.22398" />
+                rpy="-1.570796 0 0" />
             <parent link="/head/wam2" />
-            <child link="/head/kinect2/rgb" />
-        </joint>
-        <link name="/head/kinect2/depth">
-        </link>
-        <joint
-            name="/head/kinect2/depth"
-            type="fixed">
-            <origin
-                xyz="-0.052 0. 0."
-                rpy="0. 0. 0." />
-            <parent link="/head/kinect2/rgb" />
-            <child link="/head/kinect2/depth" />
+            <child link="/head/kinect2_link"  />
         </joint>
         <link name="/stargazer_lens" />

Commit message: first guess at fixed transform for xtion on  herb

File: robots/fixed_transforms.urdf.xacro (robot description, xacro)
@@ -57,4 +57,14 @@
             <parent link="/head/wam2" />
             <child link="/head/kinect2_link"  />
+        </joint>
+        <link name="/head/skel_depth_frame" />
+        <joint
+            name="/head/skel_depth_frame"
+            type="fixed">
+            <origin
+                xyz="0.15837 0.03257 0.14936"
+                rpy="1.57079 -1.57019 1.57079" />
+            <parent link="/head/wam2" />
+            <child link="/head/skel_depth_frame"  />
         </joint>
         <link name="/stargazer_lens" />

Commit message: Changed extrinsics to correct-er

File: robots/fixed_transforms.urdf.xacro (robot description, xacro)
@@ -56,5 +56,15 @@
                 rpy="1.57079 -1.57019 1.57079" />
             <parent link="/head/wam2" />
-            <child link="/head/kinect2_link"  />
+            <child link="/head/kinect2_extrinsics_correction"  />
+        </joint>
+        <link name="/head/kinect2_extrinsics_correction" />
+        <joint
+            name="/head/kinect2_extrinsics_correction"
+            type="fixed">
+            <origin
+                xyz="0 0 0"
+                rpy="-0.065 0 0" />
+            <child link="/head/kinect2_link" />
+            <parent link="/head/kinect2_extrinsics_correction"  />
         </joint>
         <link name="/head/skel_depth_frame" />

Commit message: Set mass of fixed_transforms to zero.

File: robots/fixed_transforms.urdf.xacro (robot description, xacro)
@@ -1,4 +1,10 @@
 <robot xmlns:xacro="http://www.ros.org/wiki/xacro" name="fixed_transforms">
     <!-- Fixed Transforms -->
+    <xacro:macro name="no_inertial">
+      <inertial>
+        <mass value="0"/>
+        <inertia ixx="0" ixy="0" ixz="0" iyy="0" iyz="0" izz="0"/>
+      </inertial>
+    </xacro:macro>
     <xacro:macro name="fixed_transforms">
         <!-- LEFT WAM -->
@@ -15,5 +21,7 @@
         </joint>
         -->
-        <link name="/left/wam0" />
+        <link name="/left/wam0">
+          <xacro:no_inertia/>
+        </link>
         <joint
             name="/left/wam0"
@@ -26,5 +34,7 @@
         </joint>
         <!-- RIGHT WAM -->
-        <link name="/right/wam0" />
+        <link name="/right/wam0">
+          <xacro:no_inertia/>
+        </link>
         <joint
             name="/right/wam0"
@@ -37,5 +47,7 @@
         </joint>
         <!-- HEAD -->
-        <link name="/head/wam0" />
+        <link name="/head/wam0">
+          <xacro:no_inertia/>
+        </link>
         <joint
             name="/head/wam0"
@@ -48,5 +60,7 @@
         </joint>
         <!-- CAMERAS -->
-        <link name="/head/kinect2_link" />
+        <link name="/head/kinect2_link">
+          <xacro:no_inertia/>
+        </link>
         <joint
             name="/head/kinect2_link"
@@ -58,5 +72,7 @@
             <child link="/head/kinect2_extrinsics_correction"  />
         </joint>
-        <link name="/head/kinect2_extrinsics_correction" />
+        <link name="/head/kinect2_extrinsics_correction">
+          <xacro:no_inertia/>
+        </link>
         <joint
             name="/head/kinect2_extrinsics_correction"
@@ -68,5 +84,7 @@
             <parent link="/head/kinect2_extrinsics_correction"  />
         </joint>
-        <link name="/head/skel_depth_frame" />
+        <link name="/head/skel_depth_frame">
+          <xacro:no_inertia/>
+        </link>
         <joint
             name="/head/skel_depth_frame"
@@ -79,5 +97,7 @@
             <child link="/head/skel_depth_frame"  />
         </joint>
-        <link name="/stargazer_lens" />
+        <link name="/stargazer_lens">
+          <xacro:no_inertia/>
+        </link>
         <joint
             name="/stargazer_lens"
@@ -90,7 +110,31 @@
         </joint>
        <!-- HOKUYO -->
-       <link name="/base_hokuyo_front"/>
-       <link name="/base_hokuyo_right"/>
-       <link name="/base_hokuyo_left"/>
+       <link name="/base_hokuyo_front">
+          <xacro:no_inertia/>
+       </link>
+       <joint
+             name="/base_hokuyo_front"
+             type="fixed">
+             <origin
+                  xyz = "0.219 0 0.072"
+                  rpy = "0 0 3.1416"/>
+             <parent link="/herb_base"/>
+             <child link="/base_hokuyo_front"/>
+       </joint>
+       <link name="/base_hokuyo_right">
+          <xacro:no_inertia/>
+       </link>
+       <joint
+             name="/base_hokuyo_right"
+             type="fixed">
+             <origin
+                  xyz = "-0.32942801046380998 -0.31715770603423998 0.0811784"
+                  rpy = "-2.10565775700533 0 3.1416"/>
+             <parent link="/herb_base"/>
+             <child link="/base_hokuyo_right"/>
+       </joint>
+       <link name="/base_hokuyo_left">
+          <xacro:no_inertia/>
+       </link>
        <joint
              name="/base_hokuyo_left"
@@ -102,23 +146,6 @@
              <child link="/base_hokuyo_left"/>
        </joint>
-       <joint
-             name="/base_hokuyo_right"
-             type="fixed">
-             <origin
-                  xyz = "-0.32942801046380998 -0.31715770603423998 0.0811784"
-                  rpy = "-2.10565775700533 0 3.1416"/>
-             <parent link="/herb_base"/>
-             <child link="/base_hokuyo_right"/>
-       </joint>
-       <joint
-             name="/base_hokuyo_front"
-             type="fixed">
-             <origin
-                  xyz = "0.219 0 0.072"
-                  rpy = "0 0 3.1416"/>
-             <parent link="/herb_base"/>
-             <child link="/base_hokuyo_front"/>
-       </joint>
         <!-- SEGWAY -->
+        <!-- TODO: This should have no inertia. -->
         <link name="/base_link"/>
         <joint
@@ -132,5 +159,7 @@
         </joint>
         <!-- CASTER WHEEL -->
-        <link name="/caster_contact" />
+        <link name="/caster_contact">
+          <xacro:no_inertia/>
+        </link>
         <joint
             name="/caster_contact"

Commit message: fix no_inertia macro spelling

File: robots/fixed_transforms.urdf.xacro (robot description, xacro)
@@ -1,5 +1,5 @@
 <robot xmlns:xacro="http://www.ros.org/wiki/xacro" name="fixed_transforms">
     <!-- Fixed Transforms -->
-    <xacro:macro name="no_inertial">
+    <xacro:macro name="no_inertia">
       <inertial>
         <mass value="0"/>

Commit message: add tiny mass instead of 0 mass for 0 inertia

File: robots/fixed_transforms.urdf.xacro (robot description, xacro)
@@ -3,5 +3,5 @@
     <xacro:macro name="no_inertia">
       <inertial>
-        <mass value="0"/>
+        <mass value="0.00000001"/>
         <inertia ixx="0" ixy="0" ixz="0" iyy="0" iyz="0" izz="0"/>
       </inertial>
