Commit message: update urdf files for herb 3.0 base and frame
TODO: correctly position arms and test

File: robots/fixed_transforms.urdf.xacro (robot description, xacro)
@@ -9,16 +9,4 @@
     <xacro:macro name="fixed_transforms">
         <!-- LEFT WAM -->
-        <!--
-        <link name="left/wam_base" />
-        <joint
-            name="left/wam_base"
-            type="fixed">
-            <origin
-                xyz="-.267 .331 0.685"
-                rpy="3.1416 -1.570796 0." />
-            <parent link="/herb_base" />
-            <child link="left/wam_base" />
-        </joint>
-        -->
         <link name="/left/wam0">
           <xacro:no_inertia/>
@@ -46,128 +34,29 @@
             <child link="/right/wam0" />
         </joint>
-        <!-- HEAD -->
-        <link name="/head/wam0">
+	<!-- TODO: /head/skel_depth_frame ? -->
+        <link name="stargazer_lens">
           <xacro:no_inertia/>
         </link>
         <joint
-            name="/head/wam0"
-            type="fixed">
-            <origin
-                xyz="-0.21908  0.0  1.27298"
-                rpy="0. 0. 0." />
-            <parent link="/herb_base" />
-            <child link="/head/wam0" />
-        </joint>
-        <!-- CAMERAS -->
-        <link name="/head/kinect2_link">
-          <xacro:no_inertia/>
-        </link>
-        <joint
-            name="/head/kinect2_link"
-            type="fixed">
-            <origin
-                xyz="0.15837 0.03257 0.09936"
-                rpy="1.57079 -1.57019 1.57079" />
-            <parent link="/head/wam2" />
-            <child link="/head/kinect2_extrinsics_correction"  />
-        </joint>
-        <link name="/head/kinect2_extrinsics_correction">
-          <xacro:no_inertia/>
-        </link>
-        <joint
-            name="/head/kinect2_extrinsics_correction"
-            type="fixed">
-            <origin
-                xyz="0 0 0"
-                rpy="-0.195 0 0" />
-            <child link="/head/kinect2_link" />
-            <parent link="/head/kinect2_extrinsics_correction"  />
-        </joint>
-        <link name="/head/skel_depth_frame">
-          <xacro:no_inertia/>
-        </link>
-        <joint
-            name="/head/skel_depth_frame"
-            type="fixed">
-                <!--rpy="1.57079 -1.57019 1.57079" /> -->
-            <origin
-                xyz="0.15837 0.10257 0.09936"
-                rpy="0 1.57019 0" />
-            <parent link="/head/wam2" />
-            <child link="/head/skel_depth_frame"  />
-        </joint>
-        <link name="/stargazer_lens">
-          <xacro:no_inertia/>
-        </link>
-        <joint
-            name="/stargazer_lens"
+            name="stargazer_lens"
             type="fixed">
             <origin
                 xyz="-0.3024 0.2068 1.0258"
                 rpy="0. 0. 0." />
-            <parent link="/herb_base" />
-            <child link="/stargazer_lens" />
+            <parent link="herb_frame" />
+            <child link="stargazer_lens" />
         </joint>
-       <!-- HOKUYO -->
-       <link name="/base_hokuyo_front">
+        <!-- Dummy link to match ROS conventions. -->
+        <link name="base_link">
           <xacro:no_inertia/>
-       </link>
-       <joint
-             name="/base_hokuyo_front"
-             type="fixed">
-             <origin
-                  xyz = "0.219 0 0.072"
-                  rpy = "0 0 3.1416"/>
-             <parent link="/herb_base"/>
-             <child link="/base_hokuyo_front"/>
-       </joint>
-       <link name="/base_hokuyo_right">
-          <xacro:no_inertia/>
-       </link>
-       <joint
-             name="/base_hokuyo_right"
-             type="fixed">
-             <origin
-                  xyz = "-0.32942801046380998 -0.31715770603423998 0.0811784"
-                  rpy = "-2.10565775700533 0 3.1416"/>
-             <parent link="/herb_base"/>
-             <child link="/base_hokuyo_right"/>
-       </joint>
-       <link name="/base_hokuyo_left">
-          <xacro:no_inertia/>
-       </link>
-       <joint
-             name="/base_hokuyo_left"
-             type="fixed">
-             <origin
-                  xyz = "-0.28613688816430005 0.25414007607683997 0.0811784"
-                  rpy = "2.0320379447076999 0 3.1416"/>
-             <parent link="/herb_base"/>
-             <child link="/base_hokuyo_left"/>
-       </joint>
-        <!-- SEGWAY -->
-        <!-- TODO: This should have no inertia. -->
-        <link name="/base_link"/>
+	</link>
         <joint
-             name="/base_link"
+             name="base_link"
              type="fixed">
              <origin
                  xyz="0 0 0"
                  rpy="0 0 0"/>
-             <parent link="/herb_base"/>
-             <child link="/base_link"/>
-        </joint>
-        <!-- CASTER WHEEL -->
-        <link name="/caster_contact">
-          <xacro:no_inertia/>
-        </link>
-        <joint
-            name="/caster_contact"
-            type="fixed">
-            <origin
-                xyz="-0.3175 0. 0."
-                rpy="0. 0. 0." />
-            <parent link="/herb_base" />
-            <child link="/caster_contact" />
+             <parent link="neobotix_base"/>
+             <child link="base_link"/>
         </joint>
     </xacro:macro>

File: robots/herb.urdf.xacro (robot description, xacro)
@@ -60,10 +60,10 @@
   <joint name="/left/wam_mount" type="fixed">
     <origin xyz="-0.266700 0.332276 0.694588" rpy="0 ${-pi/2} ${pi}"/>
-    <parent link="/herb_base"/>
+    <parent link="herb_frame"/>
     <child link="/left/wam_base"/>
   </joint>
   <joint name="/right/wam_mount" type="fixed">
     <origin xyz="-0.266700 -0.049121 0.694588" rpy="0 ${-pi/2} ${pi}"/>
-    <parent link="/herb_base"/>
+    <parent link="herb_frame"/>
     <child link="/right/wam_base"/>
   </joint>

File: robots/herb_base.urdf.xacro (robot description, xacro)
@@ -1,145 +1,318 @@
 <robot xmlns:xacro="http://www.ros.org/wiki/xacro" name="herb_base">
   <xacro:macro name="herb_base" params="prefix">
-    <link name="${prefix}/herb_base">
-      <inertial>
-        <origin xyz="-0.0809027982480422 0.00803042872866252 0.350693951417865" rpy="0 0 0"/>
-        <mass value="118.064183849969"/>
-        <inertia
-            ixx="9.67307679892718" ixy="-0.109440074935232" ixz="-2.47806317387667"
-            iyx="0.00000000000000" iyy="10.2602519302075"   iyz="0.237417248956334"
-            izx="0.00000000000000" izy="0.00000000000000"   izz="5.27441929623381"/>
-      </inertial>
-      <visual>
-        <origin xyz="0 0 0" rpy="0 0 0"/>
-        <geometry>
-          <mesh filename="package://herb_description/meshes/base/herb_base.dae"/>
-        </geometry>
-        <material name="">
-          <color rgba="0.086 0.408 0.565 1"/>
-        </material>
-      </visual>
-      <collision>
-        <geometry>
-          <mesh filename="package://herb_description/meshes/base/herb_base_collision.STL"/>
-        </geometry>
-      </collision>
-    </link>
-    <link name="${prefix}/segway_wheel_left">
-      <inertial>
-        <origin xyz="1.46252801536129E-12 4.14215883814961E-12 0.0471293756901144" rpy="0 0 0"/>
-        <mass value="6.7355511743555"/>
-        <inertia
-            ixx="0.092576479522193" ixy="-2.98851956896402E-06" ixz="1.06719826192435E-09"
-            iyx="0.000000000000000" iyy="0.0925839088729686"    iyz="3.02916843456587E-09"
-            izx="0.000000000000000" izy="0.0000000000000000"    izz="0.178365793214305"/>
-      </inertial>
-      <visual>
-        <origin xyz="0 0 0" rpy="0 0 0"/>
-        <geometry>
-          <mesh filename="package://herb_description/meshes/segway/segway_wheel_left.dae"/>
-        </geometry>
-        <material name="">
-          <color rgba="0.2 0.2 0.2 1"/>
-        </material>
-      </visual>
-      <collision>
-        <geometry>
-          <mesh filename="package://herb_description/meshes/segway/segway_wheel_left_collision.STL"/>
-        </geometry>
-      </collision>
-    </link>
-    <joint name="${prefix}/segway_wheel_left" type="continuous">
-      <origin xyz="0 0.231771918932663 0.23158735611353" rpy="-1.5707963267949 -0.115508699092541 0"/>
-      <parent link="${prefix}/herb_base"/>
-      <child link="${prefix}/segway_wheel_left"/>
-      <axis xyz="0 0 -1"/>
-    </joint>
-    <link name="${prefix}/segway_wheel_right">
-      <inertial>
-        <origin xyz="-1.06512021424976E-15 4.39884240144295E-12 0.0471293756901144" rpy="0 0 0"/>
-        <mass value="6.7355511743555"/>
-        <inertia
-            ixx="0.0925754265920571" ixy="-1.49287030220407E-10" ixz="-1.57504574648507E-16"
-            iyx="0.0000000000000000" iyy="0.0925849618031043"    iyz="3.21166212934922E-09"
-            izx="0.0000000000000000" izy="0.0000000000000000"    izz="0.178365793214305"/>
-      </inertial>
-      <visual>
-        <origin xyz="0 0 0" rpy="0 0 0"/>
-        <geometry>
-          <mesh filename="package://herb_description/meshes/segway/segway_wheel_right.dae"/>
-        </geometry>
-        <material name="">
-          <color rgba="0.2 0.2 0.2 1"/>
-        </material>
-      </visual>
-      <collision>
-        <geometry>
-          <mesh filename="package://herb_description/meshes/segway/segway_wheel_right_collision.STL"/>
-        </geometry>
-      </collision>
-    </link>
-    <joint name="${prefix}/segway_wheel_right" type="continuous">
-      <origin xyz="0 -0.231771918932663 0.231587356113537" rpy="-1.5707963267949 0.0751085369855802 3.14159265358979"/>
-      <parent link="${prefix}/herb_base"/>
-      <child link="${prefix}/segway_wheel_right"/>
-      <axis xyz="0 0 1"/>
-    </joint>
-    <link name="${prefix}/head/wam1">
-      <inertial>
-        <origin xyz="-0.000143379867888344 -0.0221150249825213 -0.0159634421249915" rpy="0 0 0"/>
-        <mass value="0.699914058257394"/>
-        <inertia
-            ixx="0.00280646384099311" ixy="6.06589910190362E-06" ixz="1.10356402708704E-06"
-            iyx="0.00000000000000000" iyy="0.000592185892279803" iyz="-0.000170166312219621"
-            izx="0.00000000000000000" izy="0.000000000000000000" izz="0.00264000882290309"/>
-      </inertial>
-      <visual>
-        <origin xyz="0 0 0" rpy="0 0 0"/>
-        <geometry>
-          <mesh filename="package://herb_description/meshes/head/head_wam1.dae"/>
-        </geometry>
-        <material name="">
-          <color rgba="0.086 0.408 0.565 1"/>
-        </material>
-      </visual>
-      <collision>
-        <geometry>
-        <mesh filename="package://herb_description/meshes/head/head_wam1_collision.STL"/></geometry>
-      </collision>
-    </link>
-    <joint name="${prefix}/head/wam1" type="fixed">
-      <origin xyz="-0.219043 0 1.282513" rpy="0 0 0"/>
-      <parent link="${prefix}/herb_base"/>
-      <child link="${prefix}/head/wam1"/>
-      <axis xyz="0 0 1"/>
-    </joint>
-    <link name="${prefix}/head/wam2">
-      <inertial>
-        <origin xyz="0.00676836020340077 0.0512494218238631 0.00803256112914554" rpy="0 0 0"/>
-        <mass value="1.54049400601599"/>
-        <inertia
-            ixx="0.0067835645951359" ixy="-0.000318213388742608" ixz="-0.000190037318422281"
-            iyx="0.0000000000000000" iyy="0.00662131693308525"   iyz="-0.000833945040621095"
-            izx="0.0000000000000000" izy="0.00000000000000000"   izz="0.00344340957107467"/>
-      </inertial>
-      <visual>
-        <origin xyz="0 0 0" rpy="0 0 0"/>
-        <geometry>
-          <mesh filename="package://herb_description/meshes/head/head_wam2.dae"/>
-        </geometry>
-        <material name="">
-          <color rgba="0.63921568627451 0.63921568627451 0.686274509803922 1"/>
-        </material>
-      </visual>
-      <collision>
-        <geometry>
-        <mesh filename="package://herb_description/meshes/head/head_wam2_collision.STL"/></geometry>
-      </collision>
-    </link>
-    <joint name="${prefix}/head/wam2" type="fixed">
-      <origin xyz="0 0 0" rpy="1.5707963267949 0.3 4.20797196041016E-14"/>
-      <parent link="${prefix}/head/wam1"/>
-      <child link="${prefix}/head/wam2"/>
-      <axis xyz="0 0 1"/>
+    <link
+        name="herb_frame">
+      <!--check inertias and mass-->
+      <inertial>
+        <origin
+            xyz="0 0 0"
+            rpy="0 0 0" />
+        <mass
+            value="75.88" />
+        <inertia
+            ixx="11.92524"
+            ixy="0.00418"
+            ixz="0.00448"
+            iyy="4.13145"
+            iyz="2.60056"
+            izz="10.77706" />
+      </inertial>
+      <visual>
+        <origin
+            xyz="0 0 0"
+            rpy="1.57075 0 3.141592" />
+        <geometry>
+          <mesh
+              filename="package://herb_description/meshes/base/herb_frame.STL" />
+        </geometry>
+        <material
+            name="">
+          <color
+              rgba="0.3 0 0 1" />
+        </material>
+      </visual>
+      <collision>
+        <origin
+            xyz="0 0 0"
+            rpy="1.57075 0 -1.57075" />
+        <geometry>
+          <mesh
+              filename="package://herb_description/meshes/base/herb_frame_collision.STL" />
+        </geometry>
+      </collision>
+    </link>
+    <link
+        name="neobotix_base">
+      <!--check inertias and mass-->
+      <inertial>
+        <origin
+            xyz="0 -0.074086 -1.040385"
+            rpy="0 0 0" />
+        <mass
+            value="80" />
+        <inertia
+            ixx="9.25557"
+            ixy="0.00548"
+            ixz="0.00573"
+            iyy="7.60171"
+            iyz="1.02901"
+            izz="9.76036" />
+      </inertial>
+      <visual>
+        <origin
+            xyz="0 0 0"
+            rpy="0 0 0"/>
+        <geometry>
+          <mesh
+              filename="package://herb_description/meshes/base/herb_neobotix_base.STL" />
+        </geometry>
+        <material
+            name="">
+          <color
+              rgba="0.3 0.3 0.3 1" />
+        </material>
+      </visual>
+      <collision>
+        <origin
+            xyz="0 0 0"
+            rpy="1.57075 0 1.57075" />
+        <geometry>
+          <mesh
+              filename="package://herb_description/meshes/base/herb_neobotix_base_collision.STL" />
+        </geometry>
+      </collision>
+    </link>
+    <joint
+        name="frame_to_base"
+        type="fixed">
+      <origin
+          xyz="0 -0.074086 -1.040385"
+          rpy="0 0 3.141592" />
+      <parent
+          link="herb_frame" />
+      <child
+          link="neobotix_base" />
+    </joint>
+    <link
+        name="neck_pan">
+      <!--check inertias and mass-->
+      <inertial>
+        <origin
+            xyz="0 0.124900 0.050806"
+            rpy="0 0 0" />
+        <mass
+            value="0.81" />
+        <inertia
+            ixx="0.00694"
+            ixy="0"
+            ixz="0"
+            iyy="0.00713"
+            iyz="0"
+            izz="0.00081" />
+      </inertial>
+      <visual>
+        <origin
+            xyz="0 0 0"
+            rpy="0 0 0" />
+        <geometry>
+          <mesh
+              filename="package://herb_description/meshes/head/herb_neck_pan.STL" />
+        </geometry>
+        <material
+            name="">
+          <color
+              rgba="0.5 0.5 0.5 1" />
+        </material>
+      </visual>
+      <collision>
+        <origin
+            xyz="0 0 0"
+            rpy="-1.57075 0 0" />
+        <geometry>
+          <mesh
+              filename="package://herb_description/meshes/head/herb_neck_pan_collision.STL" />
+        </geometry>
+      </collision>
+    </link>
+    <joint
+        name="frame_to_neck_pan"
+        type="revolute">
+      <axis
+          xyz="0 0 1" />
+      <!--velocity is arbitrary; check against real values-->
+      <limit
+          effort="4.0"
+          lower="-1.57075"
+          upper="1.57075"
+          velocity="1" />
+      <origin
+          xyz="0 0.124900 0.050806"
+          rpy="3.141592 0 0" />
+      <parent
+          link="herb_frame" />
+      <child
+          link="neck_pan" />
+    </joint>
+    <link
+        name="neck_tilt" >
+      <inertial>
+        <origin
+            xyz="0 0.124900 0.142633"
+            rpy="0 0 0" />
+        <mass
+            value="0.32" />
+        <inertia
+            ixx="0.00046"
+            ixy="0"
+            ixz="-0.00002"
+            iyy="0.00142"
+            iyz="0"
+            izz="0.00120" />
+      </inertial>
+      <visual>
+        <origin
+            xyz="0 0 0"
+            rpy="0 0 0" />
+        <geometry>
+          <mesh
+              filename="package://herb_description/meshes/head/herb_neck_tilt.STL" />
+        </geometry>
+        <material
+            name="">
+          <color
+              rgba="0.5 0.5 0.5 1" />
+        </material>
+      </visual>
+      <collision>
+        <origin
+            xyz="0 0 0"
+            rpy="-1.57075 0 3.141592" />
+        <geometry>
+          <mesh
+              filename="package://herb_description/meshes/head/herb_neck_tilt_collision.STL" />
+        </geometry>
+      </collision>
+    </link>
+    <joint
+        name="pan_neck_to_tilt_neck"
+        type="revolute">
+      <axis
+          xyz="1 0 0" />
+      <!--velocity is arbitrary; check against real values-->
+      <limit
+          effort="24.0"
+          lower="-1.57075"
+          upper="1.57075"
+          velocity="1" />
+      <origin
+          xyz="0 0 -0.0919"
+          rpy="0 0 0" />
+      <parent
+          link="neck_pan" />
+      <child
+          link="neck_tilt" />
+    </joint>
+    <link
+        name="crl_head">
+      <!--check inertias and mass-->
+      <inertial>
+        <origin
+            xyz="0.001 0.181699 0.377811"
+            rpy="0 0 0" />
+        <mass
+            value="3.01" />
+        <inertia
+            ixx="0.02735"
+            ixy="-0.00053"
+            ixz="0.00024"
+            iyy="0.00962"
+            iyz="-0.00521"
+            izz="0.02487" />
+      </inertial>
+      <visual>
+        <origin
+            xyz="0 0 0"
+            rpy="0 0 0" />
+        <geometry>
+          <mesh
+              filename="package://herb_description/meshes/head/herb_crl_head.STL" />
+        </geometry>
+        <material
+            name="">
+          <color
+              rgba="0 0 0 1" />
+        </material>
+      </visual>
+      <collision>
+        <origin
+            xyz="-0.003895 -0.236 0.0575"
+            rpy="0 3.141592 0" />
+        <geometry>
+          <mesh
+              filename="package://herb_description/meshes/head/herb_crl_head_collision.STL" />
+        </geometry>
+      </collision>
+    </link>
+    <joint
+        name="tilt_neck_to_crl_head"
+        type="fixed">
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
Commit message: fixed frame

File: robots/fixed_transforms.urdf.xacro (robot description, xacro)
@@ -3,5 +3,5 @@
     <xacro:macro name="no_inertia">
       <inertial>
-        <mass value="0"/>
+        <mass value="0.001"/>
         <inertia ixx="0" ixy="0" ixz="0" iyy="0" iyz="0" izz="0"/>
       </inertial>

File: robots/herb_base.urdf.xacro (robot description, xacro)
@@ -63,5 +63,5 @@
       <origin
           xyz="0 0 1.05"
-          rpy="0 0 -1.57075" />
+          rpy="0 0 0" />
       <parent
           link="base_footprint" />
@@ -164,13 +164,8 @@
     <joint
         name="frame_to_neck_pan"
-        type="revolute">
+        type="fixed">
       <axis
           xyz="0 0 1" />
       <!--velocity dimensions assumed to be rad/s-->
-      <limit
-          effort="2.0"
-          lower="-1.57075"
-          upper="1.57075"
-          velocity="6.28319" />
       <origin
           xyz="0 0.124900 0.050806"
@@ -223,16 +218,11 @@
     <joint
         name="pan_neck_to_tilt_neck"
-        type="revolute">
+        type="fixed">
       <axis
           xyz="1 0 0" />
       <!--velocity dimensions assumed to be rad/s-->
-      <limit
-          effort="12.0"
-          lower="-1.57075"
-          upper="1.57075"
-          velocity="4.18879" />
       <origin
           xyz="0 0 -0.0919"
-          rpy="0 0 0" />
+          rpy="0 -0.698132 0" />
       <parent
           link="neck_pan" />
@@ -241,5 +231,5 @@
     </joint>
     <link
-        name="crl_head">
+        name="multisense/head">
       <!--check inertias and mass-->
       <inertial>
@@ -287,8 +277,8 @@
           link="neck_tilt" />
       <child
-          link="crl_head" />
+          link="multisense/head" />
       <origin
           xyz="-0.003895 -0.0575 -0.236"
-          rpy="-1.57075 0 0" />
+          rpy="-3.14159 0 0" />
     </joint>
     <link
@@ -336,5 +326,5 @@
         type="fixed">
       <parent
-          link="crl_head" />
+          link="multisense/head" />
       <child
           link="kinect" />
