Commit message: reorganize urdf + cleanup fixed transforms

File: robots/fixed_transforms.urdf.xacro (robot description, xacro)
@@ -8,56 +8,29 @@
     </xacro:macro>
     <xacro:macro name="fixed_transforms">
-        <!-- LEFT WAM -->
-        <link name="/left/wam0">
-          <xacro:no_inertia/>
-        </link>
-        <joint
-            name="/left/wam0"
-            type="fixed">
-            <origin
-                xyz="0.22 0.14 .346"
-                rpy="0. 0. 0." />
-            <parent link="/left/wam_base" />
-            <child link="/left/wam0" />
-        </joint>
-        <!-- RIGHT WAM -->
-        <link name="/right/wam0">
-          <xacro:no_inertia/>
-        </link>
-        <joint
-            name="/right/wam0"
-            type="fixed">
-            <origin
-                xyz="0.22 0.14 .346"
-                rpy="0. 0. 0." />
-            <parent link="/right/wam_base" />
-            <child link="/right/wam0" />
-        </joint>
-	<!-- TODO: /head/skel_depth_frame ? -->
-        <link name="stargazer_lens">
-          <xacro:no_inertia/>
-        </link>
-        <joint
-            name="stargazer_lens"
-            type="fixed">
-            <origin
-                xyz="-0.3024 0.2068 1.0258"
-                rpy="0. 0. 0." />
-            <parent link="herb_frame" />
-            <child link="stargazer_lens" />
-        </joint>
-        <!-- Dummy link to match ROS conventions. -->
-        <link name="base_link">
-          <xacro:no_inertia/>
-	</link>
-        <joint
-             name="base_link"
-             type="fixed">
-             <origin
-                 xyz="0 0 0"
-                 rpy="0 0 0"/>
-             <parent link="neobotix_base"/>
-             <child link="base_link"/>
-        </joint>
-    </xacro:macro>
+    <!-- LEFT WAM -->
+    <link name="/left/wam0">
+      <xacro:no_inertia/>
+    </link>
+    <joint
+        name="/left/wam0"
+        type="fixed">
+        <origin
+            xyz="0.22 0.14 .346"
+            rpy="0. 0. 0." />
+        <parent link="/left/wam_base" />
+        <child link="/left/wam0" />
+    </joint>
+    <!-- RIGHT WAM -->
+    <link name="/right/wam0">
+      <xacro:no_inertia/>
+    </link>
+    <joint
+        name="/right/wam0"
+        type="fixed">
+        <origin
+            xyz="0.22 0.14 .346"
+            rpy="0. 0. 0." />
+        <parent link="/right/wam_base" />
+        <child link="/right/wam0" />
+    </joint>
 </robot>

File: robots/herb_base.urdf.xacro (robot description, xacro)
@@ -1,8 +1,8 @@
 <robot xmlns:xacro="http://www.ros.org/wiki/xacro" name="herb_base">
   <xacro:macro name="herb_base" params="prefix">
-    <link name="base_footprint">
-      <inertial>
-        <origin
-            xyz="0 0 0"
+    <link name="base_link">
+      <inertial>
+        <origin
+            xyz="-0.074086 0 -0.051244"
             rpy="0 0 0" />
         <mass
@@ -17,4 +17,67 @@
       </inertial>
     </link>
+    <joint
+        name="root_to_neobotix"
+        type="fixed">
+      <origin
+          xyz="0 0 0"
+          rpy="0 0 1.57075" />
+      <parent
+          link="base_link" />
+      <child
+          link="neobotix_base" />
+    </joint>
+    <link
+        name="neobotix_base">
+      <!--check inertias and mass-->
+      <inertial>
+        <origin
+            xyz="0 0 0"
+            rpy="0 0 0" />
+        <mass
+            value="80" />
+        <inertia
+            ixx="9.25557"
+            ixy="0.00548"
+            ixz="0.00573"
+            iyy="7.60171"
+            iyz="1.02901"
+            izz="9.76036" />
+      </inertial>
+      <visual>
+        <origin
+            xyz="0 0 0"
+            rpy="0 0 0"/>
+        <geometry>
+          <mesh
+              filename="package://herb_description/meshes/base/herb_neobotix_base.STL" />
+        </geometry>
+        <material
+            name="">
+          <color
+              rgba="0.3 0.3 0.3 1" />
+        </material>
+      </visual>
+      <collision>
+        <origin
+            xyz="0 0 0"
+            rpy="1.57075 0 1.57075" />
+        <geometry>
+          <mesh
+              filename="package://herb_description/meshes/base/herb_neobotix_base_collision.STL" />
+        </geometry>
+      </collision>
+    </link>
+    <joint
+        name="neobotix_to_frame"
+        type="fixed">
+      <origin
+          xyz="0 -0.074086 1.101244"
+          rpy="0 0 3.141592" />
+      <parent
+          link="neobotix_base" />
+      <child
+          link="herb_frame" />
+    </joint>
     <link
         name="herb_frame">
@@ -58,67 +121,4 @@
       </collision>
     </link>
-    <joint
-        name="root_to_frame"
-        type="fixed">
-      <origin
-          xyz="0 0 1.05"
-          rpy="0 0 -1.57075" />
-      <parent
-          link="base_footprint" />
-      <child
-          link="herb_frame" />
-    </joint>
-    <link
-        name="neobotix_base">
-      <!--check inertias and mass-->
-      <inertial>
-        <origin
-            xyz="0 -0.074086 -1.101244"
-            rpy="0 0 0" />
-        <mass
-            value="80" />
-        <inertia
-            ixx="9.25557"
-            ixy="0.00548"
-            ixz="0.00573"
-            iyy="7.60171"
-            iyz="1.02901"
-            izz="9.76036" />
-      </inertial>
-      <visual>
-        <origin
-            xyz="0 0 0"
-            rpy="0 0 0"/>
-        <geometry>
-          <mesh
-              filename="package://herb_description/meshes/base/herb_neobotix_base.STL" />
-        </geometry>
-        <material
-            name="">
-          <color
-              rgba="0.3 0.3 0.3 1" />
-        </material>
-      </visual>
-      <collision>
-        <origin
-            xyz="0 0 0"
-            rpy="1.57075 0 1.57075" />
-        <geometry>
-          <mesh
-              filename="package://herb_description/meshes/base/herb_neobotix_base_collision.STL" />
-        </geometry>
-      </collision>
-    </link>
-    <joint
-        name="frame_to_base"
-        type="fixed">
-      <origin
-          xyz="0 -0.074086 -1.101244"
-          rpy="0 0 3.141592" />
-      <parent
-          link="herb_frame" />
-      <child
-          link="neobotix_base" />
-    </joint>
     <link
         name="neck_pan">
