Commit message: Added joint limits and stuff.

File: config/bh280_params.urdf.xacro (robot description, xacro)
@@ -1,8 +1,9 @@
 <template xmlns:xacro="http://www.ros.org/wiki/xacro">
     <xacro:property name="pi" value="3.14159265359"/>
+    <!-- FIXME: Fix the joint efforts. -->
     <xacro:macro name="bh280_finger" params="index">
         <!-- proximal joint -->
         <joint name="j${index}1">
-            <limit lower="0" upper="${140*(pi/180)}" effort="" velocity=""/>
+            <limit lower="0" upper="${140*(pi/180)}" effort="0" velocity="2.0"/>
         </joint>
         <!-- Frame 2 (finger inner link frame) with fingertip torque sensor -->
@@ -10,13 +11,13 @@
             <inertial>
                 <origin xyz="0.023133 0.00078642 0.00052792"/>
-                <mass>0.062139</mass>
+                <mass value="0.062139"/>
                 <inertia ixx="4.8162e-006" ixy="5.7981e-007" ixz="-7.2483e-007"
                                            iyy="4.3317e-005" iyz="-2.6653e-009"
-                                                             izz=" 4.4441e-005"/>
+                                                             izz= "4.4441e-005"/>
             </inertial>
         </link>
         <!-- distal joint -->
         <joint name="j${index}2">
-            <limit lower="0" upper="${48*(pi/180)}" effort="" velocity=""/>
+            <limit lower="0" upper="${48*(pi/180)}" effort="0" velocity="2.0"/>
         </joint>
         <!-- Frame 3 (fingertip frame) with fingertip pressure pad -->
@@ -24,8 +25,8 @@
             <inertial>
                 <origin xyz="0.02295 0.0010739 0.00041752"/>
-                <mass>0.04166</mass>
+                <mass value="0.04166"/>
                 <inertia ixx="3.1199e-006" ixy="4.5115e-007" ixz="-2.9813e-007"
                                            iyy="1.6948e-005" iyz="-1.8635e-008"
-                                                             izz=" 1.5809e-005"/>
+                                                             izz= "1.5809e-005"/>
             </inertial>
         </link>
@@ -33,5 +34,5 @@
     <xacro:macro name="bh280_spread" params="index">
         <joint name="j${index}0">
-            <limit lower="0" upper="${180*(pi/180)}" effort="" velocity=""/>
+            <limit lower="0" upper="${180*(pi/180)}" effort="0" velocity="2.0"/>
         </joint>
         <!-- Frame 1 (finger spread frame) -->
@@ -39,5 +40,5 @@
             <inertial>
                 <origin xyz="0.030616 -7.3219e-005 -0.011201"/>
-                <mass>0.14109</mass>
+                <mass value="0.14109"/>
                 <inertia ixx="2.0672e-005" ixy="2.6024e-007" ixz="6.3481e-006"
                                            iyy="7.4105e-005" iyz="1.7118e-008"
@@ -50,8 +51,8 @@
         <inertial>
             <origin xyz="5.0019e-005 -0.0044561 0.037268"/>
-            <mass>0.60858</mass>
+            <mass value="0.60858"/>
             <inertia ixx="0.0006986" ixy="2.7577e-007" ixz="-7.8138e-007"
                                      iyy="0.00050354"  iyz="-6.44e-005"
-                                                       izz="0.00062253"/>
+                                                       izz= "0.00062253"/>
         </inertial>
     </link>

File: config/wam_params.urdf.xacro (robot description, xacro)
@@ -6,9 +6,8 @@
         <inertial>
             <origin xyz="-0.02017671 -0.26604706 -0.14071720"/>
-            <mass>9.97059584</mass>
+            <mass value="9.97059584"/>
             <inertia ixx="0.10916849" ixy="0.00640270" ixz="0.02557874"
                                       iyy="0.18294303" iyz="0.00161433"
                                                        izz="0.11760385"/>
-            <inertia ixx="" ixy="" ixz="" iyy="" iyz="" izz=""/>
         </inertial>
     </link>
@@ -16,8 +15,8 @@
         <inertial>
             <origin xyz="-0.00443422 0.12189039 -0.00066489"/>
-            <mass>10.76768767</mass>
+            <mass value="10.76768767"/>
             <inertia ixx="0.13488033" ixy="-0.00213041" ixz="-0.00012485"
-                                      iyy=" 0.11328369" iyz=" 0.00068555"
-                                                        izz=" 0.09046330"/>
+                                      iyy= "0.11328369" iyz= "0.00068555"
+                                                        izz= "0.09046330"/>
         </inertial>
     </link>
@@ -25,8 +24,8 @@
         <inertial>
             <origin xyz="-0.00236983 0.03105614 0.01542114"/>
-            <mass>3.87493756</mass>
-            <inertia ixx="0.02140958" ixy="0.00027172" ixz=" 0.00002461"
+            <mass value="3.87493756"/>
+            <inertia ixx="0.02140958" ixy="0.00027172" ixz="+0.00002461"
                                       iyy="0.01377875" iyz="-0.00181920"
-                                                       izz=" 0.01558906"/>
+                                                       izz= "0.01558906"/>
         </inertial>
     </link>
@@ -34,8 +33,8 @@
         <inertial>
             <origin xyz="-0.03825858 0.20750770 0.00003309"/>
-            <mass>1.80228141</mass>
-            <inertia ixx="0.05911077" ixy="-0.00249612" ixz=" 0.00000738"
-                                      iyy=" 0.00324550" iyz="-0.00001767"
-                                                        izz=" 0.05927043"/>
+            <mass value="1.80228141"/>
+            <inertia ixx="0.05911077" ixy="-0.00249612" ixz= "0.00000738"
+                                      iyy= "0.00324550" iyz="-0.00001767"
+                                                        izz= "0.05927043"/>
         </inertial>
     </link>
@@ -44,8 +43,8 @@
         <inertial>
             <origin xyz="0.00498512 -0.00022942 0.13271662"/>
-            <mass>2.40016804</mass>
+            <mass value="2.40016804"/>
             <inertia ixx="0.01491672" ixy="0.00001741" ixz="-0.00150604"
                                       iyy="0.01482922" iyz="-0.00002109"
-                                                       izz=" 0.00294463"/>
+                                                       izz= "0.00294463"/>
         </inertial>
     </link>
@@ -53,8 +52,8 @@
         <inertial>
             <origin xyz="0.00008921 0.00511217 0.00435824"/>
-            <mass>0.12376019</mass>
+            <mass value="0.12376019"/>
             <inertia ixx="0.00005029" ixy="0.00000020" ixz="-0.00000005"
                                       iyy="0.00007582" iyz="-0.00000359"
-                                                       izz=" 0.00006270"/>
+                                                       izz= "0.00006270"/>
         </inertial>
     </link>
@@ -62,8 +61,8 @@
         <inertial>
             <origin xyz="-0.00012262 -0.01703194 0.02468336"/>
-            <mass>0.41797364</mass>
+            <mass value="0.41797364"/>
             <inertia ixx="0.00055516" ixy="0.00000061" ixz="-0.00000074"
                                       iyy="0.00024367" iyz="-0.00004590"
-                                                       izz=" 0.00045358"/>
+                                                       izz= "0.00045358"/>
         </inertial>
     </link>
@@ -73,7 +72,7 @@
         <inertial>
             <origin xyz="-0.00007974 0.00016313 -0.00323552"/>
-            <mass>0.06864753</mass>
+            <mass value="0.06864753"/>
             <inertia ixx="0.00003773" ixy="-0.00000019" ixz="0.00000000"
-                                      iyy=" 0.00003806" iyz="0.00000000"
+                                      iyy= "0.00003806" iyz="0.00000000"
                                                         izz="0.00007408"/>
         </inertial>
@@ -106,5 +105,5 @@
     </joint>
     <joint name="j7">
-        <limit lower="${-172*(pi/180)}" upper="${-172*(pi/180)}" effort="0.174" velocity="2.5"/>
+        <limit lower="${-172*(pi/180)}" upper="${172*(pi/180)}" effort="0.174" velocity="2.5"/>
     </joint>
 </template>

Commit message: Fixed the BH model.

File: config/bh280_params.urdf.xacro (robot description, xacro)
@@ -48,5 +48,5 @@
     </xacro:macro>
     <!-- Frame W with palm pad -->
-    <link name="base_link">
+    <link name="hand_base">
         <inertial>
             <origin xyz="5.0019e-005 -0.0044561 0.037268"/>

File: robots/BHD280_URDF.URDF (robot description, URDF)
Before this commit: robot BHD280_URDF, 9 links, 8 joints
Links:
- removed link base_link
- added link hand_base, mass 0.377966381303299; collision mesh filename=package://BHD280_URDF/meshes/hand_base.STL; visual mesh filename=package://BHD280_URDF/meshes/hand_base.STL
- link finger0_1: mass 31321.1214212939 -> 31321.121421294
- link finger2_1: mass 31321.1214212939 -> 31321.121421294
Joints:
- joint j00: parent base_link -> hand_base
- joint j01: origin xyz=0.0500000000000005 0.000799999999999978 0 rpy=1.5707963267949 0 0 -> xyz=0.0500000000000006 0.000799999999999964 0 rpy=1.5707963267949 0 0
- joint j02: origin xyz=0.0699356847396221 0.003 0.000200000000006962 rpy=-3.77533479986348E-14 -4.45260733378639E-14 0.698131700822416 -> xyz=0.069935684739622 0.00300000000000003 0.000200000000006934 rpy=-3.77533479986348E-14 -4.45260733378639E-14 0.698131700822416
- joint j10: parent base_link -> hand_base
- joint j11: origin xyz=0.0499991459461259 0.000799999999999367 -0.000292240753933679 rpy=1.5707963267949 0 -4.93038065763132E-32 -> xyz=0.0499991459461259 0.000799999999999367 -0.000292240753933651 rpy=1.5707963267949 0 -4.93038065763132E-32
- joint j12: origin xyz=0.0699356847396194 0.00300000000000614 0.000199999999999378 rpy=1.95799899548702E-16 2.29686057908074E-16 0.700079983587682 -> xyz=0.0699356847396164 0.00300000000001083 0.000199999999999378 rpy=1.95799899548702E-16 2.29686057908074E-16 0.700079983587682
- joint j21: parent base_link -> hand_base

File: robots/WAM_URDF.URDF (robot description, URDF)
Before this commit: robot WAM_URDF, 8 links, 7 joints
Links:
- link wam2: mass 0.437815219798136 -> 0.437815219798137
- link wam3: mass 5.1434314783609E-05 -> 5.14343147836089E-05
Joints:
- joint j7: origin xyz=0 -0.0600000000000009 0 rpy=1.5707963267949 0 0 -> xyz=0 0 0 rpy=1.5707963267949 0 0

File: robots/herb.urdf.xacro (robot description, xacro)
@@ -9,9 +9,9 @@
         <xacro:bh280 prefix="${prefix}"/>
         <xacro:wam prefix="${prefix}"/>
-        <joint name="${prefix}/mount" type="fixed">
+        <joint name="${prefix}/hand_mount" type="fixed">
             <!-- The force/torque sensor is 12 mm thick. -->
-            <origin xyz="0 0 0.012" rpy="0 0 ${-pi/2}"/>
+            <origin xyz="0 0 0.072" rpy="0 0 ${pi/2}"/>
             <parent link="${prefix}/wam7"/>
-            <child link="${prefix}/base_link"/>
+            <child link="${prefix}/hand_base"/>
         </joint>
     </xacro:macro>

Commit message: Fixing mimic joints

File: config/bh280_params.urdf.xacro (robot description, xacro)
@@ -20,4 +20,5 @@
         <joint name="j${index}2">
             <limit lower="0" upper="${48*(pi/180)}" effort="0" velocity="2.0"/>
+            <mimic joint="j${index}1" multiplier="${45./140.}" offset="0.0"/>
         </joint>
         <!-- Frame 3 (fingertip frame) with fingertip pressure pad -->
@@ -29,4 +30,21 @@
                                            iyy="1.6948e-005" iyz="-1.8635e-008"
                                                              izz= "1.5809e-005"/>
+            </inertial>
+        </link>
+    </xacro:macro>
+    <!-- Define the spread for 1 seperately so we can do the mimic joint -->
+    <xacro:macro name="bh280_spread1">
+        <joint name="j10">
+            <limit lower="0" upper="${180*(pi/180)}" effort="0" velocity="2.0"/>
+            <mimic joint="j00" multiplier="1" offset="0"/>
+        </joint>
+        <!-- Frame 1 (finger spread frame) -->
+        <link name="finger1_0">
+            <inertial>
+                <origin xyz="0.030616 -7.3219e-005 -0.011201"/>
+                <mass value="0.14109"/>
+                <inertia ixx="2.0672e-005" ixy="2.6024e-007" ixz="6.3481e-006"
+                                           iyy="7.4105e-005" iyz="1.7118e-008"
+                                                             izz="6.8207e-005"/>
             </inertial>
         </link>
@@ -59,5 +77,5 @@
     <!-- Fingers -->
     <xacro:bh280_spread index="0"/>
-    <xacro:bh280_spread index="1"/>
+    <xacro:bh280_spread1 />
     <xacro:bh280_finger index="0"/>
     <xacro:bh280_finger index="1"/>

Commit message: Fixed the spread joint on the BH280.

File: config/bh280_params.urdf.xacro (robot description, xacro)
@@ -33,11 +33,19 @@
         </link>
     </xacro:macro>
-    <!-- Define the spread for 1 seperately so we can do the mimic joint -->
-    <xacro:macro name="bh280_spread1">
-        <joint name="j10">
+    <xacro:macro name="bh280_spread">
+        <!-- Frame 0 spread -->
+        <link name="finger0_0">
+            <inertial>
+                <origin xyz="0.030616 -7.3219e-005 -0.011201"/>
+                <mass value="0.14109"/>
+                <inertia ixx="2.0672e-005" ixy="2.6024e-007" ixz="6.3481e-006"
+                                           iyy="7.4105e-005" iyz="1.7118e-008"
+                                                             izz="6.8207e-005"/>
+            </inertial>
+        </link>
+        <joint name="j00">
             <limit lower="0" upper="${180*(pi/180)}" effort="0" velocity="2.0"/>
-            <mimic joint="j00" multiplier="1" offset="0"/>
         </joint>
-        <!-- Frame 1 (finger spread frame) -->
+        <!-- Frame 1 spread (mimic joint) -->
         <link name="finger1_0">
             <inertial>
@@ -49,19 +57,8 @@
             </inertial>
         </link>
-    </xacro:macro>
-    <xacro:macro name="bh280_spread" params="index">
-        <joint name="j${index}0">
-            <limit lower="0" upper="${180*(pi/180)}" effort="0" velocity="2.0"/>
+        <joint name="j10">
+            <limit lower="${-180*(pi/180)}" upper="0" effort="0" velocity="2.0"/>
+            <mimic joint="j00" multiplier="-1" offset="0"/>
         </joint>
-        <!-- Frame 1 (finger spread frame) -->
-        <link name="finger${index}_0">
-            <inertial>
-                <origin xyz="0.030616 -7.3219e-005 -0.011201"/>
-                <mass value="0.14109"/>
-                <inertia ixx="2.0672e-005" ixy="2.6024e-007" ixz="6.3481e-006"
-                                           iyy="7.4105e-005" iyz="1.7118e-008"
-                                                             izz="6.8207e-005"/>
-            </inertial>
-        </link>
     </xacro:macro>
     <!-- Frame W with palm pad -->
@@ -75,7 +72,5 @@
         </inertial>
     </link>
-    <!-- Fingers -->
-    <xacro:bh280_spread index="0"/>
-    <xacro:bh280_spread1 />
+    <xacro:bh280_spread/>
     <xacro:bh280_finger index="0"/>
     <xacro:bh280_finger index="1"/>

Commit message: Fixed the axis of the finger spread joint.

File: config/bh280_params.urdf.xacro (robot description, xacro)
@@ -58,6 +58,6 @@
         </link>
         <joint name="j10">
-            <limit lower="${-180*(pi/180)}" upper="0" effort="0" velocity="2.0"/>
-            <mimic joint="j00" multiplier="-1" offset="0"/>
+            <limit lower="0" upper="${180*(pi/180)}" effort="0" velocity="2.0"/>
+            <mimic joint="j00" multiplier="1" offset="0"/>
         </joint>
     </xacro:macro>

Commit message: Fixed an incorrect (and huge) link mass on BH280.

File: config/bh280_params.urdf.xacro (robot description, xacro)
@@ -23,5 +23,5 @@
         </joint>
         <!-- Frame 3 (fingertip frame) with fingertip pressure pad -->
-        <link name="finger${index}_1">
+        <link name="finger${index}_2">
             <inertial>
                 <origin xyz="0.02295 0.0010739 0.00041752"/>

Commit message: Generate a DAE file. Fixed joint limits.

File: config/bh280_params.urdf.xacro (robot description, xacro)
@@ -4,5 +4,5 @@
     <xacro:macro name="bh280_finger" params="index">
         <!-- proximal joint -->
-        <joint name="j${index}1">
+        <joint name="j${index}1" type="revolute">
             <limit lower="0" upper="${140*(pi/180)}" effort="0" velocity="2.0"/>
         </joint>
@@ -18,5 +18,5 @@
         </link>
         <!-- distal joint -->
-        <joint name="j${index}2">
+        <joint name="j${index}2" type="revolute">
             <limit lower="0" upper="${48*(pi/180)}" effort="0" velocity="2.0"/>
             <mimic joint="j${index}1" multiplier="${45./140.}" offset="0.0"/>
@@ -44,5 +44,5 @@
             </inertial>
         </link>
-        <joint name="j00">
+        <joint name="j00" type="revolute">
             <limit lower="0" upper="${180*(pi/180)}" effort="0" velocity="2.0"/>
         </joint>
@@ -57,5 +57,5 @@
             </inertial>
         </link>
-        <joint name="j10">
+        <joint name="j10" type="revolute">
             <limit lower="0" upper="${180*(pi/180)}" effort="0" velocity="2.0"/>
             <mimic joint="j00" multiplier="1" offset="0"/>

File: config/wam_params.urdf.xacro (robot description, xacro)
@@ -85,24 +85,24 @@
          [2] http://support.barrett.com/wiki/WAM/CableTorqueLimits
     -->
-    <joint name="j1">
+    <joint name="j1" type="revolute">
         <!-- HERB's J1 joints are modified to have a +180 degree offset. -->
         <limit lower="${30*(pi/180)}" upper="${330*(pi/180)}" effort="1.8" velocity="0.75"/>
     </joint>
-    <joint name="j2">
+    <joint name="j2" type="revolute">
         <limit lower="${-113*(pi/180)}" upper="${113*(pi/180)}" effort="1.8" velocity="0.75"/>
     </joint>
-    <joint name="j3">
+    <joint name="j3" type="revolute">
         <limit lower="${-157*(pi/180)}" upper="${157*(pi/180)}" effort="1.8" velocity="2.0"/>
     </joint>
-    <joint name="j4">
+    <joint name="j4" type="revolute">
         <limit lower="${-50*(pi/180)}" upper="${180*(pi/180)}" effort="1.6" velocity="2.0"/>
     </joint>
-    <joint name="j5">
+    <joint name="j5" type="revolute">
         <limit lower="${-273*(pi/180)}" upper="${71*(pi/180)}" effort="0.6" velocity="2.5"/>
     </joint>
-    <joint name="j6">
+    <joint name="j6" type="revolute">
         <limit lower="${-90*(pi/180)}" upper="${90*(pi/180)}" effort="0.6" velocity="2.5"/>
     </joint>
-    <joint name="j7">
+    <joint name="j7" type="revolute">
         <limit lower="${-172*(pi/180)}" upper="${172*(pi/180)}" effort="0.174" velocity="2.5"/>
     </joint>
