Commit message: Changing joint limits to match those hardcoded in owd

File: config/wam_params.urdf.xacro (robot description, xacro)
@@ -78,32 +78,32 @@
         </inertial>
     </link>
-    <!-- The joint limits [1] and torque values [2] were copied from Barrett's
-         online documentation. The velocity limits are set to the default
+    <!-- The torque values [1] were copied from Barrett's
+         online documentation. The joint limits are set to the default
+         values used in OWD as of 10/9/2015. The velocity limits are set to the default
          values used in OWD as of 7/15/2013. The soft limits specified in the
          safety controller are padded by 0.1 radians.
-         [1] http://support.barrett.com/wiki/WAM/KinematicsJointRangesConversionFactors
-         [2] http://support.barrett.com/wiki/WAM/CableTorqueLimits
+         [1] http://support.barrett.com/wiki/WAM/CableTorqueLimits
     -->
     <joint name="j1" type="revolute">
         <!-- HERB's J1 joints are modified to have a +180 degree offset. -->
-        <limit lower="${30*(pi/180)}" upper="${330*(pi/180)}" effort="1.8" velocity="0.75"/>
+        <limit lower="${-2.60+pi}" upper="${2.60+pi}" effort="1.8" velocity="0.75"/>
     </joint>
     <joint name="j2" type="revolute">
-        <limit lower="${-113*(pi/180)}" upper="${113*(pi/180)}" effort="1.8" velocity="0.75"/>
+        <limit lower="-1.96" upper="1.96" effort="1.8" velocity="0.75"/>
     </joint>
     <joint name="j3" type="revolute">
-        <limit lower="${-157*(pi/180)}" upper="${157*(pi/180)}" effort="1.8" velocity="2.0"/>
+        <limit lower="-2.73" upper="2.73" effort="1.8" velocity="2.0"/>
     </joint>
     <joint name="j4" type="revolute">
-        <limit lower="${-50*(pi/180)}" upper="${180*(pi/180)}" effort="1.6" velocity="2.0"/>
+        <limit lower="-0.86" upper="3.13" effort="1.6" velocity="2.0"/>
     </joint>
     <joint name="j5" type="revolute">
-        <limit lower="${-273*(pi/180)}" upper="${71*(pi/180)}" effort="0.6" velocity="2.5"/>
+        <limit lower="-4.79" upper="1.30" effort="0.6" velocity="2.5"/>
     </joint>
     <joint name="j6" type="revolute">
-        <limit lower="${-90*(pi/180)}" upper="${90*(pi/180)}" effort="0.6" velocity="2.5"/>
+        <limit lower="-1.56" upper="1.56" effort="0.6" velocity="2.5"/>
     </joint>
     <joint name="j7" type="revolute">
-        <limit lower="${-172*(pi/180)}" upper="${172*(pi/180)}" effort="0.174" velocity="2.5"/>
+        <limit lower="-2.99" upper="2.99" effort="0.174" velocity="2.5"/>
     </joint>
 </template>

Commit message: use inertial values from owd for WAM

File: config/wam_params.urdf.xacro (robot description, xacro)
@@ -1,5 +1,5 @@
 <template xmlns:xacro="http://www.ros.org/wiki/xacro">
     <xacro:property name="pi" value="3.14159265359"/>
-    <!-- Inertial parameters were copied from the Barrett WAM User Manual,
+    <!-- Inertial mass and COM are from OWD, other inertial parameters were copied from the Barrett WAM User Manual,
          version AC_02. -->
     <link name="wam_base">
@@ -15,8 +15,8 @@
         <inertial>
             <origin xyz="-0.00443422 0.12189039 -0.00066489"/>
-            <mass value="10.76768767"/>
-            <inertia ixx="0.13488033" ixy="-0.00213041" ixz="-0.00012485"
-                                      iyy= "0.11328369" iyz= "0.00068555"
-                                                        izz= "0.09046330"/>
+            <mass value="8.3936"/>
+            <inertia ixx="0.0003506" ixy="-0.00213041" ixz="-0.00012485"
+                                     iyy="0.1326795"   iyz= "0.00068555"
+                                                       izz= "0.0006286"/>
         </inertial>
     </link>
@@ -24,8 +24,8 @@
         <inertial>
             <origin xyz="-0.00236983 0.03105614 0.01542114"/>
-            <mass value="3.87493756"/>
-            <inertia ixx="0.02140958" ixy="0.00027172" ixz="+0.00002461"
-                                      iyy="0.01377875" iyz="-0.00181920"
-                                                       izz= "0.01558906"/>
+            <mass value="4.8487"/>
+            <inertia ixx="-0.000002230" ixy= "0.00027172" ixz="+0.00002461"
+                                        iyy="-0.0213924"  iyz="-0.00181920"
+                                                          izz= "0.0133754"/>
         </inertial>
     </link>
@@ -33,8 +33,8 @@
         <inertial>
             <origin xyz="-0.03825858 0.20750770 0.00003309"/>
-            <mass value="1.80228141"/>
-            <inertia ixx="0.05911077" ixy="-0.00249612" ixz= "0.00000738"
-                                      iyy= "0.00324550" iyz="-0.00001767"
-                                                        izz= "0.05927043"/>
+            <mass value="1.7251"/>
+            <inertia ixx="-0.0387565" ixy="-0.00249612" ixz= "0.00000738"
+                                      iyy= "0.2179078"  iyz="-0.00001767"
+                                                        izz= "0.0000252"/>
         </inertial>
     </link>
@@ -44,7 +44,7 @@
             <origin xyz="0.00498512 -0.00022942 0.13271662"/>
             <mass value="2.40016804"/>
-            <inertia ixx="0.01491672" ixy="0.00001741" ixz="-0.00150604"
-                                      iyy="0.01482922" iyz="-0.00002109"
-                                                       izz= "0.00294463"/>
+            <inertia ixx="0.00498512" ixy= "0.00001741" ixz="-0.00150604"
+                                      iyy="-0.00022942" iyz="-0.00002109"
+                                                        izz= "0.13271662"/>
         </inertial>
     </link>
@@ -52,8 +52,8 @@
         <inertial>
             <origin xyz="0.00008921 0.00511217 0.00435824"/>
-            <mass value="0.12376019"/>
-            <inertia ixx="0.00005029" ixy="0.00000020" ixz="-0.00000005"
-                                      iyy="0.00007582" iyz="-0.00000359"
-                                                       izz= "0.00006270"/>
+            <mass value="0.35655692"/>
+            <inertia ixx="0.00005483" ixy="0.00000020" ixz="-0.00000005"
+                                      iyy="0.02886286" iyz="-0.00000359"
+                                                       izz= "0.00148493"/>
         </inertial>
     </link>
@@ -61,8 +61,8 @@
         <inertial>
             <origin xyz="-0.00012262 -0.01703194 0.02468336"/>
-            <mass value="0.41797364"/>
-            <inertia ixx="0.00055516" ixy="0.00000061" ixz="-0.00000074"
-                                      iyy="0.00024367" iyz="-0.00004590"
-                                                       izz= "0.00045358"/>
+            <mass value="0.40915886"/>
+            <inertia ixx="-0.00005923" ixy= "0.00000061" ixz="-0.00000074"
+                                       iyy="-0.01686123" iyz="-0.00004590"
+                                                         izz= "0.02419052"/>
         </inertial>
     </link>
@@ -73,7 +73,7 @@
             <origin xyz="-0.00007974 0.00016313 -0.00323552"/>
             <mass value="0.06864753"/>
-            <inertia ixx="0.00003773" ixy="-0.00000019" ixz="0.00000000"
-                                      iyy= "0.00003806" iyz="0.00000000"
-                                                        izz="0.00007408"/>
+            <inertia ixx="0.00014836" ixy="-0.00000019" ixz= "0.00000000"
+                                      iyy= "0.00007252" iyz= "0.00000000"
+                                                        izz="-0.1232352"/>
         </inertial>
     </link>

Commit message: wrong place for COM

File: config/wam_params.urdf.xacro (robot description, xacro)
@@ -1,5 +1,5 @@
 <template xmlns:xacro="http://www.ros.org/wiki/xacro">
     <xacro:property name="pi" value="3.14159265359"/>
-    <!-- Inertial mass and COM are from OWD, other inertial parameters were copied from the Barrett WAM User Manual,
+    <!-- Inertial parameters were copied from the Barrett WAM User Manual,
          version AC_02. -->
     <link name="wam_base">
@@ -14,27 +14,27 @@
     <link name="wam1">
         <inertial>
-            <origin xyz="-0.00443422 0.12189039 -0.00066489"/>
+            <origin xyz="0.0003506 0.1326795 0.0006286"/>
             <mass value="8.3936"/>
-            <inertia ixx="0.0003506" ixy="-0.00213041" ixz="-0.00012485"
-                                     iyy="0.1326795"   iyz= "0.00068555"
-                                                       izz= "0.0006286"/>
+            <inertia ixx="0.13488033" ixy="-0.00213041" ixz="-0.00012485"
+                                      iyy= "0.11328369" iyz= "0.00068555"
+                                                        izz= "0.09046330"/>
         </inertial>
     </link>
     <link name="wam2">
         <inertial>
-            <origin xyz="-0.00236983 0.03105614 0.01542114"/>
+            <origin xyz="-0.000002230 -0.0213924 0.0133754"/>
             <mass value="4.8487"/>
-            <inertia ixx="-0.000002230" ixy= "0.00027172" ixz="+0.00002461"
-                                        iyy="-0.0213924"  iyz="-0.00181920"
-                                                          izz= "0.0133754"/>
+            <inertia ixx="0.02140958" ixy="0.00027172" ixz="+0.00002461"
+                                      iyy="0.01377875" iyz="-0.00181920"
+                                                       izz= "0.01558906"/>
         </inertial>
     </link>
     <link name="wam3">
         <inertial>
-            <origin xyz="-0.03825858 0.20750770 0.00003309"/>
+            <origin xyz="-0.0387565 0.2179078 0.0000252"/>
             <mass value="1.7251"/>
-            <inertia ixx="-0.0387565" ixy="-0.00249612" ixz= "0.00000738"
-                                      iyy= "0.2179078"  iyz="-0.00001767"
-                                                        izz= "0.0000252"/>
+            <inertia ixx="0.05911077" ixy="-0.00249612" ixz= "0.00000738"
+                                      iyy= "0.00324550" iyz="-0.00001767"
+                                                        izz= "0.05927043"/>
         </inertial>
     </link>
@@ -44,25 +44,25 @@
             <origin xyz="0.00498512 -0.00022942 0.13271662"/>
             <mass value="2.40016804"/>
-            <inertia ixx="0.00498512" ixy= "0.00001741" ixz="-0.00150604"
-                                      iyy="-0.00022942" iyz="-0.00002109"
-                                                        izz= "0.13271662"/>
+            <inertia ixx="0.01491672" ixy="0.00001741" ixz="-0.00150604"
+                                      iyy="0.01482922" iyz="-0.00002109"
+                                                       izz= "0.00294463"/>
         </inertial>
     </link>
     <link name="wam5">
         <inertial>
-            <origin xyz="0.00008921 0.00511217 0.00435824"/>
+            <origin xyz="0.00005483 0.02886286 0.00148493"/>
             <mass value="0.35655692"/>
-            <inertia ixx="0.00005483" ixy="0.00000020" ixz="-0.00000005"
-                                      iyy="0.02886286" iyz="-0.00000359"
-                                                       izz= "0.00148493"/>
+            <inertia ixx="0.00005029" ixy="0.00000020" ixz="-0.00000005"
+                                      iyy="0.00007582" iyz="-0.00000359"
+                                                       izz= "0.00006270"/>
         </inertial>
     </link>
     <link name="wam6">
         <inertial>
-            <origin xyz="-0.00012262 -0.01703194 0.02468336"/>
+            <origin xyz="-0.00005923 -0.01686123 0.02419052"/>
             <mass value="0.40915886"/>
-            <inertia ixx="-0.00005923" ixy= "0.00000061" ixz="-0.00000074"
-                                       iyy="-0.01686123" iyz="-0.00004590"
-                                                         izz= "0.02419052"/>
+            <inertia ixx="0.00055516" ixy="0.00000061" ixz="-0.00000074"
+                                      iyy="0.00024367" iyz="-0.00004590"
+                                                       izz= "0.00045358"/>
         </inertial>
     </link>
@@ -71,9 +71,9 @@
     <link name="wam7">
         <inertial>
-            <origin xyz="-0.00007974 0.00016313 -0.00323552"/>
+            <origin xyz="0.00014836 0.00007252 -0.1232352"/>
             <mass value="0.06864753"/>
-            <inertia ixx="0.00014836" ixy="-0.00000019" ixz= "0.00000000"
-                                      iyy= "0.00007252" iyz= "0.00000000"
-                                                        izz="-0.1232352"/>
+            <inertia ixx="0.00003773" ixy="-0.00000019" ixz="0.00000000"
+                                      iyy= "0.00003806" iyz="0.00000000"
+                                                        izz="0.00007408"/>
         </inertial>
     </link>

Commit message: Fixed COM offsets to match OWD.

File: config/wam_params.urdf.xacro (robot description, xacro)
@@ -12,7 +12,8 @@
         </inertial>
     </link>
+    <!-- TODO: Set wam0 to zero mass. -->
     <link name="wam1">
         <inertial>
-            <origin xyz="0.0003506 0.1326795 0.0006286"/>
+            <origin xyz="0.0003506  0.0006286 -0.1326795"/>
             <mass value="8.3936"/>
             <inertia ixx="0.13488033" ixy="-0.00213041" ixz="-0.00012485"
@@ -23,5 +24,5 @@
     <link name="wam2">
         <inertial>
-            <origin xyz="-0.000002230 -0.0213924 0.0133754"/>
+            <origin xyz="-0.000223  -0.0133754 -0.0213924"/>
             <mass value="4.8487"/>
             <inertia ixx="0.02140958" ixy="0.00027172" ixz="+0.00002461"
@@ -32,5 +33,5 @@
     <link name="wam3">
         <inertial>
-            <origin xyz="-0.0387565 0.2179078 0.0000252"/>
+            <origin xyz="0.0062435 0.0000252 0.3320922"/>
             <mass value="1.7251"/>
             <inertia ixx="0.05911077" ixy="-0.00249612" ixz= "0.00000738"
@@ -42,5 +43,5 @@
     <link name="wam4">
         <inertial>
-            <origin xyz="0.00498512 -0.00022942 0.13271662"/>
+            <origin xyz="-0.04001488 -0.13271662 -0.00022942"/>
             <mass value="2.40016804"/>
             <inertia ixx="0.01491672" ixy="0.00001741" ixz="-0.00150604"
@@ -51,5 +52,5 @@
     <link name="wam5">
         <inertial>
-            <origin xyz="0.00005483 0.02886286 0.00148493"/>
+            <origin xyz="0.00005483 0.00148493 0.27113714"/>
             <mass value="0.35655692"/>
             <inertia ixx="0.00005029" ixy="0.00000020" ixz="-0.00000005"
@@ -60,5 +61,5 @@
     <link name="wam6">
         <inertial>
-            <origin xyz="-0.00005923 -0.01686123 0.02419052"/>
+            <origin xyz="-0.00005923 -0.02419052 -0.01686123"/>
             <mass value="0.40915886"/>
             <inertia ixx="0.00055516" ixy="0.00000061" ixz="-0.00000074"
@@ -71,5 +72,5 @@
     <link name="wam7">
         <inertial>
-            <origin xyz="0.00014836 0.00007252 -0.1232352"/>
+            <origin xyz="0 0 0.104"/>
             <mass value="0.06864753"/>
             <inertia ixx="0.00003773" ixy="-0.00000019" ixz="0.00000000"

Commit message: Revert "Fixed COM offsets to match OWD."
This reverts commit 91af45d67f3f96a066d3a5e7847ea461561cabe4.

File: config/wam_params.urdf.xacro (robot description, xacro)
@@ -12,8 +12,7 @@
         </inertial>
     </link>
-    <!-- TODO: Set wam0 to zero mass. -->
     <link name="wam1">
         <inertial>
-            <origin xyz="0.0003506  0.0006286 -0.1326795"/>
+            <origin xyz="0.0003506 0.1326795 0.0006286"/>
             <mass value="8.3936"/>
             <inertia ixx="0.13488033" ixy="-0.00213041" ixz="-0.00012485"
@@ -24,5 +23,5 @@
     <link name="wam2">
         <inertial>
-            <origin xyz="-0.000223  -0.0133754 -0.0213924"/>
+            <origin xyz="-0.000002230 -0.0213924 0.0133754"/>
             <mass value="4.8487"/>
             <inertia ixx="0.02140958" ixy="0.00027172" ixz="+0.00002461"
@@ -33,5 +32,5 @@
     <link name="wam3">
         <inertial>
-            <origin xyz="0.0062435 0.0000252 0.3320922"/>
+            <origin xyz="-0.0387565 0.2179078 0.0000252"/>
             <mass value="1.7251"/>
             <inertia ixx="0.05911077" ixy="-0.00249612" ixz= "0.00000738"
@@ -43,5 +42,5 @@
     <link name="wam4">
         <inertial>
-            <origin xyz="-0.04001488 -0.13271662 -0.00022942"/>
+            <origin xyz="0.00498512 -0.00022942 0.13271662"/>
             <mass value="2.40016804"/>
             <inertia ixx="0.01491672" ixy="0.00001741" ixz="-0.00150604"
@@ -52,5 +51,5 @@
     <link name="wam5">
         <inertial>
-            <origin xyz="0.00005483 0.00148493 0.27113714"/>
+            <origin xyz="0.00005483 0.02886286 0.00148493"/>
             <mass value="0.35655692"/>
             <inertia ixx="0.00005029" ixy="0.00000020" ixz="-0.00000005"
@@ -61,5 +60,5 @@
     <link name="wam6">
         <inertial>
-            <origin xyz="-0.00005923 -0.02419052 -0.01686123"/>
+            <origin xyz="-0.00005923 -0.01686123 0.02419052"/>
             <mass value="0.40915886"/>
             <inertia ixx="0.00055516" ixy="0.00000061" ixz="-0.00000074"
@@ -72,5 +71,5 @@
     <link name="wam7">
         <inertial>
-            <origin xyz="0 0 0.104"/>
+            <origin xyz="0.00014836 0.00007252 -0.1232352"/>
             <mass value="0.06864753"/>
             <inertia ixx="0.00003773" ixy="-0.00000019" ixz="0.00000000"

Commit message: Fixed <inertial> <origin> orientation.

File: config/wam_params.urdf.xacro (robot description, xacro)
@@ -5,5 +5,5 @@
     <link name="wam_base">
         <inertial>
-            <origin xyz="-0.02017671 -0.26604706 -0.14071720"/>
+            <origin xyz="0 0 0" rpy="0 0 0"/>
             <mass value="9.97059584"/>
             <inertia ixx="0.10916849" ixy="0.00640270" ixz="0.02557874"
@@ -14,5 +14,5 @@
     <link name="wam1">
         <inertial>
-            <origin xyz="0.0003506 0.1326795 0.0006286"/>
+            <origin xyz="0.000351 0.000629 -0.132680" rpy="-1.570796 0 0"/>
             <mass value="8.3936"/>
             <inertia ixx="0.13488033" ixy="-0.00213041" ixz="-0.00012485"
@@ -23,5 +23,5 @@
     <link name="wam2">
         <inertial>
-            <origin xyz="-0.000002230 -0.0213924 0.0133754"/>
+            <origin xyz="-0.000223 -0.013375 -0.021392" rpy="1.570796 0 0"/>
             <mass value="4.8487"/>
             <inertia ixx="0.02140958" ixy="0.00027172" ixz="+0.00002461"
@@ -32,5 +32,5 @@
     <link name="wam3">
         <inertial>
-            <origin xyz="-0.0387565 0.2179078 0.0000252"/>
+            <origin xyz="0.006243 0.000025 0.332092" rpy="-1.570796 0 0"/>
             <mass value="1.7251"/>
             <inertia ixx="0.05911077" ixy="-0.00249612" ixz= "0.00000738"
@@ -42,5 +42,5 @@
     <link name="wam4">
         <inertial>
-            <origin xyz="0.00498512 -0.00022942 0.13271662"/>
+            <origin xyz="-0.040015 -0.132717 -0.000229" rpy="1.570796 0 0"/>
             <mass value="2.40016804"/>
             <inertia ixx="0.01491672" ixy="0.00001741" ixz="-0.00150604"
@@ -51,5 +51,5 @@
     <link name="wam5">
         <inertial>
-            <origin xyz="0.00005483 0.02886286 0.00148493"/>
+            <origin xyz="0.000055 0.001485 0.271137" rpy="-1.570796 0 0"/>
             <mass value="0.35655692"/>
             <inertia ixx="0.00005029" ixy="0.00000020" ixz="-0.00000005"
@@ -60,5 +60,5 @@
     <link name="wam6">
         <inertial>
-            <origin xyz="-0.00005923 -0.01686123 0.02419052"/>
+            <origin xyz="-0.000059 -0.024191 -0.016861" rpy="1.570796 0 0"/>
             <mass value="0.40915886"/>
             <inertia ixx="0.00055516" ixy="0.00000061" ixz="-0.00000074"
@@ -71,5 +71,5 @@
     <link name="wam7">
         <inertial>
-            <origin xyz="0.00014836 0.00007252 -0.1232352"/>
+            <origin xyz="0 0 0.104" rpy="0 0 0"/>
             <mass value="0.06864753"/>
             <inertia ixx="0.00003773" ixy="-0.00000019" ixz="0.00000000"
