Commit message: Changed head velocity limits to match OWD/Pantilt.

File: config/herb_params.urdf.xacro (robot description, xacro)
@@ -2,8 +2,8 @@
     <xacro:property name="pi" value="3.14159265359"/>
     <joint name="head/wam1">
-        <limit lower="${-160*(pi/180)}" upper="${160*(pi/180)}" effort="0.517" velocity="3.0"/>
+        <limit lower="${-160*(pi/180)}" upper="${160*(pi/180)}" effort="0.517" velocity="2.5"/>
     </joint>
     <joint name="head/wam2">
-        <limit lower="${-71.5*(pi/180)}" upper="${71.5*(pi/180)}" effort="0.110" velocity="3.0"/>
+        <limit lower="${-71.5*(pi/180)}" upper="${71.5*(pi/180)}" effort="0.110" velocity="2.5"/>
     </joint>
 </template>

Commit message: Force the head joints to be revolute.
These were exported from SolidWorks as CONTINUOUS.

File: config/herb_params.urdf.xacro (robot description, xacro)
@@ -1,8 +1,8 @@
 <template xmlns:xacro="http://www.ros.org/wiki/xacro">
     <xacro:property name="pi" value="3.14159265359"/>
-    <joint name="head/wam1">
+    <joint name="head/wam1" type="revolute">
         <limit lower="${-160*(pi/180)}" upper="${160*(pi/180)}" effort="0.517" velocity="2.5"/>
     </joint>
-    <joint name="head/wam2">
+    <joint name="head/wam2" type="revolute">
         <limit lower="${-71.5*(pi/180)}" upper="${71.5*(pi/180)}" effort="0.110" velocity="2.5"/>
     </joint>

Commit message: remove revolute head params: actually fixed joint

File: config/herb_params.urdf.xacro (robot description, xacro)
@@ -1,9 +1,3 @@
 <template xmlns:xacro="http://www.ros.org/wiki/xacro">
     <xacro:property name="pi" value="3.14159265359"/>
-    <joint name="head/wam1" type="revolute">
-        <limit lower="${-160*(pi/180)}" upper="${160*(pi/180)}" effort="0.517" velocity="2.5"/>
-    </joint>
-    <joint name="head/wam2" type="revolute">
-        <limit lower="${-71.5*(pi/180)}" upper="${71.5*(pi/180)}" effort="0.110" velocity="2.5"/>
-    </joint>
 </template>

File: robots/HERB_BASE_URDF.URDF (robot description, URDF)
Before this commit: robot HERB_BASE_URDF, 5 links, 4 joints
Joints:
- joint head/wam2: type continuous -> fixed
